File: GVS-32U4/GVS-32U4.sch (KiCad schematic (older format))
At the start: 47 parts, among them J1 USB-B, K1 CONN_3, K10 CONN_3, K11 CONN_3, K12 CONN_3, K13 CONN_3, K14 CONN_3, K15 CONN_3, K16 CONN_3, K17 CONN_3, K18 CONN_3, K19 CONN_3, K2 CONN_3, K20 CONN_3, K21 CONN_3, K22 CONN_3, K23 CONN_3, K24 CONN_3, K25 CONN_3, K26 CONN_3, K27 CONN_3, K3 CONN_3, K4 CONN_3, K5 CONN_3, K6 CONN_3, K7 CONN_3, K8 CONN_3, K9 CONN_3, P1 CONN_2, U1 ATMEGA32U4-AU, U2 AP1117, X1 16MHz

Commit message: GVS-32U4 layout done
Parts:
- removed K1, K10, K11, K12, K13, K14, K15, K16, K17, K18, K19, K2, K20, K21, K22, K23, K24, K25, K26, K3, K4, K5, K6, K7, K8, K9: CONN_3, symbol CONN_3
- added J10, J11, J12, J13, J14, J15, J16, J17, J18, J19, J2, J20, J21, J22, J23, J24, J25, J26, J27, J3, J4, J5, J6, J7, J8, J9: GVS, PIN_ARRAY_3X1, symbol GVS
- C2, C3: value C -> 0.1uF; footprint (none) -> SM0805
- J28: renamed from K27; footprint (none) -> PIN_ARRAY_3X1
- J29: renamed from P1; footprint (none) -> PIN_ARRAY_2X1
- U2: footprint (none) -> SOT223
- X1: footprint (none) -> RESON_3PIN

Commit message: update 32u4 gvs board
Parts:
- removed J4: GVS, PIN_ARRAY_3X1, symbol GVS
- added J30, J4: CONN_2, symbol CONN_2
Connections:
- wire segments 182 -> 183

Commit message: Updated the GVS-32U4 and USB-GPSX2 designs
Parts:
- C1: Vendor (none) -> Mouser; VendorPN (none) -> 77-VJ0805Y105MXQTBC
- C2, C3, C5: Vendor (none) -> Mouser; VendorPN (none) -> 581-08055C104KAT9A
- C4: Vendor (none) -> Mouser; VendorPN (none) -> 581-0805YD106K
- DS2: Vendor (none) -> Mouser; VendorPN (none) -> 859-LTST-C170KRKT
- F1: Vendor (none) -> Mouser; VendorPN (none) -> 504-PTS120615V050
- J1: Vendor (none) -> Mouser; VendorPN (none) -> 798-UX60SC-MB-5ST80
- J10, J11, J12, J13, J14, J15, J16, J17, J18, J19, J2, J20, J21, J22, J23, J24, J25, J26, J27, J28, J3, J5, J6, J7, J8, J9: Vendor (none) -> Mouser; VendorPN (none) -> 649-69190-103HLF
- J29, J30, J4: Vendor (none) -> Mouser; VendorPN (none) -> 649-93287-202HLF
- MTG1, MTG2, MTG3, MTG4: Vendor (none) -> N/A; VendorPN (none) -> 4-40 Hole
- R1, R2: Vendor (none) -> Mouser; VendorPN (none) -> 260-22-RC
- R3: Vendor (none) -> Mouser; VendorPN (none) -> 652-CR0805JW-271ELF
- R9: Vendor (none) -> Mouser; VendorPN (none) -> 260-10K-RC
- U1: Vendor (none) -> Mouser; VendorPN (none) -> 556-ATMEGA32U4-AU
- U2: Vendor (none) -> Mouser; VendorPN (none) -> 621-AP1117Y50G-13
- X1: Vendor (none) -> Mouser; VendorPN (none) -> 81-CSTLS16M0X51-A0
