File: GVS-32U4/GVS-32U4-X3.sch (KiCad schematic (older format))
At the start: 52 parts, among them J1 USB-B, J10 GVS, J11 GVS, J12 GVS, J13 GVS, J14 GVS, J15 GVS, J16 GVS, J17 GVS, J18 GVS, J19 GVS, J2 GVS, J20 GVS, J21 GVS, J22 GVS, J23 GVS, J24 GVS, J25 GVS, J26 GVS, J27 GVS, J28 CONN_3, J29 CONN_2, J3 GVS, J30 CONN_2, J4 GVS, J5 GVS, J6 GVS, J7 GVS, J8 CONN_2, J9 GVS, U1 ATMEGA32U4-AU, U2 AP1117, X1 16MHz

Commit message: GVS-32U4 updates for Rev X3.
Parts:
- added C8: 0.1uF, SM0805, symbol C
- added C9: 0.01uF, SM0805, symbol C
- added L1: 10uH, SM0805, symbol INDUCTOR
- J30, J8: footprint (none) -> PIN_ARRAY_2X1
- R4: footprint (none) -> SM0805
Connections:
- net labels added: AVCC, VUSB
- net labels removed: VFUSE
- wire segments 188 -> 196
Changed lines of the file:
@@
-EESchema Schematic File Version 2  date 5/7/2013 1:24:17 PM
+EESchema Schematic File Version 2  date 27/06/2013 10:09:17
 LIBS:transistors
 LIBS:special
@@
 LIBS:atmega32u4bb-from_eagle
 LIBS:DougsSch
-LIBS:GVS-32U4-X2-cache
+LIBS:GVS-32U4-X3-cache
 EELAYER 27 0
 EELAYER END
@@
 Sheet 1 1
 Title "GVS-32U4"
-Date "7 may 2013"
+Date "27 jun 2013"
 Rev "X1"
-Comp "AA6PR"
+Comp "dougspcbdesigns.pbworks.com"
 Comment1 ""
 Comment2 ""
@@
 	3500 850  3500 800
 Wire Wire Line
-	3200 1500 3200 2250
-Wire Wire Line
 	10150 6950 10150 7050
 Wire Wire Line
@@
 	1750 2250 1750 1950
 Wire Wire Line
-	3800 2050 3200 2050
+	3200 2050 3800 2050
 Wire Wire Line
 	3200 2250 3800 2250
-Connection ~ 3200 2050
 Wire Wire Line
 	3800 2150 3650 2150
@@
 F 0 "J8" V 7800 3350 40  0000 C CNN
 F 1 "CONN_2" V 7900 3350 40  0000 C CNN
-F 2 "" H 7850 3350 60  0001 C CNN
+F 2 "PIN_ARRAY_2X1" H 7850 3350 60  0001 C CNN
 F 3 "" H 7850 3350 60  0001 C CNN
 	1    7850 3350
@@
 $EndComp
 $Comp
-L +5V #PWR01
+L +5V #PWR6
 U 1 1 50A3DD27
 P 6550 1550
-F 0 "#PWR01" H 6550 1640 20  0001 C CNN
+F 0 "#PWR6" H 6550 1640 20  0001 C CNN
 F 1 "+5V" H 6550 1640 30  0000 C CNN
 F 2 "" H 6550 1550 60  0001 C CNN
@@
 F 0 "R4" V 6630 1850 50  0000 C CNN
 F 1 "10K" V 6550 1850 50  0000 C CNN
-F 2 "" H 6550 1850 60  0001 C CNN
+F 2 "SM0805" H 6550 1850 60  0001 C CNN
 F 3 "" H 6550 1850 60  0001 C CNN
 	1    6550 1850
@@
 F 0 "J30" V 10100 5200 40  0000 C CNN
 F 1 "CONN_2" V 10200 5200 40  0000 C CNN
-F 2 "" H 10150 5200 60  0001 C CNN
+F 2 "PIN_ARRAY_2X1" H 10150 5200 60  0001 C CNN
 F 3 "" H 10150 5200 60  0001 C CNN
 F 4 "Mouser" H 10150 5200 60  0001 C CNN "Vendor"
@@
 VIN
 $Comp
-L GND #PWR02
+L GND #PWR21
 U 1 1 5055FD17
 P 1500 6600
-F 0 "#PWR02" H 1500 6600 30  0001 C CNN
+F 0 "#PWR21" H 1500 6600 30  0001 C CNN
 F 1 "GND" H 1500 6530 30  0001 C CNN
 F 2 "" H 1500 6600 60  0001 C CNN
@@
 $EndComp
 $Comp
-L +5V #PWR03
+L +5V #PWR15
 U 1 1 5055F853
 P 9600 4400
-F 0 "#PWR03" H 9600 4490 20  0001 C CNN
+F 0 "#PWR15" H 9600 4490 20  0001 C CNN
 F 1 "+5V" H 9600 4490 30  0000 C CNN
 F 2 "" H 9600 4400 60  0001 C CNN
@@
 $EndComp
 $Comp
-L GND #PWR04
+L GND #PWR18
 U 1 1 5055F84C
 P 9700 5450
-F 0 "#PWR04" H 9700 5450 30  0001 C CNN
+F 0 "#PWR18" H 9700 5450 30  0001 C CNN
 F 1 "GND" H 9700 5380 30  0001 C CNN
 F 2 "" H 9700 5450 60  0001 C CNN
@@
 $EndComp
 Text Label 2100 1350 0    60   ~ 0
-VFUSE
+VUSB
 Text Label 2650 4850 0    60   ~ 0
-VFUSE
+VUSB
 $Comp
 L C C3
@@
 $EndComp
 $Comp
-L GND #PWR05
+L GND #PWR10
 U 1 1 5055E039
 P 3000 3700
-F 0 "#PWR05" H 3000 3700 30  0001 C CNN
+F 0 "#PWR10" H 3000 3700 30  0001 C CNN
 F 1 "GND" H 3000 3630 30  0001 C CNN
 F 2 "" H 3000 3700 60  0001 C CNN
@@
 $EndComp
 $Comp
-L +5V #PWR06
+L +5V #PWR5
 U 1 1 5055D7A5
 P 3200 1500
-F 0 "#PWR06" H 3200 1590 20  0001 C CNN
+F 0 "#PWR5" H 3200 1590 20  0001 C CNN
 F 1 "+5V" H 3200 1590 30  0000 C CNN
 F 2 "" H 3200 1500 60  0001 C CNN
@@
 $EndComp
 $Comp
-L +5V #PWR07
+L +5V #PWR1
 U 1 1 5055D7A1
 P 3500 800
-F 0 "#PWR07" H 3500 890 20  0001 C CNN
+F 0 "#PWR1" H 3500 890 20  0001 C CNN
 F 1 "+5V" H 3500 890 30  0000 C CNN
 F 2 "" H 3500 800 60  0001 C CNN
@@
 PF0
 $Comp
-L +5V #PWR08
+L +5V #PWR2
 U 1 1 5055D48E
 P 7300 1300
-F 0 "#PWR08" H 7300 1390 20  0001 C CNN
+F 0 "#PWR2" H 7300 1390 20  0001 C CNN
 F 1 "+5V" H 7300 1390 30  0000 C CNN
 F 2 "" H 7300 1300 60  0001 C CNN
@@
 $EndComp
 $Comp
-L GND #PWR09
+L GND #PWR12
 U 1 1 5055D48D
 P 7400 3900
-F 0 "#PWR09" H 7400 3900 30  0001 C CNN
+F 0 "#PWR12" H 7400 3900 30  0001 C CNN
 F 1 "GND" H 7400 3830 30  0001 C CNN
 F 2 "" H 7400 3900 60  0001 C CNN
@@
 $EndComp
 $Comp
-L GND #PWR010
+L GND #PWR13
 U 1 1 5055D47C
 P 8600 3900
-F 0 "#PWR010" H 8600 3900 30  0001 C CNN
+F 0 "#PWR13" H 8600 3900 30  0001 C CNN
 F 1 "GND" H 8600 3830 30  0001 C CNN
 F 2 "" H 8600 3900 60  0001 C CNN
@@
 $EndComp
 $Comp
-L +5V #PWR011
+L +5V #PWR3
 U 1 1 5055D47B
 P 8500 1300
-F 0 "#PWR011" H 8500 1390 20  0001 C CNN
+F 0 "#PWR3" H 8500 1390 20  0001 C CNN
 F 1 "+5V" H 8500 1390 30  0000 C CNN
 F 2 "" H 8500 1300 60  0001 C CNN
@@
 $EndComp
 $Comp
-L +5V #PWR012
+L +5V #PWR4
 U 1 1 5055D3F5
 P 9700 1300
-F 0 "#PWR012" H 9700 1390 20  0001 C CNN
+F 0 "#PWR4" H 9700 1390 20  0001 C CNN
 F 1 "+5V" H 9700 1390 30  0000 C CNN
 F 2 "" H 9700 1300 60  0001 C CNN
@@
 $EndComp
 $Comp
-L GND #PWR013
+L GND #PWR14
 U 1 1 5055D3E5
 P 9800 3900
-F 0 "#PWR013" H 9800 3900 30  0001 C CNN
+F 0 "#PWR14" H 9800 3900 30  0001 C CNN
 F 1 "GND" H 9800 3830 30  0001 C CNN
 F 2 "" H 9800 3900 60  0001 C CNN
@@
 NoConn ~ 3800 3050
 $Comp
-L +5V #PWR014
+L +5V #PWR22
 U 1 1 50510DFF
 P 700 7050
-F 0 "#PWR014" H 700 7140 20  0001 C CNN
+F 0 "#PWR22" H 700 7140 20  0001 C CNN
 F 1 "+5V" H 700 7140 30  0000 C CNN
 F 2 "" H 700 7050 60  0001 C CNN
@@
 $EndComp
 $Comp
-L GND #PWR015
+L GND #PWR25
 U 1 1 4EE20D15
 P 700 7900
-F 0 "#PWR015" H 700 7900 30  0001 C CNN
+F 0 "#PWR25" H 700 7900 30  0001 C CNN
 F 1 "GND" H 700 7830 30  0001 C CNN
 F 2 "" H 700 7900 60  0001 C CNN
@@
 $EndComp
 $Comp
-L GND #PWR016
+L GND #PWR23
 U 1 1 4EE20D00
 P 10150 7050
-F 0 "#PWR016" H 10150 7050 30  0001 C CNN
+F 0 "#PWR23" H 10150 7050 30  0001 C CNN
 F 1 "GND" H 10150 6980 30  0001 C CNN
 F 2 "" H 10150 7050 60  0001 C CNN
@@
 $EndComp
 $Comp
-L GND #PWR017
+L GND #PWR8
 U 1 1 4EE20C7E
 P 2200 3050
-F 0 "#PWR017" H 2200 3050 30  0001 C CNN
+F 0 "#PWR8" H 2200 3050 30  0001 C CNN
 F 1 "GND" H 2200 2980 30  0001 C CNN
 F 2 "" H 2200 3050 60  0001 C CNN
@@
 $EndComp
 $Comp
-L GND #PWR018
+L GND #PWR16
 U 1 1 4EE20C5D
 P 3800 4550
-F 0 "#PWR018" H 3800 4550 30  0001 C CNN
+F 0 "#PWR16" H 3800 4550 30  0001 C CNN
 F 1 "GND" H 3800 4480 30  0001 C CNN
 F 2 "" H 3800 4550 60  0001 C CNN
@@
 $EndComp
 $Comp
-L GND #PWR019
+L GND #PWR9
 U 1 1 4EE20C49
 P 1750 3150
-F 0 "#PWR019" H 1750 3150 30  0001 C CNN
+F 0 "#PWR9" H 1750 3150 30  0001 C CNN
 F 1 "GND" H 1750 3080 30  0001 C CNN
 F 2 "" H 1750 3150 60  0001 C CNN
@@
 $EndComp
 $Comp
-L +5V #PWR020
+L +5V #PWR7
 U 1 1 4EE20B8A
 P 3650 2150
-F 0 "#PWR020" H 3650 2240 20  0001 C CNN
+F 0 "#PWR7" H 3650 2240 20  0001 C CNN
 F 1 "+5V" H 3650 2240 30  0000 C CNN
 F 2 "" H 3650 2150 60  0001 C CNN
@@
 $EndComp
 $Comp
-L +5V #PWR021
+L +5V #PWR20
 U 1 1 4EE20B74
 P 10150 5850
-F 0 "#PWR021" H 10150 5940 20  0001 C CNN
+F 0 "#PWR20" H 10150 5940 20  0001 C CNN
 F 1 "+5V" H 10150 5940 30  0000 C CNN
 F 2 "" H 10150 5850 60  0001 C CNN
@@
 $EndComp
 $Comp
-L +5V #PWR022
+L +5V #PWR17
 U 1 1 4EE20B0F
 P 3600 5100
-F 0 "#PWR022" H 3600 5190 20  0001 C CNN
+F 0 "#PWR17" H 3600 5190 20  0001 C CNN
 F 1 "+5V" H 3600 5190 30  0000 C CNN
 F 2 "" H 3600 5100 60  0001 C CNN
@@
 Connection ~ 700  7800
 Connection ~ 1500 7100
+Wire Wire Line
+	3200 1500 3200 2050
+Text Label 3250 2250 0    60   ~ 0
+AVCC
+Wire Wire Line
+	5200 5700 5200 5700
+Wire Wire Line
+	5200 5700 5200 5800
+$Comp
+L INDUCTOR L1
+U 1 1 51CC4856
+P 5200 6100
+F 0 "L1" V 5150 6100 40  0000 C CNN
+F 1 "10uH" V 5300 6100 40  0000 C CNN
+F 2 "SM0805" V 5100 6100 60  0000 C CNN
+F 3 "" H 5200 6100 60  0000 C CNN
+	1    5200 6100
+	1    0    0    -1
+$EndComp
+$Comp
+L C C8
+U 1 1 51CC4865
+P 5200 6900
+F 0 "C8" H 5250 7000 50  0000 L CNN
+F 1 "0.1uF" H 5250 6800 50  0000 L CNN
+F 2 "SM0805" V 5050 6900 60  0000 C CNN
+F 3 "" H 5200 6900 60  0000 C CNN
+	1    5200 6900
+	1    0    0    -1
+$EndComp
+Wire Wire Line
+	5200 6400 5200 6700
+Wire Wire Line
+	5200 7100 5200 7300
+$Comp
+L GND #PWR24
+U 1 1 51CC4A77
+P 5200 7300
+F 0 "#PWR24" H 5200 7300 30  0001 C CNN
+F 1 "GND" H 5200 7230 30  0001 C CNN
+F 2 "" H 5200 7300 60  0000 C CNN
+F 3 "" H 5200 7300 60  0000 C CNN
+	1    5200 7300
+	1    0    0    -1
+$EndComp
+$Comp
+L +5V #PWR19
+U 1 1 51CC4AC8
+P 5200 5700
+F 0 "#PWR19" H 5200 5790 20  0001 C CNN
+F 1 "+5V" H 5200 5790 30  0000 C CNN
+F 2 "" H 5200 5700 60  0000 C CNN
+F 3 "" H 5200 5700 60  0000 C CNN
+	1    5200 5700
+	1    0    0    -1
+$EndComp
+Wire Wire Line
+	5200 6550 5700 6550
+Connection ~ 5200 6550
+Text Label 5350 6550 0    60   ~ 0
+AVCC
+Wire Wire Line
+	3800 3050 2600 3050
+Wire Wire Line
+	2600 3050 2600 3250
+$Comp
+L C C9
+U 1 1 51CC4FC9
+P 2600 3450
+F 0 "C9" H 2650 3550 50  0000 L CNN
+F 1 "0.01uF" H 2650 3350 50  0000 L CNN
+F 2 "SM0805" V 2450 3450 60  0000 C CNN
+F 3 "" H 2600 3450 60  0000 C CNN
+	1    2600 3450
+	1    0    0    -1
+$EndComp
+Wire Wire Line
+	2600 3650 2600 3800
+$Comp
+L GND #PWR11
+U 1 1 51CC50DF
+P 2600 3800
+F 0 "#PWR11" H 2600 3800 30  0001 C CNN
+F 1 "GND" H 2600 3730 30  0001 C CNN
+F 2 "" H 2600 3800 60  0000 C CNN
+F 3 "" H 2600 3800 60  0000 C CNN
+	1    2600 3800
+	1    0    0    -1
+$EndComp
 $EndSCHEMATC
