File: GVS-32U4/GVS-32U4-X1/GVS-32U4.sch (KiCad schematic (older format))
At the start: 48 parts, among them J1 USB-B, J10 GVS, J11 GVS, J12 GVS, J13 GVS, J14 GVS, J15 GVS, J16 GVS, J17 GVS, J18 GVS, J19 GVS, J2 GVS, J20 GVS, J21 GVS, J22 GVS, J23 GVS, J24 GVS, J25 GVS, J26 GVS, J27 GVS, J28 CONN_3, J29 CONN_2, J3 GVS, J30 CONN_2, J4 CONN_2, J5 GVS, J6 GVS, J7 GVS, J8 GVS, J9 GVS, U1 ATMEGA32U4-AU, U2 AP1117, X1 16MHz

Commit message: stuff
Connections:
- wire segments 183 -> 246
Changed lines of the file:
@@
-EESchema Schematic File Version 2  date 11/8/2012 10:05:01 AM
+EESchema Schematic File Version 2  date Tue 04 Dec 2012 07:22:51 PM EST
 LIBS:transistors
-LIBS:special
-LIBS:power
 LIBS:microcontrollers
 LIBS:device
-LIBS:contrib
 LIBS:conn
 LIBS:atmel
-LIBS:atmega32u4bb-from_eagle
-LIBS:DougsSch
+LIBS:GVS-32U4
 LIBS:GVS-32U4-cache
 EELAYER 25  0
@@
 Sheet 1 1
 Title "GVS-32U4"
-Date "8 nov 2012"
+Date "5 dec 2012"
 Rev "X1"
 Comp "AA6PR"
@@
 Comment4 ""
 $EndDescr
+$Comp
+L +3.3V #PWR014
+U 1 1 504A95D8
+P 3050 2800
+F 0 "#PWR014" H 3050 2760 30  0001 C CNN
+F 1 "+3.3V" H 3050 2910 30  0000 C CNN
+	1    3050 2800
+	1    0    0    -1
+$EndComp
+Wire Wire Line
+	3050 2800 3050 2850
+Connection ~ 3050 2850
 $Comp
 L CONN_2 J4
@@
 	3750 6450 3750 6400
 Wire Wire Line
-	3750 6450 1500 6450
+	3750 6450 2700 6450
+Wire Wire Line
+	2700 6450 1800 6450
+Wire Wire Line
+	1800 6450 1500 6450
 Wire Wire Line
 	1500 6050 1350 6050
 Wire Wire Line
-	1350 5850 2150 5850
+	1350 5850 1800 5850
+Wire Wire Line
+	1800 5850 2150 5850
 Connection ~ 3450 5800
 Wire Wire Line
@@
 	9600 4900 9800 4900
 Wire Wire Line
-	9700 5450 9700 4500
+	9700 5450 9700 5100
+Wire Wire Line
+	9700 5100 9700 4800
+Wire Wire Line
+	9700 4800 9700 4500
 Wire Wire Line
 	9700 4500 9800 4500
@@
 Connection ~ 700  7100
 Wire Wire Line
-	700  7050 700  7300
+	700  7050 700  7100
+Wire Wire Line
+	700  7100 700  7300
 Connection ~ 3200 1650
 Wire Wire Line
@@
 	2200 3050 2200 2850
 Wire Wire Line
-	3800 4550 3800 3850
+	3800 4550 3800 4350
+Wire Wire Line
+	3800 4350 3800 4250
+Wire Wire Line
+	3800 4250 3800 4150
+Wire Wire Line
+	3800 4150 3800 4050
+Wire Wire Line
+	3800 4050 3800 3850
 Wire Wire Line
 	3800 2150 3650 2150
 Connection ~ 3200 2050
 Wire Wire Line
-	3200 2250 3800 2250
+	3200 2250 3700 2250
+Wire Wire Line
+	3700 2250 3800 2250
 Wire Wire Line
 	3800 2050 3200 2050
@@
 Wire Wire Line
 	1750 1350 1750 1450
-Connection ~ 3050 2850
-Wire Wire Line
-	2750 2850 3800 2850
+Wire Wire Line
+	2750 2850 3050 2850
+Wire Wire Line
+	3050 2850 3800 2850
 Wire Wire Line
 	10150 5950 10150 5850
 Wire Wire Line
-	3050 2800 3050 2850
-Wire Wire Line
-	1750 3150 1750 2550
+	1750 3150 1750 2950
+Wire Wire Line
+	1750 2950 1750 2550
 Wire Wire Line
 	10150 6950 10150 7050
 Wire Wire Line
-	3200 1500 3200 2250
+	3200 1500 3200 1650
+Wire Wire Line
+	3200 1650 3200 1950
+Wire Wire Line
+	3200 1950 3200 2050
+Wire Wire Line
+	3200 2050 3200 2250
 Wire Wire Line
 	3500 850  3500 800
@@
 	1050 2950 1050 2850
 Wire Wire Line
-	1750 2950 1050 2950
+	1750 2950 1150 2950
+Wire Wire Line
+	1150 2950 1050 2950
 Connection ~ 1750 2950
 Wire Wire Line
@@
 	1100 7100 1100 7300
 Wire Wire Line
-	1100 7700 1100 7850
+	1100 7700 1100 7800
+Wire Wire Line
+	1100 7800 1100 7850
 Wire Wire Line
 	700  7700 700  7800
@@
 	9800 1450 9900 1450
 Wire Wire Line
-	9800 3900 9800 1450
+	9800 3900 9800 3550
+Wire Wire Line
+	9800 3550 9800 3250
+Wire Wire Line
+	9800 3250 9800 2950
+Wire Wire Line
+	9800 2950 9800 2650
+Wire Wire Line
+	9800 2650 9800 2350
+Wire Wire Line
+	9800 2350 9800 2050
+Wire Wire Line
+	9800 2050 9800 1750
+Wire Wire Line
+	9800 1750 9800 1450
 Wire Wire Line
 	9800 3250 9900 3250
@@
 	9700 3650 9900 3650
 Wire Wire Line
-	9700 1300 9700 3650
+	9700 1300 9700 1550
+Wire Wire Line
+	9700 1550 9700 1850
+Wire Wire Line
+	9700 1850 9700 2150
+Wire Wire Line
+	9700 2150 9700 2450
+Wire Wire Line
+	9700 2450 9700 2750
+Wire Wire Line
+	9700 2750 9700 3050
+Wire Wire Line
+	9700 3050 9700 3350
+Wire Wire Line
+	9700 3350 9700 3650
 Wire Wire Line
 	9700 1850 9900 1850
@@
 	8500 1850 8700 1850
 Wire Wire Line
-	8500 1300 8500 3650
+	8500 1300 8500 1550
+Wire Wire Line
+	8500 1550 8500 1850
+Wire Wire Line
+	8500 1850 8500 2150
+Wire Wire Line
+	8500 2150 8500 2450
+Wire Wire Line
+	8500 2450 8500 2750
+Wire Wire Line
+	8500 2750 8500 3050
+Wire Wire Line
+	8500 3050 8500 3350
+Wire Wire Line
+	8500 3350 8500 3650
 Wire Wire Line
 	8500 3650 8700 3650
@@
 	8600 3250 8700 3250
 Wire Wire Line
-	8600 3900 8600 1450
+	8600 3900 8600 3550
+Wire Wire Line
+	8600 3550 8600 3250
+Wire Wire Line
+	8600 3250 8600 2950
+Wire Wire Line
+	8600 2950 8600 2650
+Wire Wire Line
+	8600 2650 8600 2350
+Wire Wire Line
+	8600 2350 8600 2050
+Wire Wire Line
+	8600 2050 8600 1750
+Wire Wire Line
+	8600 1750 8600 1450
 Wire Wire Line
 	8600 1450 8700 1450
@@
 	7400 1450 7500 1450
 Wire Wire Line
-	7400 3900 7400 1450
+	7400 3900 7400 3550
+Wire Wire Line
+	7400 3550 7400 3250
+Wire Wire Line
+	7400 3250 7400 2950
+Wire Wire Line
+	7400 2950 7400 2650
+Wire Wire Line
+	7400 2650 7400 2350
+Wire Wire Line
+	7400 2350 7400 2050
+Wire Wire Line
+	7400 2050 7400 1750
+Wire Wire Line
+	7400 1750 7400 1450
 Wire Wire Line
 	7400 3250 7500 3250
@@
 	7300 3650 7500 3650
 Wire Wire Line
-	7300 1300 7300 3650
+	7300 1300 7300 1550
+Wire Wire Line
+	7300 1550 7300 1850
+Wire Wire Line
+	7300 1850 7300 2450
+Wire Wire Line
+	7300 2450 7300 2750
+Wire Wire Line
+	7300 2750 7300 3050
+Wire Wire Line
+	7300 3050 7300 3350
+Wire Wire Line
+	7300 3350 7300 3650
 Wire Wire Line
 	7300 1850 7500 1850
@@
 	700  7800 1100 7800
 Wire Wire Line
-	3450 5500 3450 5900
+	3450 5500 3450 5800
+Wire Wire Line
+	3450 5800 3450 5900
 Wire Wire Line
 	3450 5500 3300 5500
 Wire Wire Line
-	3300 5900 3750 5900
+	3300 5900 3450 5900
+Wire Wire Line
+	3450 5900 3750 5900
 Wire Wire Line
 	3750 5900 3750 6000
@@
 	3450 4850 2450 4850
 Wire Wire Line
-	1500 6600 1500 6050
+	1500 6600 1500 6450
+Wire Wire Line
+	1500 6450 1500 6050
 Connection ~ 1500 6450
 Wire Wire Line
-	9600 4400 9600 4900
+	9600 4400 9600 4600
+Wire Wire Line
+	9600 4600 9600 4900
 Text Label 9250 5300 0    60   ~ 0
 RST
@@
 	1    0    0    -1
 $EndComp
-$Comp
-L +3.3V #PWR014
-U 1 1 504A95D8
-P 3050 2800
-F 0 "#PWR014" H 3050 2760 30  0001 C CNN
-F 1 "+3.3V" H 3050 2910 30  0000 C CNN
-	1    3050 2800
-	1    0    0    -1
-$EndComp

Commit message: created gvs-32u4
Connections:
- net labels added: PF6, PF7
- net labels removed: PF2, PF3
- wire segments 246 -> 183
