File: OneWireLogger/OneWireLogger-X1/OneWireL-05.sch (KiCad schematic (older format))
At the start: 7 parts, among them SW2 SW5WAY

Commit message: One Wire Data Logger stuff
Parts:
- added TP6: TST, PIN_ARRAY_1, symbol TST
Connections:
- net SW5WAY: now also TP6.1
Changed lines of the file:
@@
-EESchema Schematic File Version 2  date 03/09/2013 12:08:25
+EESchema Schematic File Version 2  date 28/08/2013 13:19:36
 LIBS:power
 LIBS:device
@@
 Sheet 6 7
 Title ""
-Date "3 sep 2013"
+Date "10 jul 2013"
 Rev ""
 Comp ""
@@
 	3350 3300 3350 3400
 Connection ~ 3350 3400
+$Comp
+L TST TP6
+U 1 1 51DDBBDE
+P 5050 1850
+F 0 "TP6" H 5050 2150 40  0000 C CNN
+F 1 "TST" H 5050 2100 30  0000 C CNN
+F 2 "PIN_ARRAY_1" V 5150 2100 60  0000 C CNN
+F 3 "~" H 5050 1850 60  0000 C CNN
+	1    5050 1850
+	1    0    0    -1
+$EndComp
+Wire Wire Line
+	5050 1850 5050 1950
+Connection ~ 5050 1950
 $EndSCHEMATC
