File: PulseGenerator/PulseGenerator.sch (KiCad schematic (older format))
At the start: 25 parts, among them P1 CONN_2, P2 CONN_2, U1 74AC14

Commit message: PulseGen and others updates
Parts:
- C2: value 100uF -> 47uF
Changed lines of the file:
@@
-EESchema Schematic File Version 2  date 11/06/2013 08:30:01
+EESchema Schematic File Version 2
 LIBS:power
 LIBS:device
 LIBS:conn
 LIBS:74xx
-LIBS:DougsSch
 LIBS:PulseGenerator-cache
 EELAYER 27 0
@@
 Sheet 1 1
 Title ""
-Date "22 may 2013"
+Date "2 nov 2014"
 Rev ""
 Comp ""
@@
 P 1950 7500
 F 0 "C2" H 2000 7600 50  0000 L CNN
-F 1 "100uF" H 2000 7400 50  0000 L CNN
+F 1 "47uF" H 2000 7400 50  0000 L CNN
 F 2 "C1.5V8V" H 1950 7500 60  0000 C CNN
 F 3 "~" H 1950 7500 60  0000 C CNN

Commit message: glossing pwbs
Parts:
- PB1, PB2: Mfg (none) -> Amphenol; MfgPN (none) -> 31-5431-10RFX; Vendor (none) -> Mouser; VendorPN (none) -> 523-31-5431-10RFX
- U1: Mfg (none) -> TI; MfgPN (none) -> SN74AC14DR; Vendor (none) -> Mouser; VendorPN (none) -> 595-SN74AC14DR
Other:
- note added: "Not installed"
- moved on the sheet: C1, PA1, PA2, PB1, R1, R2, R3, R4, R5, R6, R7, R8
