File: CPLD-MAX5-100/CPLD-MAX5-100.sch (KiCad schematic (older format))
At the start: 19 parts

Commit message: worked on CPLD card
Parts:
- added U?: JTAG-10, Pin_Headers:Pin_Header_Straight_2x05, symbol JTAG-10
- C?: value C -> 10uF
- C? (x6): value C -> 0.1uF
- C? (x2): value C -> 47uF
- U?: footprint MODULE -> CPLD-MAX5-100:TQFP-100_14x14mm_Pitch0.5mm
- U?: value AP1117 -> AP1117-3.3V
- U?: value AP1117 -> AP1117-1.8V
Connections:
- net labels added: +5V
- wire segments 230 -> 299
Other:
- note added: "+5V\nGND"
Changed lines of the file:
@@
 LIBS:5M160ZT100
 LIBS:DougsSch
+LIBS:JTAG
 LIBS:CPLD-MAX5-100-cache
 EELAYER 25 0
@@
 U 1 1 5556375E
 P 8650 4950
-F 0 "U?" H 8650 4850 50  0000 C CNN
-F 1 "5M160ZT100" H 8650 5050 50  0000 C CNN
-F 2 "MODULE" H 8650 4950 50  0001 C CNN
+F 0 "U?" H 9350 7500 50  0000 C CNN
+F 1 "5M160ZT100" H 9350 2250 50  0000 C CNN
+F 2 "CPLD-MAX5-100:TQFP-100_14x14mm_Pitch0.5mm" H 7150 2200 50  0000 C CNN
 F 3 "DOCUMENTATION" H 8650 4950 50  0001 C CNN
 	1    8650 4950
@@
 P 3150 1850
 F 0 "U?" H 3250 1600 50  0000 C CNN
-F 1 "AP1117" H 3150 2100 50  0000 C CNN
+F 1 "AP1117-3.3V" H 3150 2100 50  0000 C CNN
 F 2 "SMD_Packages:SOT-223" H 3400 2200 60  0000 C CNN
 F 3 "" H 3150 1850 60  0000 C CNN
@@
 $EndComp
 Wire Wire Line
-	5050 1850 8300 1850
+	5050 1850 5300 1850
+Wire Wire Line
+	5300 1850 5550 1850
+Wire Wire Line
+	5550 1850 5800 1850
+Wire Wire Line
+	5800 1850 6400 1850
+Wire Wire Line
+	6400 1850 8200 1850
+Wire Wire Line
+	8200 1850 8300 1850
 Wire Wire Line
 	8200 1850 8200 2150
@@
 Connection ~ 8200 1850
 Wire Wire Line
-	3450 1850 4450 1850
+	3450 1850 3600 1850
+Wire Wire Line
+	3600 1850 3850 1850
+Wire Wire Line
+	3850 1850 4100 1850
+Wire Wire Line
+	4100 1850 4350 1850
+Wire Wire Line
+	4350 1850 4450 1850
 Wire Wire Line
 	4350 1850 4350 1350
 Wire Wire Line
-	4350 1350 12500 1350
+	4350 1350 8500 1350
+Wire Wire Line
+	8500 1350 8600 1350
+Wire Wire Line
+	8600 1350 8700 1350
+Wire Wire Line
+	8700 1350 8850 1350
+Wire Wire Line
+	8850 1350 8950 1350
+Wire Wire Line
+	8950 1350 9050 1350
+Wire Wire Line
+	9050 1350 12500 1350
 Wire Wire Line
 	8500 1350 8500 2150
@@
 Connection ~ 8950 1350
 Wire Wire Line
-	1600 1850 2850 1850
-Wire Wire Line
-	1600 2300 5800 2300
+	1600 1850 2000 1850
+Wire Wire Line
+	2000 1850 2250 1850
+Wire Wire Line
+	2250 1850 2500 1850
+Wire Wire Line
+	2500 1850 2700 1850
+Wire Wire Line
+	2700 1850 2850 1850
+Wire Wire Line
+	1600 2300 2000 2300
+Wire Wire Line
+	2000 2300 2250 2300
+Wire Wire Line
+	2250 2300 2500 2300
+Wire Wire Line
+	2500 2300 3150 2300
+Wire Wire Line
+	3150 2300 3600 2300
+Wire Wire Line
+	3600 2300 3850 2300
+Wire Wire Line
+	3850 2300 4100 2300
+Wire Wire Line
+	4100 2300 4750 2300
+Wire Wire Line
+	4750 2300 5300 2300
+Wire Wire Line
+	5300 2300 5550 2300
+Wire Wire Line
+	5550 2300 5800 2300
 $Comp
 L GND #PWR?
@@
 	8250 7900 8250 8050
 Wire Wire Line
-	8250 8050 9050 8050
-Wire Wire Line
-	9050 7900 9050 8200
+	8250 8050 8350 8050
+Wire Wire Line
+	8350 8050 8450 8050
+Wire Wire Line
+	8450 8050 8550 8050
+Wire Wire Line
+	8550 8050 8650 8050
+Wire Wire Line
+	8650 8050 8750 8050
+Wire Wire Line
+	8750 8050 8850 8050
+Wire Wire Line
+	8850 8050 8950 8050
+Wire Wire Line
+	8950 8050 9050 8050
+Wire Wire Line
+	9050 7900 9050 8050
+Wire Wire Line
+	9050 8050 9050 8200
 Wire Wire Line
 	8950 7900 8950 8050
@@
 P 2000 2050
 F 0 "C?" H 2025 2150 50  0000 L CNN
-F 1 "C" H 2025 1950 50  0000 L CNN
+F 1 "10uF" H 2025 1950 50  0000 L CNN
 F 2 "Capacitors_SMD:C_0805" H 2038 1900 30  0000 C CNN
 F 3 "" H 2000 2050 60  0000 C CNN
@@
 	3150 2150 3150 2300
 Wire Wire Line
-	1600 2150 1600 2400
+	1600 2150 1600 2300
+Wire Wire Line
+	1600 2300 1600 2400
 Wire Wire Line
 	2000 1900 2000 1850
@@
 P 1150 2100
 F 0 "P?" H 1150 2250 50  0000 C CNN
-F 1 "CONN_01X02" V 1250 2100 50  0000 C CNN
+F 1 "CONN_01X02" H 1150 1950 50  0000 C CNN
 F 2 "" H 1150 2100 60  0000 C CNN
 F 3 "" H 1150 2100 60  0000 C CNN
@@
 	10700 7000 10700 8500
 Wire Wire Line
-	10700 8500 12700 8500
-Wire Wire Line
-	12600 4000 12600 8500
+	10700 8500 12600 8500
+Wire Wire Line
+	12600 8500 12700 8500
+Wire Wire Line
+	12600 4000 12600 5500
+Wire Wire Line
+	12600 5500 12600 7000
+Wire Wire Line
+	12600 7000 12600 8500
 Wire Wire Line
 	12600 7000 12700 7000
@@
 	12500 7400 12700 7400
 Wire Wire Line
-	12500 1350 12500 7400
+	12500 1350 12500 2900
+Wire Wire Line
+	12500 2900 12500 4400
+Wire Wire Line
+	12500 4400 12500 5900
+Wire Wire Line
+	12500 5900 12500 7400
 Wire Wire Line
 	12500 5900 12700 5900
@@
 	14300 7400 14200 7400
 Wire Wire Line
-	14300 1050 14300 7400
+	14300 1050 14300 2900
+Wire Wire Line
+	14300 2900 14300 4400
+Wire Wire Line
+	14300 4400 14300 5900
+Wire Wire Line
+	14300 5900 14300 7400
 Wire Wire Line
 	14300 1050 2700 1050
@@
 	15700 3950 15700 3850
 Wire Wire Line
-	14500 3850 16050 3850
+	14500 3850 15700 3850
+Wire Wire Line
+	15700 3850 15800 3850
+Wire Wire Line
+	15800 3850 16050 3850
 Wire Wire Line
 	15800 3850 15800 3950
@@
 	15700 4450 15700 4550
 Wire Wire Line
-	15700 4550 16050 4550
+	15700 4550 15800 4550
+Wire Wire Line
+	15800 4550 16050 4550
 Wire Wire Line
 	15800 4550 15800 4450
 Wire Wire Line
-	16050 3850 16050 8550
+	16050 3850 16050 4550
+Wire Wire Line
+	16050 4550 16050 5500
+Wire Wire Line
+	16050 5500 16050 6850
+Wire Wire Line
+	16050 6850 16050 7550
+Wire Wire Line
+	16050 7550 16050 8500
+Wire Wire Line
+	16050 8500 16050 8550
 Connection ~ 15800 4550
 Connection ~ 15800 3850
@@
 	15700 6950 15700 6850
 Wire Wire Line
-	14600 6850 16050 6850
-Wire Wire Line
-	16050 7550 15700 7550
+	14600 6850 15700 6850
+Wire Wire Line
+	15700 6850 15800 6850
+Wire Wire Line
+	15800 6850 16050 6850
+Wire Wire Line
+	15700 7550 15800 7550
+Wire Wire Line
+	15800 7550 16050 7550
 Wire Wire Line
 	15700 7550 15700 7450
@@
 P 2250 2050
 F 0 "C?" H 2275 2150 50  0000 L CNN
-F 1 "C" H 2275 1950 50  0000 L CNN
+F 1 "0.1uF" H 2275 1950 50  0000 L CNN
 F 2 "Capacitors_SMD:C_0805" H 2288 1900 30  0000 C CNN
 F 3 "" H 2250 2050 60  0000 C CNN
@@
 P 2500 2050
 F 0 "C?" H 2525 2150 50  0000 L CNN
-F 1 "C" H 2525 1950 50  0000 L CNN
+F 1 "0.1uF" H 2525 1950 50  0000 L CNN
 F 2 "Capacitors_SMD:C_0805" H 2538 1900 30  0000 C CNN
 F 3 "" H 2500 2050 60  0000 C CNN
@@
 P 3600 2050
 F 0 "C?" H 3625 2150 50  0000 L CNN
-F 1 "C" H 3625 1950 50  0000 L CNN
+F 1 "47uF" H 3625 1950 50  0000 L CNN
 F 2 "Capacitors_SMD:C_0805" H 3638 1900 30  0000 C CNN
 F 3 "" H 3600 2050 60  0000 C CNN
@@
 P 3850 2050
 F 0 "C?" H 3875 2150 50  0000 L CNN
-F 1 "C" H 3875 1950 50  0000 L CNN
+F 1 "0.1uF" H 3875 1950 50  0000 L CNN
 F 2 "Capacitors_SMD:C_0805" H 3888 1900 30  0000 C CNN
 F 3 "" H 3850 2050 60  0000 C CNN
@@
 P 4100 2050
 F 0 "C?" H 4125 2150 50  0000 L CNN
-F 1 "C" H 4125 1950 50  0000 L CNN
+F 1 "0.1uF" H 4125 1950 50  0000 L CNN
 F 2 "Capacitors_SMD:C_0805" H 4138 1900 30  0000 C CNN
 F 3 "" H 4100 2050 60  0000 C CNN
@@
 P 5300 2050
 F 0 "C?" H 5325 2150 50  0000 L CNN
-F 1 "C" H 5325 1950 50  0000 L CNN
+F 1 "47uF" H 5325 1950 50  0000 L CNN
 F 2 "Capacitors_SMD:C_0805" H 5338 1900 30  0000 C CNN
 F 3 "" H 5300 2050 60  0000 C CNN
@@
 P 5550 2050
 F 0 "C?" H 5575 2150 50  0000 L CNN
-F 1 "C" H 5575 1950 50  0000 L CNN
+F 1 "0.1uF" H 5575 1950 50  0000 L CNN
 F 2 "Capacitors_SMD:C_0805" H 5588 1900 30  0000 C CNN
 F 3 "" H 5550 2050 60  0000 C CNN
@@
 P 5800 2050
 F 0 "C?" H 5825 2150 50  0000 L CNN
-F 1 "C" H 5825 1950 50  0000 L CNN
+F 1 "0.1uF" H 5825 1950 50  0000 L CNN
 F 2 "Capacitors_SMD:C_0805" H 5838 1900 30  0000 C CNN
 F 3 "" H 5800 2050 60  0000 C CNN
@@
 P 4750 1850
 F 0 "U?" H 4850 1600 50  0000 C CNN
-F 1 "AP1117" H 4750 2100 50  0000 C CNN
+F 1 "AP1117-1.8V" H 4750 2100 50  0000 C CNN
 F 2 "SMD_Packages:SOT-223" H 5000 2200 60  0000 C CNN
 F 3 "" H 4750 1850 60  0000 C CNN
@@
 	1    0    0    -1
 $EndComp
+$Comp
+L JTAG-10 U?
+U 1 1 555A1751
+P 4500 3550
+F 0 "U?" H 4700 4150 50  0000 C CNN
+F 1 "JTAG-10" H 4800 2950 50  0000 C CNN
+F 2 "Pin_Headers:Pin_Header_Straight_2x05" V 3950 3550 50  0000 C CNN
+F 3 "DOCUMENTATION" H 4500 3550 50  0001 C CNN
+	1    4500 3550
+	1    0    0    -1
+$EndComp
+Wire Wire Line
+	5300 3200 7450 3200
+Wire Wire Line
+	7450 3300 5300 3300
+Wire Wire Line
+	5300 3400 7450 3400
+Wire Wire Line
+	7450 3500 5300 3500
+Wire Wire Line
+	4500 2700 4500 2500
+Wire Wire Line
+	4500 2500 6400 2500
+Wire Wire Line
+	6400 2500 6400 1850
+Connection ~ 6400 1850
+Text Label 1700 1850 0    60   ~ 0
++5V
+Text Label 1700 2300 0    60   ~ 0
+GND
+Wire Wire Line
+	4550 4400 4550 4500
+Wire Wire Line
+	4550 4500 4550 4600
+$Comp
+L GND #PWR?
+U 1 1 555A4021
+P 4550 4600
+F 0 "#PWR?" H 4550 4350 50  0001 C CNN
+F 1 "GND" H 4550 4450 50  0000 C CNN
+F 2 "" H 4550 4600 60  0000 C CNN
+F 3 "" H 4550 4600 60  0000 C CNN
+	1    4550 4600
+	1    0    0    -1
+$EndComp
+Wire Wire Line
+	4450 4400 4450 4500
+Wire Wire Line
+	4450 4500 4550 4500
+Connection ~ 4550 4500
+Text Notes 1050 2200 2    60   ~ 0
++5V\nGND
 $EndSCHEMATC

Commit message: Add QFP library and CPLD card layout
Parts:
- removed P? (x2): CONN_02X10, symbol CONN_02X10
- added MTG1, MTG2, MTG3, MTG4: CONN_01X01, dougsLib:MTG-6-32, symbol CONN_01X01
- added P2, P3, P4, P5, P? (x4): CONN_01X10, Pin_Headers:Pin_Header_Straight_2x05, symbol CONN_01X10
- P1: renamed from P?; footprint (none) -> dougsLib:TB2-5MM
- U4: renamed from U?; footprint CPLD-MAX5-100:TQFP-100_14x14mm_Pitch0.5mm -> Housings_QFP:TQFP-100_14x14mm_Pitch0.5mm
- U5, U6, U7, U8: renamed from U?; footprint MODULE -> Housings_SOIC:SOIC-20_7.5x12.8mm_Pitch1.27mm
- gave numbers to parts that had none: 12
Connections:
- wire segments 299 -> 208
- no-connect marks 0 -> 7

Commit message: CPLD layout
Parts:
- added C10, C11, C12, C13, C14, C15, C16, C17, C18, C19, C20, C21, C22, C23, C24, C25: 0.1uF, Capacitors_SMD:C_0805, symbol C
- added J2, J3: CONN_01X03, Pin_Headers:Pin_Header_Straight_1x03, symbol CONN_01X03
- added TP1, TP2, TP3: CONN_01X02, Pin_Headers:Pin_Header_Straight_1x02, symbol CONN_01X02
- added U10, U11, U12, U9: TXS0108, dougsLib:SOG20, symbol TXS0108
- C1, C4, C7: footprint Capacitors_SMD:C_0805 -> Capacitors_SMD:C_1206
- U5, U6, U7, U8: footprint Housings_SOIC:SOIC-20_7.5x12.8mm_Pitch1.27mm -> dougsLib:SOG20
- gave numbers to parts that had none: 4
- renumbered U2 to J1
Connections:
- net labels added: +1V8, +3.3V, TCK, TDI, TDO, TMS, VRINGA, VRINGB
- wire segments 208 -> 421
Other:
- note added: "5V\n\n3.3V"
- moved on the sheet: C1, C2, C3, C4, C5, C6, C7, C8, C9, J1, MTG1, MTG2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
