File: XR-2206/KiCAD/XR2206.sch (KiCad schematic (older format))
At the start: 16 parts, among them J1 CONN_2, J2 CONN_2, J3 CONN_2, U1 XR2206

Commit message: MyMenu updates
Connections:
- wire segments 42 -> 52
Other:
- moved on the sheet: C1, C3, R3, R6, R7
Changed lines of the file:
@@
-EESchema Schematic File Version 2  date 06/03/2013 12:50:37
+EESchema Schematic File Version 2
 LIBS:power
 LIBS:device
@@
 LIBS:contrib
 LIBS:XR2206-cache
-EELAYER 27 0
+EELAYER 25 0
 EELAYER END
 $Descr A 11000 8500
@@
 Comment4 ""
 $EndDescr
-Text Notes 2850 3700 2    60   ~ 0
+Text Notes 2800 3900 2    60   ~ 0
 G\n\nADJ
 NoConn ~ 6950 5750
@@
 $EndComp
 Wire Wire Line
-	3850 2950 7700 2950
+	3850 2950 5300 2950
+Wire Wire Line
+	5300 2950 7450 2950
+Wire Wire Line
+	7450 2950 7700 2950
 Wire Wire Line
 	7650 3850 6800 3850
@@
 Connection ~ 6650 3950
 Wire Wire Line
-	6550 3950 6900 3950
+	6450 3950 6650 3950
+Wire Wire Line
+	6650 3950 6900 3950
 Connection ~ 3850 3650
 Wire Wire Line
@@
 	4550 3550 4750 3550
 Wire Wire Line
-	4450 3850 4750 3850
+	4350 3850 4750 3850
 Wire Wire Line
 	4750 3650 4200 3650
 Wire Wire Line
-	4200 3650 4200 3600
+	4200 3650 4200 3500
 Wire Wire Line
 	5850 4350 6000 4350
@@
 Connection ~ 5300 2950
 Wire Wire Line
-	3850 5250 3850 3550
-Wire Wire Line
-	4750 4350 3950 4350
-Wire Wire Line
-	3950 4350 3950 4250
-Wire Wire Line
-	3950 4250 4000 4250
-Wire Wire Line
-	7550 5200 3850 5200
+	3850 5250 3850 5200
+Wire Wire Line
+	3850 5200 3850 4750
+Wire Wire Line
+	3850 4750 3850 4150
+Wire Wire Line
+	3850 4150 3850 3650
+Wire Wire Line
+	3850 3650 3850 3450
+Wire Wire Line
+	4750 4350 4150 4350
+Wire Wire Line
+	4150 4350 4150 4250
+Wire Wire Line
+	4150 4250 4200 4250
+Wire Wire Line
+	7550 5200 6000 5200
+Wire Wire Line
+	6000 5200 5300 5200
+Wire Wire Line
+	5300 5200 3850 5200
 Connection ~ 6000 5200
 Wire Wire Line
 	7550 3150 7700 3150
 Wire Wire Line
-	3950 3850 3350 3850
+	4050 3850 3350 3850
 Wire Wire Line
 	6900 4250 6650 4250
@@
 	6650 4250 6650 3950
 Wire Wire Line
-	5950 3950 6050 3950
-Wire Wire Line
-	7400 4250 7550 4250
+	5950 3950 6150 3950
+Wire Wire Line
+	7200 4250 7550 4250
 Connection ~ 7550 4250
 Wire Wire Line
@@
 Connection ~ 3850 4750
 Wire Wire Line
-	7550 3150 7550 5200
+	7550 3150 7550 4250
+Wire Wire Line
+	7550 4250 7550 5200
 Wire Wire Line
 	7550 4050 7650 4050
@@
 L CP1 C3
 U 1 1 511BA085
-P 3850 3350
-F 0 "C3" H 3900 3450 50  0000 L CNN
-F 1 "4.7uF" H 3900 3250 50  0000 L CNN
-F 2 "" H 3850 3350 60  0001 C CNN
-F 3 "" H 3850 3350 60  0001 C CNN
-	1    3850 3350
+P 3850 3300
+F 0 "C3" H 3900 3400 50  0000 L CNN
+F 1 "4.7uF" H 3900 3200 50  0000 L CNN
+F 2 "" H 3850 3300 60  0001 C CNN
+F 3 "" H 3850 3300 60  0001 C CNN
+	1    3850 3300
 	1    0    0    -1
 $EndComp
@@
 L R R7
 U 1 1 501123C8
-P 7150 4250
-F 0 "R7" V 7250 4250 50  0000 C CNN
-F 1 "5.1K" V 7150 4250 50  0000 C CNN
-F 2 "" H 7150 4250 60  0001 C CNN
-F 3 "" H 7150 4250 60  0001 C CNN
-	1    7150 4250
+P 7050 4250
+F 0 "R7" V 7150 4250 50  0000 C CNN
+F 1 "5.1K" V 7050 4250 50  0000 C CNN
+F 2 "" H 7050 4250 60  0001 C CNN
+F 3 "" H 7050 4250 60  0001 C CNN
+	1    7050 4250
 	0    1    1    0
 $EndComp
@@
 L R R6
 U 1 1 501123BB
-P 7150 3950
-F 0 "R6" V 7250 3950 50  0000 C CNN
-F 1 "5.1K" V 7150 3950 50  0000 C CNN
-F 2 "" H 7150 3950 60  0001 C CNN
-F 3 "" H 7150 3950 60  0001 C CNN
-	1    7150 3950
+P 7050 3950
+F 0 "R6" V 7150 3950 50  0000 C CNN
+F 1 "5.1K" V 7050 3950 50  0000 C CNN
+F 2 "" H 7050 3950 60  0001 C CNN
+F 3 "" H 7050 3950 60  0001 C CNN
+	1    7050 3950
 	0    1    1    0
 $EndComp
@@
 L R R3
 U 1 1 4FDBE56E
-P 4250 4250
-F 0 "R3" V 4330 4250 50  0000 C CNN
-F 1 "220" V 4250 4250 50  0000 C CNN
-F 2 "" H 4250 4250 60  0001 C CNN
-F 3 "" H 4250 4250 60  0001 C CNN
-	1    4250 4250
+P 4350 4250
+F 0 "R3" V 4430 4250 50  0000 C CNN
+F 1 "220" V 4350 4250 50  0000 C CNN
+F 2 "" H 4350 4250 60  0001 C CNN
+F 3 "" H 4350 4250 60  0001 C CNN
+	1    4350 4250
 	0    1    1    0
 $EndComp
@@
 L C C1
 U 1 1 4FDBC755
-P 4200 3400
-F 0 "C1" H 4250 3500 50  0000 L CNN
-F 1 "0.1uF" H 4250 3300 50  0000 L CNN
-F 2 "" H 4200 3400 60  0001 C CNN
-F 3 "" H 4200 3400 60  0001 C CNN
-	1    4200 3400
+P 4200 3350
+F 0 "C1" H 4250 3450 50  0000 L CNN
+F 1 "0.1uF" H 4250 3250 50  0000 L CNN
+F 2 "" H 4200 3350 60  0001 C CNN
+F 3 "" H 4200 3350 60  0001 C CNN
+	1    4200 3350
 	1    0    0    -1
 $EndComp
@@
 $EndComp
 Wire Wire Line
-	7450 3950 7400 3950
+	7450 3950 7200 3950
 Connection ~ 7450 2950
+Connection ~ 7550 4050
+Connection ~ 3400 3450
+Connection ~ 6300 3700
 $EndSCHEMATC
