File: RPI-I2C-HUB/RPI-I2C-HUB.kicad_pcb (KiCad board)
At the start: 2 copper layers, 49 x 49 mm, 32 parts, among them J1 I2CINT-5PIN, J2 I2CINT-5PIN, J3 I2CINT-5PIN, J4 I2CINT-5PIN, P1 RASPIO, U1 PCA9544A

Commit message: new console card
Other:
- outline, holes or cut-outs redrawn
- board text added: "INT SCL GND"
- board text added: "INT SCL SDA"
- board text added: "INT SCL SDA +V GND"
- board text added: "P2= 3.3V"
- board text added: "PWB REV X3"
- board text removed: "INT SCK GND"
- board text removed: "INT SCK SDA"
- board text removed: "INT SCK SDA +V GND"
- board text removed: "P2=3.3V"
- board text removed: "PWB REV X2"
Changed lines of the file:
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@@
     (links 79)
     (no_connects 0)
-    (area -10.999999 -7.85 61 51.246)
+    (area -10.999999 -8.85 61 51.246)
     (thickness 1.6)
-    (drawings 26)
+    (drawings 28)
     (tracks 220)
     (zones 0)
@@
     (0 F.Cu signal)
     (31 B.Cu signal)
-    (36 B.SilkS user hide)
+    (36 B.SilkS user)
     (37 F.SilkS user)
     (38 B.Mask user)
@@
     (fp_line (start -2 1.5) (end 2 1.5) (layer B.SilkS) (width 0.65))
   )
-  (gr_text "INT\nSCK\n\n\nGND" (at 34.29 41.91 180) (layer F.SilkS)
+  (gr_line (start 36 13) (end 49 13) (angle 90) (layer Edge.Cuts) (width 0.1))
+  (gr_line (start 34 11) (end 34 0) (angle 90) (layer Edge.Cuts) (width 0.1))
+  (gr_arc (start 36 11) (end 36 13) (angle 90) (layer Edge.Cuts) (width 0.1))
+  (dimension 13 (width 0.3) (layer Eco1.User)
+    (gr_text "13.000 mm" (at 54.35 6.5 270) (layer Eco1.User)
+      (effects (font (size 1.5 1.5) (thickness 0.3)))
+    )
+    (feature1 (pts (xy 34 13) (xy 55.7 13)))
+    (feature2 (pts (xy 34 0) (xy 55.7 0)))
+    (crossbar (pts (xy 53 0) (xy 53 13)))
+    (arrow1a (pts (xy 53 13) (xy 52.413579 11.873496)))
+    (arrow1b (pts (xy 53 13) (xy 53.586421 11.873496)))
+    (arrow2a (pts (xy 53 0) (xy 52.413579 1.126504)))
+    (arrow2b (pts (xy 53 0) (xy 53.586421 1.126504)))
+  )
+  (dimension 19 (width 0.3) (layer Eco1.User)
+    (gr_text "19.000 mm" (at 43.5 -3.35) (layer Eco1.User)
+      (effects (font (size 1.5 1.5) (thickness 0.3)))
+    )
+    (feature1 (pts (xy 53 0) (xy 53 -4.7)))
+    (feature2 (pts (xy 34 0) (xy 34 -4.7)))
+    (crossbar (pts (xy 34 -2) (xy 53 -2)))
+    (arrow1a (pts (xy 53 -2) (xy 51.873496 -1.413579)))
+    (arrow1b (pts (xy 53 -2) (xy 51.873496 -2.586421)))
+    (arrow2a (pts (xy 34 -2) (xy 35.126504 -1.413579)))
+    (arrow2b (pts (xy 34 -2) (xy 35.126504 -2.586421)))
+  )
+  (dimension 34 (width 0.3) (layer Eco1.User)
+    (gr_text "34.000 mm" (at 17 -3.35) (layer Eco1.User)
+      (effects (font (size 1.5 1.5) (thickness 0.3)))
+    )
+    (feature1 (pts (xy 34 0) (xy 34 -4.7)))
+    (feature2 (pts (xy 0 0) (xy 0 -4.7)))
+    (crossbar (pts (xy 0 -2) (xy 34 -2)))
+    (arrow1a (pts (xy 34 -2) (xy 32.873496 -1.413579)))
+    (arrow1b (pts (xy 34 -2) (xy 32.873496 -2.586421)))
+    (arrow2a (pts (xy 0 -2) (xy 1.126504 -1.413579)))
+    (arrow2b (pts (xy 0 -2) (xy 1.126504 -2.586421)))
+  )
+  (dimension 53 (width 0.3) (layer Eco1.User)
+    (gr_text "53.000 mm" (at 26.5 -7.35) (layer Eco1.User)
+      (effects (font (size 1.5 1.5) (thickness 0.3)))
+    )
+    (feature1 (pts (xy 53 0) (xy 53 -8.7)))
+    (feature2 (pts (xy 0 0) (xy 0 -8.7)))
+    (crossbar (pts (xy 0 -6) (xy 53 -6)))
+    (arrow1a (pts (xy 53 -6) (xy 51.873496 -5.413579)))
+    (arrow1b (pts (xy 53 -6) (xy 51.873496 -6.586421)))
+    (arrow2a (pts (xy 0 -6) (xy 1.126504 -5.413579)))
+    (arrow2b (pts (xy 0 -6) (xy 1.126504 -6.586421)))
+  )
+  (gr_line (start 34 0) (end 0 0) (angle 90) (layer Edge.Cuts) (width 0.1))
+  (gr_text "INT\nSCL\n\n\nGND" (at 34.29 41.91 180) (layer F.SilkS)
     (effects (font (size 1.5875 1.5875) (thickness 0.3)) (justify left))
   )
-  (gr_text "INT\nSCK\nSDA" (at 15.24 34.29) (layer F.SilkS)
+  (gr_text "INT\nSCL\nSDA" (at 15.24 34.29) (layer F.SilkS)
     (effects (font (size 1.5875 1.5875) (thickness 0.3)) (justify left))
   )
-  (gr_text "INT\nSCK\nSDA\n+V\nGND" (at 34.29 20.066 180) (layer F.SilkS)
+  (gr_text "INT\nSCL\nSDA\n+V\nGND" (at 34.29 20.066 180) (layer F.SilkS)
     (effects (font (size 1.5875 1.5875) (thickness 0.3)) (justify left))
   )
-  (gr_text "INT\nSCK\nSDA\n+V\nGND" (at 15.494 16.51) (layer F.SilkS)
+  (gr_text "INT\nSCL\nSDA\n+V\nGND" (at 15.494 16.51) (layer F.SilkS)
     (effects (font (size 1.5875 1.5875) (thickness 0.3)) (justify left))
   )
@@
     (arrow2b (pts (xy 53 13) (xy 53.586421 14.126504)))
   )
-  (dimension 10 (width 0.3) (layer Eco1.User)
-    (gr_text "10.000 mm" (at 44 -6.35) (layer Eco1.User)
-      (effects (font (size 1.5 1.5) (thickness 0.3)))
-    )
-    (feature1 (pts (xy 49 13) (xy 49 -7.7)))
-    (feature2 (pts (xy 39 13) (xy 39 -7.7)))
-    (crossbar (pts (xy 39 -5) (xy 49 -5)))
-    (arrow1a (pts (xy 49 -5) (xy 47.873496 -4.413579)))
-    (arrow1b (pts (xy 49 -5) (xy 47.873496 -5.586421)))
-    (arrow2a (pts (xy 39 -5) (xy 40.126504 -4.413579)))
-    (arrow2b (pts (xy 39 -5) (xy 40.126504 -5.586421)))
-  )
-  (dimension 13 (width 0.3) (layer Eco1.User)
-    (gr_text "13.000 mm" (at 54.35 6.5 270) (layer Eco1.User)
-      (effects (font (size 1.5 1.5) (thickness 0.3)))
-    )
-    (feature1 (pts (xy 39 13) (xy 55.7 13)))
-    (feature2 (pts (xy 39 0) (xy 55.7 0)))
-    (crossbar (pts (xy 53 0) (xy 53 13)))
-    (arrow1a (pts (xy 53 13) (xy 52.413579 11.873496)))
-    (arrow1b (pts (xy 53 13) (xy 53.586421 11.873496)))
-    (arrow2a (pts (xy 53 0) (xy 52.413579 1.126504)))
-    (arrow2b (pts (xy 53 0) (xy 53.586421 1.126504)))
-  )
-  (dimension 39 (width 0.3) (layer Eco1.User)
-    (gr_text "39.000 mm" (at 19.5 -4.35) (layer Eco1.User)
-      (effects (font (size 1.5 1.5) (thickness 0.3)))
-    )
-    (feature1 (pts (xy 39 0) (xy 39 -5.7)))
-    (feature2 (pts (xy 0 0) (xy 0 -5.7)))
-    (crossbar (pts (xy 0 -3) (xy 39 -3)))
-    (arrow1a (pts (xy 39 -3) (xy 37.873496 -2.413579)))
-    (arrow1b (pts (xy 39 -3) (xy 37.873496 -3.586421)))
-    (arrow2a (pts (xy 0 -3) (xy 1.126504 -2.413579)))
-    (arrow2b (pts (xy 0 -3) (xy 1.126504 -3.586421)))
-  )
-  (gr_text P2=3.3V (at 33.655 6.731) (layer F.SilkS)
+  (gr_text "P2=\n3.3V" (at 23.368 12.446) (layer F.SilkS)
     (effects (font (size 1.5 1.5) (thickness 0.3)))
   )
@@
   )
   (gr_line (start 0 49) (end 49 49) (angle 90) (layer Edge.Cuts) (width 0.1))
-  (gr_line (start 0 0) (end 39 0) (angle 90) (layer Edge.Cuts) (width 0.1))
   (gr_line (start 49 13) (end 49 49) (angle 90) (layer Edge.Cuts) (width 0.1))
-  (gr_line (start 39 13) (end 49 13) (angle 90) (layer Edge.Cuts) (width 0.1))
-  (gr_line (start 39 0) (end 39 13) (angle 90) (layer Edge.Cuts) (width 0.1))
   (dimension 49 (width 0.3) (layer Eco1.User)
     (gr_text "49.000 mm" (at -4.35 24.5 270) (layer Eco1.User)
@@
     (effects (font (size 1.5 1.5) (thickness 0.3)))
   )
-  (gr_text "PWB REV X2" (at 8.255 8.001) (layer F.SilkS)
+  (gr_text "PWB REV X3" (at 8.255 8.001) (layer F.SilkS)
     (effects (font (size 1.27 1.27) (thickness 0.3175)))
   )
@@
   (segment (start 35.56 39.37) (end 33.04 39.37) (width 0.254) (layer B.Cu) (net 21))
   (segment (start 33.04 39.37) (end 33.02 39.35) (width 0.254) (layer B.Cu) (net 21))
+  (zone (net 3) (net_name GND) (layer B.Cu) (hatch edge 0.508)
+    (connect_pads (clearance 0.3048))
+    (min_thickness 0.254)
+    (fill yes (arc_segments 16) (thermal_gap 0.508) (thermal_bridge_width 0.508))
+    (polygon
+      (pts
+        (xy 0 0) (xy 34 0) (xy 34 13) (xy 49 13) (xy 49 49)
+        (xy 0 49)
+      )
+    )
+  )
   (zone (net 16) (net_name +3.3V) (layer F.Cu) (hatch edge 0.508)
     (connect_pads (clearance 0.3048))
@@
     (polygon
       (pts
-        (xy 0 0) (xy 39.37 0) (xy 39.37 12.7) (xy 48.26 12.7) (xy 48.26 49.53)
-        (xy 0 49.53) (xy 0 3.81)
+        (xy 0 0) (xy 34.036 0) (xy 34 13) (xy 49 13) (xy 49 49)
+        (xy 0 49) (xy 0 3.81)
       )
     )
-  )
-  (zone (net 3) (net_name GND) (layer B.Cu) (hatch edge 0.508)
-    (connect_pads (clearance 0.3048))
-    (min_thickness 0.254)
-    (fill yes (arc_segments 16) (thermal_gap 0.508) (thermal_bridge_width 0.508))
-    (polygon
-      (pts
-        (xy 0 0) (xy 39 0) (xy 39 13) (xy 49 13) (xy 49 49)
-        (xy 0 49)
-      )
-    )
