File: I2C-RPT-01/RevX2/I2C-RPT-01.kicad_pcb (KiCad board)
At the start: 2 copper layers, 49 x 49 mm, 35 parts, among them J1 I2CINT-5PIN, J2 I2CINT-5PIN, J3 I2CINT-5PIN, J4 I2CINT-5PIN, J5 I2CINT-5PIN, U1 PCA9544A

Commit message: Tweeks to the silkscreen
Other:
- board text added: "INT CK D"
- board text added: "INT SCK SDA"
- board text added: "PWB REV X2"
- board text added: "SD SC INT"
- board text added: "SDA SCK INT"
- board text removed: "INT CL D"
- board text removed: "INT SCL SDA"
- board text removed: "PWB REV X3"
- board text removed: "SD CL INT"
- board text removed: "SDA SCL INT"
Changed lines of the file:
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@@
     (effects (font (size 2.032 1.524) (thickness 0.3048)))
   )
-  (gr_text "SD\nCL\nINT" (at 198.628 99.06) (layer F.SilkS)
+  (gr_text "SD\nSC\nINT" (at 198.628 99.06) (layer F.SilkS)
+    (effects (font (size 1.651 1.524) (thickness 0.3048)) (justify right))
+  )
+  (gr_text "SDA\nSCK\nINT" (at 198.628 114.3) (layer F.SilkS)
     (effects (font (size 1.651 1.27) (thickness 0.3048)) (justify right))
   )
-  (gr_text "SDA\nSCL\nINT" (at 198.628 114.3) (layer F.SilkS)
-    (effects (font (size 1.651 1.27) (thickness 0.3048)) (justify right))
-  )
-  (gr_text "INT\nCL\nD" (at 160.782 109.855) (layer F.SilkS)
+  (gr_text "INT\nCK\nD" (at 160.782 109.855) (layer F.SilkS)
     (effects (font (size 1.651 1.27) (thickness 0.3048)) (justify left))
   )
-  (gr_text "INT\nSCL\nSDA" (at 160.909 92.71) (layer F.SilkS)
+  (gr_text "INT\nSCK\nSDA" (at 160.909 92.71) (layer F.SilkS)
     (effects (font (size 1.651 1.27) (thickness 0.3048)) (justify left))
   )
@@
     (effects (font (size 1.397 1.27) (thickness 0.3048)) (justify mirror))
   )
-  (gr_text "PWB\nREV X3" (at 168.91 123.19) (layer F.SilkS)
+  (gr_text "PWB\nREV X2" (at 168.91 123.19) (layer F.SilkS)
     (effects (font (thickness 0.3048)))
   )
