File: PULSE-GEN/Rev-X3/PULSE-GEN.sch (KiCad schematic (older format))
At the start: 25 parts, among them P1 CONN_2, P2 CONN_2, U1 74AC14

Commit message: Added 50/75 Ohm select and Test Stamp location
Parts:
- C2: footprint C1.5V8V -> Capacitors_ThroughHole:C_Radial_D5_L11_P2.5
- R2, R3, R4, R5, R6: value 240 -> 249
Changed lines of the file:
@@
 P 6100 3400
 F 0 "R2" V 6180 3400 40  0000 C CNN
-F 1 "240" V 6107 3401 40  0000 C CNN
+F 1 "249" V 6107 3401 40  0000 C CNN
 F 2 "SM0805" V 6030 3400 30  0000 C CNN
 F 3 "~" H 6100 3400 30  0000 C CNN
@@
 P 6100 3800
 F 0 "R3" V 6180 3800 40  0000 C CNN
-F 1 "240" V 6107 3801 40  0000 C CNN
+F 1 "249" V 6107 3801 40  0000 C CNN
 F 2 "SM0805" V 6030 3800 30  0000 C CNN
 F 3 "~" H 6100 3800 30  0000 C CNN
@@
 P 6100 4200
 F 0 "R4" V 6180 4200 40  0000 C CNN
-F 1 "240" V 6107 4201 40  0000 C CNN
+F 1 "249" V 6107 4201 40  0000 C CNN
 F 2 "SM0805" V 6030 4200 30  0000 C CNN
 F 3 "~" H 6100 4200 30  0000 C CNN
@@
 P 6100 4600
 F 0 "R5" V 6180 4600 40  0000 C CNN
-F 1 "240" V 6107 4601 40  0000 C CNN
+F 1 "249" V 6107 4601 40  0000 C CNN
 F 2 "SM0805" V 6030 4600 30  0000 C CNN
 F 3 "~" H 6100 4600 30  0000 C CNN
@@
 P 6100 5000
 F 0 "R6" V 6180 5000 40  0000 C CNN
-F 1 "240" V 6107 5001 40  0000 C CNN
+F 1 "249" V 6107 5001 40  0000 C CNN
 F 2 "SM0805" V 6030 5000 30  0000 C CNN
 F 3 "~" H 6100 5000 30  0000 C CNN
@@
 F 0 "C2" H 2000 7600 50  0000 L CNN
 F 1 "47uF" H 2000 7400 50  0000 L CNN
-F 2 "C1.5V8V" H 1950 7500 60  0000 C CNN
+F 2 "Capacitors_ThroughHole:C_Radial_D5_L11_P2.5" H 1950 7200 30  0000 C CNN
 F 3 "~" H 1950 7500 60  0000 C CNN
 	1    1950 7500
@@
 F 0 "C3" H 2900 7600 40  0000 L CNN
 F 1 "0.1uF" H 2906 7415 40  0000 L CNN
-F 2 "SM0805" H 2938 7350 30  0000 C CNN
+F 2 "SM0805" H 2900 7200 30  0000 C CNN
 F 3 "~" H 2900 7500 60  0000 C CNN
 	1    2900 7500
@@
 F 0 "C4" H 2400 7600 40  0000 L CNN
 F 1 "0.1uF" H 2406 7415 40  0000 L CNN
-F 2 "SM0805" H 2438 7350 30  0000 C CNN
+F 2 "SM0805" H 2400 7150 30  0000 C CNN
 F 3 "~" H 2400 7500 60  0000 C CNN
 	1    2400 7500
@@
 F 0 "DS1" H 3550 7600 50  0000 C CNN
 F 1 "LED" H 3550 7400 50  0000 C CNN
-F 2 "LED-0805" H 3550 7650 60  0000 C CNN
+F 2 "LED-0805" H 3550 7650 30  0000 C CNN
 F 3 "~" H 3550 7500 60  0000 C CNN
 	1    3550 7500
