File: Proto16-I2C/Proto16-I2C.kicad_pcb (KiCad board)
At the start: 2 copper layers, 77 x 95 mm, 45 parts, among them J1 DB25, J6 CONN_02X02, P1 CONN_01X10, P10 CONN_01X10, P11 CONN_01X10, P12 CONN_01X10, P13 CONN_01X10, P14 CONN_01X10, P15 CONN_01X10, P16 CONN_01X10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

Commit message: Some new DAS family cards
Parts:
- added H7: CONN_01X02, Pin_Headers:Pin_Header_Angled_1x02, F.Cu at (24.6, 16.8)
- moved F1 2.54 mm to (28.7, 23.6)
- renumbered J6 to H6
Connections:
- net Net-(J7-Pad10) renamed /B10
- net Net-(J7-Pad11) renamed /B11
- net Net-(J7-Pad16) renamed /B16
- net Net-(J7-Pad17) renamed /B17
- net Net-(J7-Pad18) renamed /B18
- net Net-(J7-Pad19) renamed /B19
- net Net-(J7-Pad20) renamed /B20
- net Net-(J7-Pad21) renamed /B21
- net Net-(J7-Pad22) renamed /B22
- net Net-(J7-Pad23) renamed /B23
- net Net-(J7-Pad3) renamed /B3
- net Net-(J7-Pad4) renamed /B4
- net Net-(J7-Pad5) renamed /B5
- net Net-(J7-Pad6) renamed /B6
- net Net-(J7-Pad8) renamed /B8
- net Net-(J7-Pad9) renamed /B9
- net Net-(P19-Pad2) renamed /G7
- net Net-(P19-Pad3) renamed /G6
- net Net-(P19-Pad4) renamed /G5
- net Net-(P19-Pad5) renamed /G4
- net Net-(P19-Pad6) renamed /G3
- net Net-(P19-Pad7) renamed /G2
- net Net-(P19-Pad8) renamed /G1
- net Net-(P19-Pad9) renamed /G0
- net Net-(P20-Pad2) renamed /G8
- net Net-(P20-Pad3) renamed /G9
- net Net-(P20-Pad4) renamed /G10
- net Net-(P20-Pad5) renamed /G11
- net Net-(P20-Pad6) renamed /G12
- net Net-(P20-Pad7) renamed /G13
- net Net-(P20-Pad8) renamed /G14
- net Net-(P20-Pad9) renamed /G15
- H2 pad 2: /INT1 -> /IA
- J1 pad 12: Net-(J7-Pad12) -> Net-(F1-Pad2)
- J1 pad 15: Net-(J7-Pad15) -> /B15
- J1 pad 2: Net-(J7-Pad15) -> GND
- J1 pad 24: Net-(J7-Pad12) -> /B24
- J1 pad 7: (no net) -> /B7
- P1 pad 1: +5V -> Net-(P1-Pad1)
- P1 pad 10: GND -> Net-(P1-Pad10)
- P10 pad 1: +5V -> Net-(P10-Pad1)
- P10 pad 10: GND -> Net-(P10-Pad10)
- P11 pad 1: Net-(J7-Pad12) -> Net-(P11-Pad1)
- P11 pad 10: Net-(J7-Pad15) -> Net-(P11-Pad10)
- P12 pad 1: Net-(J7-Pad12) -> Net-(P12-Pad1)
- P12 pad 10: Net-(J7-Pad15) -> Net-(P12-Pad10)
- P13 pad 1: Net-(J7-Pad12) -> Net-(P11-Pad1)
- P13 pad 10: Net-(J7-Pad15) -> Net-(P11-Pad10)
- P14 pad 1: Net-(J7-Pad12) -> Net-(P12-Pad1)
- P14 pad 10: Net-(J7-Pad15) -> Net-(P12-Pad10)
- P15 pad 1: Net-(J7-Pad12) -> Net-(P12-Pad1)
- P15 pad 10: Net-(J7-Pad15) -> Net-(P12-Pad10)
- P16 pad 1: Net-(J7-Pad12) -> Net-(P11-Pad1)
- P16 pad 10: Net-(J7-Pad15) -> Net-(P11-Pad10)
- P17 pad 1: Net-(J7-Pad12) -> /B24
- P17 pad 10: Net-(J7-Pad15) -> /B7
- P18 pad 1: Net-(J7-Pad12) -> /B7
- P18 pad 10: Net-(J7-Pad15) -> /B15
- P19 pad 1: +5V -> /IB
- P19 pad 10: GND -> /RST
- P20 pad 1: +5V -> (no net)
- P20 pad 10: GND -> /IA
- P3 pad 1: +5V -> Net-(P1-Pad1)
- P3 pad 10: GND -> Net-(P1-Pad10)
- P4 pad 1: +5V -> Net-(P10-Pad1)
- P4 pad 10: GND -> Net-(P10-Pad10)
- P7 pad 1: +5V -> Net-(P1-Pad1)
- P7 pad 10: GND -> Net-(P1-Pad10)
- P99 pad 1: +5V -> Net-(P10-Pad1)
- P99 pad 10: GND -> Net-(P10-Pad10)
- R7 pad 1: /INT1 -> /IA
- U1 pad 19: (no net) -> /IB
- U1 pad 20: /INT1 -> /IA
Routing:
- net Net-(J7-Pad12): track 56.3 -> 0.00 mm
- net Net-(J7-Pad15): track 53.5 -> 0.00 mm, vias 2 -> 0
- net /IA: track 0.00 -> 32.5 mm
- net /RST: track 7.28 -> 38.1 mm, vias 0 -> 1
- net /B24: track 0.00 -> 24.2 mm
- net /IB: track 0.00 -> 20.9 mm
- net /B15: track 0.00 -> 16.4 mm
- net /B7: track 0.00 -> 14.9 mm
- net /INT1: track 11.5 -> 0.00 mm
- net GND: track 7.32 -> 0.00 mm
- net Net-(F1-Pad2): track 28.5 -> 34.8 mm
- net Net-(P10-Pad10): track 0.00 -> 5.08 mm
- net Net-(P10-Pad1): track 0.00 -> 5.08 mm
- net Net-(P1-Pad10): track 0.00 -> 5.08 mm
- net Net-(P1-Pad1): track 0.00 -> 5.08 mm
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Other:
- board text added: "0"
- board text added: "10"
- board text added: "11"
- board text added: "12"
- board text added: "13"
- board text added: "14"
- board text added: "15"
- board text added: "16"
- board text added: "17"
- board text added: "18"
- board text added: "19"
- board text added: "2"
- board text added: "20"
- board text added: "21"
- board text added: "22"
- board text added: "23"
- board text added: "24"
- board text added: "3"
- board text added: "4"
- board text added: "5"
- board text added: "6"
- board text added: "7"
- board text added: "8"
- board text added: "9"
- board text added: "BASE ADDR EEP-x50 I/O-x20"
- board text added: "BUS"
- board text added: "DB"
- board text added: "DB PWR"
- board text added: "DIO"
- board text added: "IA"
- board text added: "IB"
- board text added: "VCC"
- board text added: "~RST"
- board text removed: "BASE ADDR EEP-x50 I/O-x20 -21"
