File: ODAS Cards/OPSOC5-95MM-01/OPSOC5-95MM-01.sch (KiCad schematic (older format))
At the start: 45 parts, among them CON1 USB-MINI-B, J1 DCJ0202, P1 DC-62, P2 CONN_01X04, P4 CONN_01X06, U1 AP1117, U2 CY8C5267AXI-LP051, U4 AP1117, Y1 Crystal_Small

Commit message: 95mm card hw
Parts:
- C17: footprint Capacitors_ThroughHole:C_Radial_D14_L25_P5 -> Capacitors_ThroughHole:C_Radial_D5_L11_P2.5; symbol CP -> CP-RESCUE-OPSOC5-95MM-01
Connections:
- wire segments 265 -> 263
Changed lines of the file:
@@
 EESchema Schematic File Version 2
-LIBS:DougsSch
+LIBS:OPSOC5-95MM-01-rescue
 LIBS:power
 LIBS:device
@@
 	2500 2400 2500 2500
 Wire Wire Line
-	2600 2300 2250 2300
-Wire Wire Line
-	2250 2300 2250 2000
+	1650 2300 2600 2300
 Text Label 1800 3450 0    60   ~ 0
 SPIMISO
@@
 	2400 3850 2400 3950
 Wire Wire Line
-	2400 3750 2400 3250
-$Comp
-L +3.3V-RESCUE-ODAS-PSOC5 #PWR024
-U 1 1 5815F767
-P 2400 3250
-F 0 "#PWR024" H 2400 3100 50  0001 C CNN
-F 1 "+3.3V" H 2400 3390 50  0000 C CNN
-F 2 "" H 2400 3250 60  0000 C CNN
-F 3 "" H 2400 3250 60  0000 C CNN
-	1    2400 3250
-	1    0    0    -1
-$EndComp
-Wire Wire Line
-	2500 3750 2400 3750
-$Comp
-L GND-RESCUE-ODAS-PSOC5 #PWR025
+	1550 3750 2500 3750
+$Comp
+L GND-RESCUE-ODAS-PSOC5 #PWR024
 U 1 1 581F7477
 P 6700 4200
-F 0 "#PWR025" H 6700 4200 30  0001 C CNN
+F 0 "#PWR024" H 6700 4200 30  0001 C CNN
 F 1 "GND" H 6700 4130 30  0001 C CNN
 F 2 "" H 6700 4200 60  0000 C CNN
@@
 NoConn ~ 8550 4250
 $Comp
-L GND-RESCUE-ODAS-PSOC5 #PWR026
+L GND-RESCUE-ODAS-PSOC5 #PWR025
 U 1 1 5820B585
 P 14850 1650
-F 0 "#PWR026" H 14850 1400 50  0001 C CNN
+F 0 "#PWR025" H 14850 1400 50  0001 C CNN
 F 1 "GND" H 14850 1500 50  0000 C CNN
 F 2 "" H 14850 1650 60  0000 C CNN
@@
 Connection ~ 1600 9950
 $Comp
-L CP C17
+L CP-RESCUE-OPSOC5-95MM-01 C17
 U 1 1 586FA9E9
 P 2300 9600
 F 0 "C17" H 2350 9700 50  0000 L CNN
 F 1 "CP" H 2350 9500 50  0000 L CNN
-F 2 "Capacitors_ThroughHole:C_Radial_D14_L25_P5" H 2300 9400 20  0000 C CNN
+F 2 "Capacitors_ThroughHole:C_Radial_D5_L11_P2.5" H 2300 9400 20  0000 C CNN
 F 3 "" H 2300 9600 60  0000 C CNN
 	1    2300 9600
@@
 	2300 9800 2300 9950
 Connection ~ 2300 9950
+Text Label 1800 3750 0    60   ~ 0
+VZ1
+Text Label 1850 2300 0    60   ~ 0
+VZ1
 $EndSCHEMATC

Commit message: pin 23 of p1
Connections:
- wire segments 263 -> 262
Changed lines of the file:
@@
 	14200 2000 15150 2000
-Wire Wire Line
-	14200 2100 15150 2100
 Wire Wire Line
 	14200 2200 15150 2200
@@
 Text Label 14400 2000 0    60   ~ 0
 P24
-Text Label 14400 2100 0    60   ~ 0
-P23
 Text Label 14400 2200 0    60   ~ 0
 P22

Commit message: Updates to match part internal pin uses
Connections:
- net labels added: LED
- net labels removed: P28
- wire segments 262 -> 263
Other:
- moved on the sheet: FID1, FID2, MTG1, MTG2, MTG3, MTG4, TEST1
Changed lines of the file:
@@
 EESchema Schematic File Version 2
 LIBS:OPSOC5-95MM-01-rescue
+LIBS:DougsSch
 LIBS:power
 LIBS:device
@@
 L COUPON TEST1
 U 1 1 53B1CE77
-P 9750 10400
-F 0 "TEST1" H 9750 10400 60  0000 C CNN
-F 1 "COUPON" H 9750 10350 60  0000 C CNN
-F 2 "LandBoards_Marking:TEST_BLK-REAR" H 9750 10300 30  0000 C CNN
-F 3 "~" H 9750 10400 60  0000 C CNN
-	1    9750 10400
+P 9500 10350
+F 0 "TEST1" H 9500 10350 60  0000 C CNN
+F 1 "COUPON" H 9500 10300 60  0000 C CNN
+F 2 "LandBoards_Marking:TEST_BLK-REAR" H 9500 10250 30  0000 C CNN
+F 3 "~" H 9500 10350 60  0000 C CNN
+	1    9500 10350
 	1    0    0    -1
 $EndComp
@@
 L CONN_1 MTG4
 U 1 1 53C6E5CF
-P 11450 10450
-F 0 "MTG4" H 11530 10450 40  0000 L CNN
-F 1 "CONN_1" H 11450 10505 30  0001 C CNN
-F 2 "LandBoards_MountHoles:MTG-6-32" H 11950 10450 30  0000 C CNN
-F 3 "" H 11450 10450 60  0000 C CNN
-	1    11450 10450
+P 11200 10400
+F 0 "MTG4" H 11280 10400 40  0000 L CNN
+F 1 "CONN_1" H 11200 10455 30  0001 C CNN
+F 2 "LandBoards_MountHoles:MTG-6-32" H 11700 10400 30  0000 C CNN
+F 3 "" H 11200 10400 60  0000 C CNN
+	1    11200 10400
 	1    0    0    -1
 $EndComp
@@
 L CONN_1 MTG3
 U 1 1 53C6E5DE
-P 11450 10350
-F 0 "MTG3" H 11530 10350 40  0000 L CNN
-F 1 "CONN_1" H 11450 10405 30  0001 C CNN
-F 2 "LandBoards_MountHoles:MTG-6-32" H 11950 10350 30  0000 C CNN
-F 3 "" H 11450 10350 60  0000 C CNN
-	1    11450 10350
+P 11200 10300
+F 0 "MTG3" H 11280 10300 40  0000 L CNN
+F 1 "CONN_1" H 11200 10355 30  0001 C CNN
+F 2 "LandBoards_MountHoles:MTG-6-32" H 11700 10300 30  0000 C CNN
+F 3 "" H 11200 10300 60  0000 C CNN
+	1    11200 10300
 	1    0    0    -1
 $EndComp
@@
 L CONN_1 MTG2
 U 1 1 53C6E5ED
-P 11450 10250
-F 0 "MTG2" H 11530 10250 40  0000 L CNN
-F 1 "CONN_1" H 11450 10305 30  0001 C CNN
-F 2 "LandBoards_MountHoles:MTG-6-32" H 11950 10250 30  0000 C CNN
-F 3 "" H 11450 10250 60  0000 C CNN
-	1    11450 10250
+P 11200 10200
+F 0 "MTG2" H 11280 10200 40  0000 L CNN
+F 1 "CONN_1" H 11200 10255 30  0001 C CNN
+F 2 "LandBoards_MountHoles:MTG-6-32" H 11700 10200 30  0000 C CNN
+F 3 "" H 11200 10200 60  0000 C CNN
+	1    11200 10200
 	1    0    0    -1
 $EndComp
@@
 L CONN_1 MTG1
 U 1 1 53C6E5FC
-P 11450 10150
-F 0 "MTG1" H 11530 10150 40  0000 L CNN
-F 1 "CONN_1" H 11450 10205 30  0001 C CNN
-F 2 "LandBoards_MountHoles:MTG-6-32" H 11950 10150 30  0000 C CNN
-F 3 "" H 11450 10150 60  0000 C CNN
-	1    11450 10150
-	1    0    0    -1
-$EndComp
-NoConn ~ 11300 10450
-NoConn ~ 11300 10350
-NoConn ~ 11300 10250
-NoConn ~ 11300 10150
+P 11200 10100
+F 0 "MTG1" H 11280 10100 40  0000 L CNN
+F 1 "CONN_1" H 11200 10155 30  0001 C CNN
+F 2 "LandBoards_MountHoles:MTG-6-32" H 11700 10100 30  0000 C CNN
+F 3 "" H 11200 10100 60  0000 C CNN
+	1    11200 10100
+	1    0    0    -1
+$EndComp
+NoConn ~ 11050 10400
+NoConn ~ 11050 10300
+NoConn ~ 11050 10200
+NoConn ~ 11050 10100
 $Comp
 L FUSE F1
@@
 L CONN_1 FID1
 U 1 1 53F2073B
-P 10900 10250
-F 0 "FID1" H 10980 10250 40  0000 L CNN
-F 1 "CONN_1" H 10900 10305 30  0001 C CNN
-F 2 "LandBoards_Marking:FIDUCIAL" H 10900 10200 30  0000 C CNN
-F 3 "" H 10900 10250 60  0000 C CNN
-	1    10900 10250
+P 10650 10200
+F 0 "FID1" H 10730 10200 40  0000 L CNN
+F 1 "CONN_1" H 10650 10255 30  0001 C CNN
+F 2 "LandBoards_Marking:FIDUCIAL" H 10650 10150 30  0000 C CNN
+F 3 "" H 10650 10200 60  0000 C CNN
+	1    10650 10200
 	1    0    0    -1
 $EndComp
@@
 L CONN_1 FID2
 U 1 1 53F2074A
-P 10900 10350
-F 0 "FID2" H 10980 10350 40  0000 L CNN
-F 1 "CONN_1" H 10900 10405 30  0001 C CNN
-F 2 "LandBoards_Marking:FIDUCIAL" H 10900 10300 30  0000 C CNN
-F 3 "" H 10900 10350 60  0000 C CNN
-	1    10900 10350
-	1    0    0    -1
-$EndComp
-NoConn ~ 10750 10250
-NoConn ~ 10750 10350
+P 10650 10300
+F 0 "FID2" H 10730 10300 40  0000 L CNN
+F 1 "CONN_1" H 10650 10355 30  0001 C CNN
+F 2 "LandBoards_Marking:FIDUCIAL" H 10650 10250 30  0000 C CNN
+F 3 "" H 10650 10300 60  0000 C CNN
+	1    10650 10300
+	1    0    0    -1
+$EndComp
+NoConn ~ 10500 10200
+NoConn ~ 10500 10300
 $Comp
 L GND-RESCUE-ODAS-PSOC5 #PWR01
@@
 	0    1    1    0
 $EndComp
-Text Label 8100 4150 0    60   ~ 0
-P28
 $Comp
 L C-RESCUE-ODAS-PSOC5 C5
@@
 P22
 Wire Wire Line
-	14200 1900 15150 1900
-Wire Wire Line
 	14200 2000 15150 2000
 Wire Wire Line
+	14200 2100 15150 2100
+Wire Wire Line
 	14200 2200 15150 2200
-Text Label 14400 1900 0    60   ~ 0
+Text Label 14400 2000 0    60   ~ 0
 P25
-Text Label 14400 2000 0    60   ~ 0
+Text Label 14400 2100 0    60   ~ 0
 P24
 Text Label 14400 2200 0    60   ~ 0
@@
 	15150 1800 15050 1800
 Wire Wire Line
-	15050 1800 15050 1600
+	15050 1600 15050 1900
 Wire Wire Line
 	1950 1100 2200 1100
@@
 Text Label 1850 2300 0    60   ~ 0
 VZ1
+Connection ~ 15050 1800
+Wire Wire Line
+	15050 1900 15150 1900
+Text Label 8050 4150 0    60   ~ 0
+LED
 $EndSCHEMATC

Commit message: PSOC card
Parts:
- renumbered CON1 to J2
Connections:
- no-connect marks 22 -> 23
Other:
- note added: "PROGRAMMING HEADER"
- note added: "SPI CONNECTOR"
- note added: "USB CONNECTOR"
- note added: "ZONE VOLTAGE SELECTION HEADERS"
- moved on the sheet: J2, P2, R6, R7
Changed lines of the file:
@@
 encoding utf-8
 Sheet 1 1
-Title "RASPBERRY PI PSOC HAT"
-Date "Saturday, December 19, 2015"
-Rev "X2"
+Title "ODAS PSOC CARD"
+Date "Monday, February 06, 2017"
+Rev "X1"
 Comp ""
 Comment1 ""
@@
 F 0 "C3" H 3075 7050 50  0000 L CNN
 F 1 "0.1uF" H 3075 6850 50  0000 L CNN
-F 2 "Capacitors_SMD:C_0805_HandSoldering" H 3050 6750 30  0000 C CNN
+F 2 "Capacitors_SMD:C_0805_HandSoldering" H 3050 6650 30  0000 C CNN
 F 3 "" H 3050 6950 60  0000 C CNN
 	1    3050 6950
@@
 F 0 "C4" H 2375 7050 50  0000 L CNN
 F 1 "0.1uF" H 2375 6850 50  0000 L CNN
-F 2 "Capacitors_SMD:C_0805_HandSoldering" H 2350 6750 30  0000 C CNN
+F 2 "Capacitors_SMD:C_0805_HandSoldering" H 2350 6700 30  0000 C CNN
 F 3 "" H 2350 6950 60  0000 C CNN
 	1    2350 6950
@@
 F 0 "H1" H 6750 4950 50  0000 C CNN
 F 1 "CONN_01X04" V 6850 4700 50  0000 C CNN
-F 2 "Pin_Headers:Pin_Header_Angled_1x04_Pitch2.54mm" H 6750 4450 20  0000 C CNN
+F 2 "Pin_Headers:Pin_Header_Angled_1x04_Pitch2.54mm" H 6850 5000 20  0000 C CNN
 F 3 "" H 6750 4700 50  0000 C CNN
 	1    6750 4700
@@
 L R-RESCUE-ODAS-PSOC5 R6
 U 1 1 581213EC
+P 1800 1000
+F 0 "R6" V 1750 850 50  0000 C CNN
+F 1 "22" V 1800 1000 50  0000 C CNN
+F 2 "Resistors_SMD:R_0805_HandSoldering" V 1730 1000 30  0000 C CNN
+F 3 "" H 1800 1000 30  0000 C CNN
+	1    1800 1000
+	0    1    1    0
+$EndComp
+$Comp
+L R-RESCUE-ODAS-PSOC5 R7
+U 1 1 58121717
 P 1800 1100
-F 0 "R6" V 1750 950 50  0000 C CNN
+F 0 "R7" V 1750 950 50  0000 C CNN
 F 1 "22" V 1800 1100 50  0000 C CNN
 F 2 "Resistors_SMD:R_0805_HandSoldering" V 1730 1100 30  0000 C CNN
@@
 $EndComp
 $Comp
-L R-RESCUE-ODAS-PSOC5 R7
-U 1 1 58121717
-P 1800 1200
-F 0 "R7" V 1750 1050 50  0000 C CNN
-F 1 "22" V 1800 1200 50  0000 C CNN
-F 2 "Resistors_SMD:R_0805_HandSoldering" V 1730 1200 30  0000 C CNN
-F 3 "" H 1800 1200 30  0000 C CNN
-	1    1800 1200
-	0    1    1    0
-$EndComp
-Wire Wire Line
-	2200 1400 2050 1400
-Wire Wire Line
-	2050 1400 2050 1650
-$Comp
 L GND-RESCUE-ODAS-PSOC5 #PWR015
 U 1 1 581227BC
-P 2050 1650
-F 0 "#PWR015" H 2050 1400 50  0001 C CNN
-F 1 "GND" H 2050 1500 50  0000 C CNN
-F 2 "" H 2050 1650 60  0000 C CNN
-F 3 "" H 2050 1650 60  0000 C CNN
-	1    2050 1650
-	1    0    0    -1
-$EndComp
+P 2100 1400
+F 0 "#PWR015" H 2100 1150 50  0001 C CNN
+F 1 "GND" H 2100 1250 50  0000 C CNN
+F 2 "" H 2100 1400 60  0000 C CNN
+F 3 "" H 2100 1400 60  0000 C CNN
+	1    2100 1400
+	1    0    0    -1
+$EndComp
+Text Label 1100 1000 0    60   ~ 0
+USB-DM
 Text Label 1100 1100 0    60   ~ 0
-USB-DM
-Text Label 1100 1200 0    60   ~ 0
 USB-DP
 Wire Wire Line
+	950  1000 1650 1000
+Wire Wire Line
 	950  1100 1650 1100
-Wire Wire Line
-	950  1200 1650 1200
 $Comp
 L Crystal_Small Y1
@@
 F 0 "Y1" H 12300 6850 50  0000 C CNN
 F 1 "Crystal_Small" H 12300 6650 50  0000 C CNN
-F 2 "Crystals:Crystal_HC49-U_Vertical" H 12300 6750 60  0000 C CNN
+F 2 "Crystals:Crystal_HC49-U_Vertical" H 11800 6800 20  0000 C CNN
 F 3 "" H 12300 6750 60  0000 C CNN
 	1    12300 6750
@@
 F 0 "C7" H 12625 6650 50  0000 L CNN
 F 1 "C" H 12625 6450 50  0000 L CNN
-F 2 "Capacitors_SMD:C_0805_HandSoldering" H 12638 6400 30  0000 C CNN
+F 2 "Capacitors_SMD:C_0805_HandSoldering" H 12600 6900 30  0000 C CNN
 F 3 "" H 12600 6550 60  0000 C CNN
 	1    12600 6550
@@
 F 0 "C10" H 12625 7050 50  0000 L CNN
 F 1 "C" H 12625 6850 50  0000 L CNN
-F 2 "Capacitors_SMD:C_0805_HandSoldering" H 12638 6800 30  0000 C CNN
+F 2 "Capacitors_SMD:C_0805_HandSoldering" H 12600 7350 30  0000 C CNN
 F 3 "" H 12600 6950 60  0000 C CNN
 	1    12600 6950
@@
 L CONN_01X04 P2
 U 1 1 58146640
-P 2800 2250
-F 0 "P2" H 2800 2500 50  0000 C CNN
-F 1 "CONN_01X04" V 2900 2250 50  0000 C CNN
-F 2 "Pin_Headers:Pin_Header_Angled_1x04" V 2950 2250 20  0000 C CNN
-F 3 "" H 2800 2250 60  0000 C CNN
-	1    2800 2250
+P 2800 2400
+F 0 "P2" H 2800 2650 50  0000 C CNN
+F 1 "CONN_01X04" V 2900 2400 50  0000 C CNN
+F 2 "Pin_Headers:Pin_Header_Angled_1x04" H 2850 2700 20  0000 C CNN
+F 3 "" H 2800 2400 60  0000 C CNN
+	1    2800 2400
 	1    0    0    1
 $EndComp
 Wire Wire Line
-	1650 2100 2600 2100
-Wire Wire Line
-	1650 2200 2600 2200
-Text Label 1850 2100 0    60   ~ 0
+	1650 2250 2600 2250
+Wire Wire Line
+	1650 2350 2600 2350
+Text Label 1850 2250 0    60   ~ 0
 SCLK1
-Text Label 1850 2200 0    60   ~ 0
+Text Label 1850 2350 0    60   ~ 0
 SDA1
 $Comp
 L GND-RESCUE-ODAS-PSOC5 #PWR017
 U 1 1 58146C6C
-P 2500 2500
-F 0 "#PWR017" H 2500 2250 50  0001 C CNN
-F 1 "GND" H 2500 2350 50  0000 C CNN
-F 2 "" H 2500 2500 60  0000 C CNN
-F 3 "" H 2500 2500 60  0000 C CNN
-	1    2500 2500
-	1    0    0    -1
-$EndComp
-Wire Wire Line
-	2600 2400 2500 2400
+P 2500 2650
+F 0 "#PWR017" H 2500 2400 50  0001 C CNN
+F 1 "GND" H 2500 2500 50  0000 C CNN
+F 2 "" H 2500 2650 60  0000 C CNN
+F 3 "" H 2500 2650 60  0000 C CNN
+	1    2500 2650
+	1    0    0    -1
+$EndComp
+Wire Wire Line
+	2600 2550 2500 2550
 Text Label 1300 9250 0    60   ~ 0
 +9V
@@
 F 0 "C12" H 1600 9700 40  0000 L CNN
 F 1 "0.1uF" H 1606 9515 40  0000 L CNN
-F 2 "Capacitors_SMD:C_0805_HandSoldering" H 1750 9450 30  0000 C CNN
+F 2 "Capacitors_SMD:C_0805_HandSoldering" H 1600 9400 20  0000 C CNN
 F 3 "~" H 1600 9600 60  0000 C CNN
 	1    1600 9600
@@
 F 0 "C13" H 3950 9700 40  0000 L CNN
 F 1 "0.1uF" H 3956 9515 40  0000 L CNN
-F 2 "Capacitors_SMD:C_0805_HandSoldering" H 4100 9450 30  0000 C CNN
+F 2 "Capacitors_SMD:C_0805_HandSoldering" H 3950 9400 30  0000 C CNN
 F 3 "~" H 3950 9600 60  0000 C CNN
 	1    3950 9600
@@
 F 0 "C15" H 5450 9700 40  0000 L CNN
 F 1 "0.1uF" H 5456 9515 40  0000 L CNN
-F 2 "Capacitors_SMD:C_0805_HandSoldering" H 5600 9450 30  0000 C CNN
+F 2 "Capacitors_SMD:C_0805_HandSoldering" H 5450 9400 30  0000 C CNN
 F 3 "~" H 5450 9600 60  0000 C CNN
 	1    5450 9600
@@
 	15000 7800 15000 8000
 Wire Wire Line
-	2500 2400 2500 2500
-Wire Wire Line
-	1650 2300 2600 2300
+	2500 2550 2500 2650
+Wire Wire Line
+	1650 2450 2600 2450
 Text Label 1800 3450 0    60   ~ 0
 SPIMISO
@@
 F 0 "P4" H 2700 3950 50  0000 C CNN
 F 1 "CONN_01X06" V 2800 3600 50  0000 C CNN
-F 2 "Pin_Headers:Pin_Header_Angled_1x06_Pitch2.54mm" V 2850 3600 20  0000 C CNN
+F 2 "Pin_Headers:Pin_Header_Angled_1x06_Pitch2.54mm" H 2850 4000 20  0000 C CNN
 F 3 "" H 2700 3600 60  0000 C CNN
 	1    2700 3600
@@
 	1    0    0    -1
 $EndComp
+NoConn ~ 3200 900
 NoConn ~ 3200 1000
-NoConn ~ 3200 1100
+NoConn ~ 3200 1200
 NoConn ~ 3200 1300
-NoConn ~ 3200 1400
-NoConn ~ 2200 1000
-NoConn ~ 2200 1300
+NoConn ~ 2200 900
+NoConn ~ 2200 1200
 NoConn ~ 8550 4250
 $Comp
@@
 $EndComp
 $Comp
-L USB-MINI-B CON1
+L USB-MINI-B J2
 U 1 1 586C1544
-P 2700 1200
-F 0 "CON1" H 2400 1550 50  0000 C CNN
-F 1 "USB-MINI-B" H 2550 850 50  0000 C CNN
-F 2 "LandBoards_Conns:USB-B-MINI" H 2700 750 50  0000 C CNN
-F 3 "" H 2700 1100 50  0000 C CNN
-	1    2700 1200
+P 2700 1100
+F 0 "J2" H 2400 1450 50  0000 C CNN
+F 1 "USB-MINI-B" H 2550 750 50  0000 C CNN
+F 2 "LandBoards_Conns:USB-B-MINI" H 2800 650 20  0000 C CNN
+F 3 "" H 2700 1000 50  0000 C CNN
+	1    2700 1100
 	1    0    0    -1
 $EndComp
@@
 F 0 "U2" H 10700 7800 50  0000 C CNN
 F 1 "CY8C5267AXI-LP051" H 10850 2400 50  0000 C CNN
-F 2 "LIBRARY:TQFP-100_14x14mm_Pitch0.5mm" H 11350 2250 50  0000 C CNN
+F 2 "LIBRARY:TQFP-100_14x14mm_Pitch0.5mm" H 11200 2300 50  0000 C CNN
 F 3 "DOCUMENTATION" H 9900 5100 50  0001 C CNN
 	1    9900 5100
@@
 	15050 1600 15050 1900
 Wire Wire Line
-	1950 1100 2200 1100
-Wire Wire Line
-	2200 1200 1950 1200
+	1950 1000 2200 1000
+Wire Wire Line
+	2200 1100 1950 1100
 Text Label 11350 5950 0    60   ~ 0
 USB-DM
@@
 F 0 "C1" H 1950 9700 40  0000 L CNN
 F 1 "10uF" H 1956 9515 40  0000 L CNN
-F 2 "Capacitors_SMD:C_1206_HandSoldering" H 2100 9450 30  0000 C CNN
+F 2 "Capacitors_SMD:C_1206_HandSoldering" H 2100 9450 20  0000 C CNN
 F 3 "~" H 1950 9600 60  0000 C CNN
 	1    1950 9600
@@
 Text Label 1800 3750 0    60   ~ 0
 VZ1
-Text Label 1850 2300 0    60   ~ 0
+Text Label 1850 2450 0    60   ~ 0
 VZ1
 Connection ~ 15050 1800
@@
 Text Label 8050 4150 0    60   ~ 0
 LED
+Text Notes 2050 2950 0    60   ~ 0
+PROGRAMMING HEADER
+Text Notes 2300 1800 0    60   ~ 0
+USB CONNECTOR
+Text Notes 2050 4300 0    60   ~ 0
+SPI CONNECTOR
+Text Notes 1400 7550 0    60   ~ 0
+ZONE VOLTAGE SELECTION HEADERS
+NoConn ~ 15150 7700
+Wire Wire Line
+	2100 1400 2100 1300
+Wire Wire Line
+	2100 1300 2200 1300
 $EndSCHEMATC
