File: ODAS Cards/ODAS-PSOC5/Rev X3/ODAS-PSOC5.kicad_pcb (KiCad board)
At the start: 2 copper layers, 55 x 95 mm, 48 parts, among them J1 DCJ0202, J2 USB-MICRO-B, P1 CONN_01X40, P2 CONN_01X04, P3 CONN_02X02, P4 CONN_01X06, U1 24C32, U2 CY8C5267AXI-LP051, U3 AP1117, U4 AP1117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

Commit message: Card pics and updates to ODAS-PSOC5
Parts:
- U3, U4: footprint TO_SOT_Packages_SMD:SOT-223 -> dougsLib:SOT223
Connections:
- U3 pad 4: +5V -> (no net)
- U4 pad 4: +3V3 -> (no net)
Other:
- board text added: "REV X3"
- board text removed: "REV X4"
