File: BeagleBoneBlack Cards/BBB-GVS-3/BBB-Conn.sch (KiCad schematic (older format))
At the start: 16 parts, among them J11 CONN_2, J25 CONN_3, U1 I2C-EEPROM

Commit message: pics and bbb-gvs
Parts:
- C1, C2, C3, C4: symbol C -> C-RESCUE-BBB-GVS-3
- D1, D2: symbol LED -> LED-RESCUE-BBB-GVS-3
- R1, R2, R3, R4, R5: symbol R -> R-RESCUE-BBB-GVS-3
Changed lines of the file:
@@
 EESchema Schematic File Version 2
-LIBS:DougsSch
+LIBS:BBB-GVS-3-rescue
 LIBS:power
 LIBS:device
 LIBS:conn
 LIBS:TXB0108
-LIBS:beaglebone
 LIBS:linear
 LIBS:memory
@@
 $EndDescr
 $Comp
-L GND #U01
+L GND-RESCUE-BBB-GVS-3 #U01
 U 1 1 53AEED58
 P 7650 3150
@@
 $EndComp
 $Comp
-L GND #U02
+L GND-RESCUE-BBB-GVS-3 #U02
 U 1 1 53AEED59
 P 6150 2250
@@
 $EndComp
 $Comp
-L C C1
+L C-RESCUE-BBB-GVS-3 C1
 U 1 1 4EB9CBCB
 P 6150 1900
+AR Path="/4EB9CBCB" Ref="C1"  Part="1"
+AR Path="/4EB0F8E9/4EB9CBCB" Ref="C1"  Part="1"
 F 0 "C1" H 6200 2000 50  0000 L CNN
 F 1 "1uF" H 6200 1800 50  0000 L CNN
@@
 $EndComp
 $Comp
-L GND #U03
+L GND-RESCUE-BBB-GVS-3 #U03
 U 1 1 53AEED5A
 P 6750 2550
@@
 $EndComp
 $Comp
-L R R5
+L R-RESCUE-BBB-GVS-3 R5
 U 1 1 4EB9CACE
 P 8750 1850
@@
 $EndComp
 $Comp
-L R R4
+L R-RESCUE-BBB-GVS-3 R4
 U 1 1 4EB9CAC9
 P 8550 1850
@@
 5V SELECTION JUMPER
 $Comp
-L C C2
+L C-RESCUE-BBB-GVS-3 C2
 U 1 1 53ADAE3E
 P 1850 2100
+AR Path="/53ADAE3E" Ref="C2"  Part="1"
+AR Path="/4EB0F8E9/53ADAE3E" Ref="C2"  Part="1"
 F 0 "C2" H 1850 2200 40  0000 L CNN
 F 1 "104" H 1856 2015 40  0000 L CNN
@@
 $EndComp
 $Comp
-L C C3
+L C-RESCUE-BBB-GVS-3 C3
 U 1 1 53ADAE4D
 P 2600 2100
+AR Path="/53ADAE4D" Ref="C3"  Part="1"
+AR Path="/4EB0F8E9/53ADAE4D" Ref="C3"  Part="1"
 F 0 "C3" H 2600 2200 40  0000 L CNN
 F 1 "104" H 2606 2015 40  0000 L CNN
@@
 $EndComp
 $Comp
-L C C4
+L C-RESCUE-BBB-GVS-3 C4
 U 1 1 53ADAE5C
 P 2900 2100
+AR Path="/53ADAE5C" Ref="C4"  Part="1"
+AR Path="/4EB0F8E9/53ADAE5C" Ref="C4"  Part="1"
 F 0 "C4" H 2900 2200 40  0000 L CNN
 F 1 "104" H 2906 2015 40  0000 L CNN
@@
 GND
 $Comp
-L LED D2
+L LED-RESCUE-BBB-GVS-3 D2
 U 1 1 53ADFF8D
 P 3550 2150
@@
 $EndComp
 $Comp
-L R R2
+L R-RESCUE-BBB-GVS-3 R2
 U 1 1 53ADFF9C
 P 3550 1550
@@
 VDD_3V3-UF
 $Comp
-L LED D1
+L LED-RESCUE-BBB-GVS-3 D1
 U 1 1 53C05879
 P 2300 2150
@@
 $EndComp
 $Comp
-L R R1
+L R-RESCUE-BBB-GVS-3 R1
 U 1 1 53C0587F
 P 2300 1550
@@
 $EndComp
 $Comp
-L R R3
+L R-RESCUE-BBB-GVS-3 R3
 U 1 1 53F103C2
 P 8400 1850
