File: ODAS Cards/ESP-32_VGA/ESP-32_VGA.sch (KiCad schematic (older format))
At the start: 40 parts, among them J1 DCJ0202, J15 Conn_01x02, J2 FTDI, J3 PS2_DIN6, J4 PS2_DIN6, J5 Conn_01x02, J7 Conn_01x05, P1 Conn_02x08_Odd_Even, P2 Conn_02x14_Odd_Even, P3 VGA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

Commit message: esp32 vga
Parts:
- removed H1: Conn_01x02, Connector_PinHeader_2.54mm:PinHeader_1x02_P2.54mm_Vertical, symbol Connector_Generic:Conn_01x02
- removed H2: Conn_02x03_Odd_Even, Connector_PinHeader_2.54mm:PinHeader_2x03_P2.54mm_Vertical, symbol Connector_Generic:Conn_02x03_Odd_Even
- removed J5: Conn_01x02, symbol Connector_Generic:Conn_01x02
- removed J7: Conn_01x05, Pin_Headers:Pin_Header_Straight_1x05_Pitch2.54mm, symbol Connector_Generic:Conn_01x05
- removed P1: Conn_02x08_Odd_Even, Pin_Headers:Pin_Header_Straight_2x08_Pitch2.54mm, symbol Connector_Generic:Conn_02x08_Odd_Even
- removed P2: Conn_02x14_Odd_Even, Pin_Headers:Pin_Header_Straight_2x14_Pitch2.54mm, symbol Connector_Generic:Conn_02x14_Counter_Clockwise
- removed P8: Conn_02x03_Odd_Even, Pin_Headers:Pin_Header_Straight_2x03_Pitch2.54mm, symbol Connector_Generic:Conn_02x03_Odd_Even
- removed R10, R7, R8, R9: 120, Resistor_SMD:R_0805_2012Metric_Pad1.15x1.40mm_HandSolder, symbol Device:R
- added H1: Conn_01x03, Connector_PinHeader_2.54mm:PinHeader_1x03_P2.54mm_Vertical, symbol Connector_Generic:Conn_01x03
- added H2: Conn_02x04_Odd_Even, Connector_PinHeader_2.54mm:PinHeader_2x04_P2.54mm_Vertical, symbol Connector_Generic:Conn_02x04_Odd_Even
- added J5: RCA-JACK, LandBoards_Conns:RCA, symbol LandBoards_Conns:RCA-JACK
- added J6: FTDI, Connector_PinHeader_2.54mm:PinHeader_1x06_P2.54mm_Horizontal, symbol LandBoards_Cards:FTDI-Slave
- added P2: Conn_02x08_Odd_Even, Connector_PinHeader_2.54mm:PinHeader_2x08_P2.54mm_Vertical, symbol Connector_Generic:Conn_02x08_Odd_Even
- added P4: Conn_01x08, Connector_PinHeader_2.54mm:PinHeader_1x08_P2.54mm_Vertical, symbol Connector_Generic:Conn_01x08
- added U3: TXS0104, Package_SO:SOIC-14_3.9x8.7mm_P1.27mm, symbol LandBoards_Semis:TXS0104
- C7: footprint (none) -> Capacitor_SMD:C_0805_2012Metric_Pad1.15x1.40mm_HandSolder
- J2: footprint Pin_Headers:Pin_Header_Straight_1x06_Pitch2.54mm -> Connector_PinHeader_2.54mm:PinHeader_1x06_P2.54mm_Horizontal
- J3, J4: footprint (none) -> LandBoards_Conns:Connector_Mini-DIN_Female_6Pin_2rows
- P3: footprint (none) -> LandBoards_Conns:DB_15F-VGA-fixed
Connections:
- net labels added: ESP3V, FTDI5V0, FTDI5V2, GPXX, GPYY, RX2
- net labels removed: FTDI5V, GP12, GP15, GP2, GP5, RX1, STM_SCL, STM_SDA
- wire segments 246 -> 209
Other:
- note removed: "MISO"
- note removed: "MOSI"
- note removed: "SCK"
- note removed: "SPI BUS"
- moved on the sheet: C1, C6, C7, F1, J1, J15, J2, J3, J4, R11, R12

Commit message: Silkscreen tweeks
Parts:
- C1, C2, C4, C5, C6: footprint Capacitors_SMD:C_0805_HandSoldering -> Capacitor_SMD:C_0805_2012Metric_Pad1.15x1.40mm_HandSolder
- C3: footprint Capacitors_SMD:C_1206_HandSoldering -> Capacitor_SMD:C_1206_3216Metric_Pad1.42x1.75mm_HandSolder
- C7: footprint Capacitor_SMD:C_0805_2012Metric_Pad1.15x1.40mm_HandSolder -> Capacitor_SMD:C_1210_3225Metric_Pad1.42x2.65mm_HandSolder
Connections:
- net labels added: GP16, GP17
- net labels removed: GPXX, GPYY
Changed lines of the file:
@@
 F 0 "C3" H 4315 2491 50  0000 L CNN
 F 1 "10uF" H 4315 2400 50  0000 L CNN
-F 2 "Capacitors_SMD:C_1206_HandSoldering" H 3950 2150 30  0000 L CNN
+F 2 "Capacitor_SMD:C_1206_3216Metric_Pad1.42x1.75mm_HandSolder" H 3950 2150 30  0000 L CNN
 F 3 "~" H 4200 2400 50  0001 C CNN
 	1    4200 2400
@@
 F 0 "C2" H 3865 2491 50  0000 L CNN
 F 1 "0.1uF" H 3865 2400 50  0000 L CNN
-F 2 "Capacitors_SMD:C_0805_HandSoldering" H 3500 1950 30  0000 L CNN
+F 2 "Capacitor_SMD:C_0805_2012Metric_Pad1.15x1.40mm_HandSolder" H 3500 1950 30  0000 L CNN
 F 3 "~" H 3750 2400 50  0001 C CNN
 	1    3750 2400
@@
 F 0 "C4" H 10865 9191 50  0000 L CNN
 F 1 "0.1uF" H 10865 9100 50  0000 L CNN
-F 2 "Capacitors_SMD:C_0805_HandSoldering" H 10400 8850 30  0000 L CNN
+F 2 "Capacitor_SMD:C_0805_2012Metric_Pad1.15x1.40mm_HandSolder" H 10150 8600 30  0000 L CNN
 F 3 "~" H 10750 9100 50  0001 C CNN
 	1    10750 9100
@@
 F 0 "C5" H 11315 9191 50  0000 L CNN
 F 1 "0.1uF" H 11315 9100 50  0000 L CNN
-F 2 "Capacitors_SMD:C_0805_HandSoldering" H 10850 8850 30  0000 L CNN
+F 2 "Capacitor_SMD:C_0805_2012Metric_Pad1.15x1.40mm_HandSolder" H 10850 8850 30  0000 L CNN
 F 3 "~" H 11200 9100 50  0001 C CNN
 	1    11200 9100
@@
 F 0 "C6" H 2215 2991 50  0000 L CNN
 F 1 "0.1uF" H 2215 2900 50  0000 L CNN
-F 2 "Capacitors_SMD:C_0805_HandSoldering" H 1750 2650 30  0000 L CNN
+F 2 "Capacitor_SMD:C_0805_2012Metric_Pad1.15x1.40mm_HandSolder" H 1750 2650 30  0000 L CNN
 F 3 "~" H 2100 2900 50  0001 C CNN
 	1    2100 2900
@@
 F 0 "C1" H 9015 6591 50  0000 L CNN
 F 1 "0.1uF" H 9015 6500 50  0000 L CNN
-F 2 "Capacitors_SMD:C_0805_HandSoldering" H 8600 5750 30  0000 L CNN
+F 2 "Capacitor_SMD:C_0805_2012Metric_Pad1.15x1.40mm_HandSolder" H 8600 5750 30  0000 L CNN
 F 3 "~" H 8900 6500 50  0001 C CNN
 	1    8900 6500
@@
 F 0 "C7" V 10102 6150 50  0000 C CNN
 F 1 "CP1" V 10011 6150 50  0000 C CNN
-F 2 "Capacitor_SMD:C_0805_2012Metric_Pad1.15x1.40mm_HandSolder" H 9850 6150 50  0001 C CNN
+F 2 "Capacitor_SMD:C_1210_3225Metric_Pad1.42x2.65mm_HandSolder" H 9850 6150 50  0001 C CNN
 F 3 "~" H 9850 6150 50  0001 C CNN
 	1    9850 6150
@@
 Text Label 9800 1250 0    50   ~ 0
 GP14
-Text Label 9800 1450 0    50   ~ 0
+Text Label 9800 1550 0    50   ~ 0
 GP35
-Text Label 9800 1550 0    50   ~ 0
+Text Label 9800 1650 0    50   ~ 0
 GP34
 Text Label 7700 4000 0    50   ~ 0
-GPXX
+GP16
 Text Label 9800 1350 0    50   ~ 0
-GPXX
-Text Label 9800 1650 0    50   ~ 0
+GP16
+Text Label 9800 1750 0    50   ~ 0
 VN
-Text Label 9800 1750 0    50   ~ 0
+Text Label 9800 1850 0    50   ~ 0
 VP
-Text Label 9800 1850 0    50   ~ 0
-EN
+Text Label 9800 1450 0    50   ~ 0
+GP17
 $Comp
 L Connector_Generic:Conn_02x08_Odd_Even P2
@@
 	9600 1350 10300 1350
 Wire Wire Line
+	9600 1550 10300 1550
+Wire Wire Line
+	9600 1650 10300 1650
+Wire Wire Line
+	9600 1750 10300 1750
+Wire Wire Line
+	9600 1850 10300 1850
+Wire Wire Line
 	9600 1450 10300 1450
-Wire Wire Line
-	9600 1550 10300 1550
-Wire Wire Line
-	9600 1650 10300 1650
-Wire Wire Line
-	9600 1750 10300 1750
-Wire Wire Line
-	9600 1850 10300 1850
 $Comp
 L power:GND #PWR0104
@@
 TX2
 Text Label 7700 4100 0    50   ~ 0
-GPYY
+GP17
 $EndSCHEMATC

Commit message: Print schematics
Parts:
- added R10, R13, R14, R7, R8, R9: 470, Resistor_SMD:R_0805_2012Metric_Pad1.15x1.40mm_HandSolder, symbol Device:R
- R1: value 470 -> 1K
Connections:
- wire segments 209 -> 222
Other:
- moved on the sheet: J3, J4, P3, R1, R2, R3, R4, R5, R6, U3
