File: I2C Cards/I2C-RPT-08/I2C-RPT-08.sch (KiCad schematic (older format))
At the start: 46 parts, among them J1 CONN_01X04, J2 CONN_02X04, J3 CONN_02X04, J4 CONN_02X04, J5 CONN_02X04, U1 PCA9548A

Commit message: I2C Repeater Card
Connections:
- net labels added: A0, A1, A2
Changed lines of the file:
@@
 	1    0    0    -1
 $EndComp
+Text Label 2150 4050 0    60   ~ 0
+A0
+Text Label 2150 3950 0    60   ~ 0
+A1
+Text Label 2150 3850 0    60   ~ 0
+A2
 $EndSCHEMATC

Commit message: Moving stuff around
Parts:
- C1, C2: symbol C -> Device:C
- COUP?1: symbol COUPON -> I2C-RPT-08-rescue:COUPON
- FID1, FID2: symbol ADAFRUIT_FIDUCIAL -> I2C-RPT-08-rescue:ADAFRUIT_FIDUCIAL
- H1, H2, H3, H4, H5, H6, H7, H8: symbol CONN_01X02 -> I2C-RPT-08-rescue:CONN_01X02
- H9: symbol CONN_02X03 -> I2C-RPT-08-rescue:CONN_02X03
- J1: symbol CONN_01X04 -> I2C-RPT-08-rescue:CONN_01X04
- J2, J3, J4, J5: symbol CONN_02X04 -> I2C-RPT-08-rescue:CONN_02X04
- MTG1, MTG2, MTG3, MTG4: symbol MTG_HOLE -> I2C-RPT-08-rescue:MTG_HOLE
- R1, R10, R11, R12, R13, R14, R15, R16, R17, R18, R19, R2, R20, R21, R22, R3, R4, R5, R6, R7, R8, R9: symbol R -> Device:R
- U1: symbol PCA9548A -> I2C-RPT-08-rescue:PCA9548A
Connections:
- wire segments 153 -> 189
