File: HamRadio/Colpitts_XTAL_Osc/CP-OSC.kicad_pcb (KiCad board)
At the start: 2 copper layers, 24.8 x 31.1 mm, 16 parts, among them J1 BNC, J2 Conn_01x06, J3 DCJ0202, P1 SMA, Q1 2N3904, Q2 2N3904

Commit message: Cards
Parts:
- C3: value 100pF -> 10nF
- P1: footprint LandBoards_Conns:SMA_EDGE -> Connector_Coaxial:SMA_Samtec_SMA-J-P-H-ST-EM1_EdgeMount
- moved P1 1.14 mm to (110.4, 78.8)
- moved J1 0.13 mm to (99.1, 78.8)
Connections:
- J2 pad 1: Net-(C1-Pad2) -> Net-(C1-Pad1)
- R1 pad 1: Net-(C1-Pad2) -> Net-(C1-Pad1)
- R2 pad 2: Net-(C1-Pad2) -> Net-(C1-Pad1)
Routing:
- net Net-(C1-Pad1): track 5.37 -> 25.0 mm, vias 0 -> 1
- net Net-(C1-Pad2): track 22.8 -> 12.4 mm
- net Net-(C3-Pad1): track 16.6 -> 18.1 mm
Other:
- rule pad_to_mask_clearance: 0.254 -> 0
- board text added: "9- 12V"
- board text added: "CP-OSC"
- board text added: "REV 2"
- board text added: "RF"
- board text removed: "REV 1"
