File: BeagleBoneBlack Cards/BBB-GVS-4/BBB-Conn.kicad_sch (KiCad schematic)
At the start: 16 parts, among them J11 CONN_2, J25 CONN_3, U1 I2C-EEPROM

Commit message: Card stuff
Parts:
- removed C3: 104, Capacitors_SMD:C_0805_HandSoldering, symbol BBB-GVS-4-rescue:C-RESCUE-BBB-GVS-3
- renumbered C4 to C2, C2 to C3, F2 to F1, F1 to F2, R5 to R1, R4 to R2, R1 to R3, R3 to R4, R2 to R5
Connections:
- net F5VDD: now reaches F2.2, J25.2 (PM)
Changed lines of the file:
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@@
   (junction (at 213.36 60.96) (diameter 0) (color 0 0 0 0)
   )
-  (junction (at 66.04 62.23) (diameter 0) (color 0 0 0 0)
-  )
   (junction (at 194.31 77.47) (diameter 0) (color 0 0 0 0)
   )
@@
   (junction (at 213.36 38.1) (diameter 0) (color 0 0 0 0)
   )
-  (junction (at 66.04 44.45) (diameter 0) (color 0 0 0 0)
-  )
   (junction (at 217.17 66.04) (diameter 0) (color 0 0 0 0)
   )
@@
   (junction (at 222.25 68.58) (diameter 0) (color 0 0 0 0)
   )
-  (wire (pts (xy 62.23 44.45) (xy 66.04 44.45))
+  (wire (pts (xy 62.23 44.45) (xy 73.66 44.45))
     (stroke (width 0) (type default) (color 0 0 0 0))
   )
@@
     (stroke (width 0) (type default) (color 0 0 0 0))
   )
-  (wire (pts (xy 66.04 62.23) (xy 73.66 62.23))
+  (wire (pts (xy 58.42 62.23) (xy 73.66 62.23))
     (stroke (width 0) (type default) (color 0 0 0 0))
   )
@@
     (stroke (width 0) (type default) (color 0 0 0 0))
   )
-  (wire (pts (xy 58.42 62.23) (xy 66.04 62.23))
-    (stroke (width 0) (type default) (color 0 0 0 0))
-  )
   (wire (pts (xy 194.31 77.47) (xy 209.55 77.47))
     (stroke (width 0) (type default) (color 0 0 0 0))
@@
     (stroke (width 0) (type default) (color 0 0 0 0))
   )
-  (wire (pts (xy 66.04 62.23) (xy 66.04 58.42))
-    (stroke (width 0) (type default) (color 0 0 0 0))
-  )
   (wire (pts (xy 156.21 38.1) (xy 173.99 38.1))
     (stroke (width 0) (type default) (color 0 0 0 0))
@@
     (stroke (width 0) (type default) (color 0 0 0 0))
   )
-  (wire (pts (xy 66.04 44.45) (xy 73.66 44.45))
-    (stroke (width 0) (type default) (color 0 0 0 0))
-  )
   (wire (pts (xy 222.25 68.58) (xy 234.95 68.58))
     (stroke (width 0) (type default) (color 0 0 0 0))
@@
     (stroke (width 0) (type default) (color 0 0 0 0))
   )
-  (wire (pts (xy 66.04 48.26) (xy 66.04 44.45))
-    (stroke (width 0) (type default) (color 0 0 0 0))
-  )
   (wire (pts (xy 173.99 63.5) (xy 173.99 38.1))
     (stroke (width 0) (type default) (color 0 0 0 0))
@@
   )
   (label "GND" (at 50.8 62.23 0)
+    (effects (font (size 1.524 1.524)) (justify left bottom))
+  )
+  (label "F5VDD" (at 77.47 81.28 0)
     (effects (font (size 1.524 1.524)) (justify left bottom))
   )
@@
   (symbol (lib_id "BBB-GVS-4-rescue:R-RESCUE-BBB-GVS-3") (at 217.17 46.99 0) (unit 1)
     (in_bom yes) (on_board yes)
-    (property "Reference" "R4" (id 0) (at 219.202 46.99 90))
+    (property "Reference" "R2" (id 0) (at 219.202 46.99 90))
     (property "Value" "5.6K" (id 1) (at 217.17 46.99 90))
     (property "Footprint" "Resistor_SMD:R_0805_2012Metric_Pad1.20x1.40mm_HandSolder" (id 2) (at 217.17 26.67 0)
@@
   (symbol (lib_id "BBB-GVS-4-rescue:R-RESCUE-BBB-GVS-3") (at 222.25 46.99 0) (unit 1)
     (in_bom yes) (on_board yes)
-    (property "Reference" "R5" (id 0) (at 224.282 46.99 90))
+    (property "Reference" "R1" (id 0) (at 224.282 46.99 90))
     (property "Value" "5.6K" (id 1) (at 222.25 46.99 90))
     (property "Footprint" "Resistor_SMD:R_0805_2012Metric_Pad1.20x1.40mm_HandSolder" (id 2) (at 222.25 30.48 0)
@@
     (pin "2")
   )
-  (symbol (lib_id "BBB-GVS-4-rescue:C-RESCUE-BBB-GVS-3") (at 156.21 48.26 0)
+  (symbol (lib_id "BBB-GVS-4-rescue:C-RESCUE-BBB-GVS-3") (at 156.21 48.26 0) (unit 1)
     (in_bom yes) (on_board yes)
     (property "Reference" "C1" (id 0) (at 157.48 45.72 0)
@@
   (symbol (lib_id "BBB-GVS-4-rescue:FUSE") (at 66.04 81.28 0) (unit 1)
     (in_bom yes) (on_board yes)
-    (property "Reference" "F1" (id 0) (at 68.58 80.01 0)
+    (property "Reference" "F2" (id 0) (at 68.58 80.01 0)
       (effects (font (size 1.016 1.016)))
     )
@@
     (pin "2")
   )
-  (symbol (lib_id "BBB-GVS-4-rescue:C-RESCUE-BBB-GVS-3") (at 46.99 53.34 0)
-    (in_bom yes) (on_board yes)
-    (property "Reference" "C2" (id 0) (at 46.99 50.8 0)
+  (symbol (lib_id "BBB-GVS-4-rescue:C-RESCUE-BBB-GVS-3") (at 46.99 53.34 0) (unit 1)
+    (in_bom yes) (on_board yes)
+    (property "Reference" "C3" (id 0) (at 46.99 50.8 0)
       (effects (font (size 1.016 1.016)) (justify left))
     )
@@
     (pin "2")
   )
-  (symbol (lib_id "BBB-GVS-4-rescue:C-RESCUE-BBB-GVS-3") (at 66.04 53.34 0)
-    (in_bom yes) (on_board yes)
-    (property "Reference" "C3" (id 0) (at 66.04 50.8 0)
-      (effects (font (size 1.016 1.016)) (justify left))
-    )
-    (property "Value" "104" (id 1) (at 66.1924 55.499 0)
-      (effects (font (size 1.016 1.016)) (justify left))
-    )
-    (property "Footprint" "Capacitors_SMD:C_0805_HandSoldering" (id 2) (at 67.31 58.42 0)
-      (effects (font (size 0.762 0.762)))
-    )
-    (property "Datasheet" "~" (id 3) (at 66.04 53.34 0)
-      (effects (font (size 1.524 1.524)))
-    )
-    (pin "1")
-    (pin "2")
-  )
-  (symbol (lib_id "BBB-GVS-4-rescue:C-RESCUE-BBB-GVS-3") (at 73.66 53.34 0)
-    (in_bom yes) (on_board yes)
-    (property "Reference" "C4" (id 0) (at 73.66 50.8 0)
+  (symbol (lib_id "BBB-GVS-4-rescue:C-RESCUE-BBB-GVS-3") (at 73.66 53.34 0) (unit 1)
+    (in_bom yes) (on_board yes)
+    (property "Reference" "C2" (id 0) (at 73.66 50.8 0)
       (effects (font (size 1.016 1.016)) (justify left))
     )
@@
   (symbol (lib_id "BBB-GVS-4-rescue:R-RESCUE-BBB-GVS-3") (at 90.17 39.37 0) (unit 1)
     (in_bom yes) (on_board yes)
-    (property "Reference" "R2" (id 0) (at 92.202 39.37 90)
+    (property "Reference" "R5" (id 0) (at 92.202 39.37 90)
       (effects (font (size 1.016 1.016)))
     )
@@
   (symbol (lib_id "BBB-GVS-4-rescue:FUSE") (at 67.31 106.68 0) (unit 1)
     (in_bom yes) (on_board yes)
-    (property "Reference" "F2" (id 0) (at 69.85 105.41 0)
+    (property "Reference" "F1" (id 0) (at 69.85 105.41 0)
       (effects (font (size 1.016 1.016)))
     )
@@
   (symbol (lib_id "BBB-GVS-4-rescue:R-RESCUE-BBB-GVS-3") (at 58.42 39.37 0) (unit 1)
     (in_bom yes) (on_board yes)
-    (property "Reference" "R1" (id 0) (at 60.452 39.37 90)
+    (property "Reference" "R3" (id 0) (at 60.452 39.37 90)
       (effects (font (size 1.016 1.016)))
     )
@@
   (symbol (lib_id "BBB-GVS-4-rescue:R-RESCUE-BBB-GVS-3") (at 213.36 46.99 0) (unit 1)
     (in_bom yes) (on_board yes)
-    (property "Reference" "R3" (id 0) (at 215.392 46.99 90))
+    (property "Reference" "R4" (id 0) (at 215.392 46.99 90))
     (property "Value" "5.6K" (id 1) (at 213.36 46.99 90))
     (property "Footprint" "Resistor_SMD:R_0805_2012Metric_Pad1.20x1.40mm_HandSolder" (id 2) (at 213.36 34.29 0)
