File: I2C Cards/SWLEDX8/SWLEDX8.kicad_sch (KiCad schematic)
At the start: 38 parts, among them P1 CONN_02X10, SW1 Switch_SPDT_x2, SW2 Switch_SPDT_x2, SW3 Switch_SPDT_x2, SW4 Switch_SPDT_x2, SW5 Switch_SPDT_x2, SW6 Switch_SPDT_x2, SW7 Switch_SPDT_x2, SW8 Switch_SPDT_x2

Commit message: More card work
Parts:
- D0: renamed from D1; footprint LEDs:LED_D5.0mm -> LED_THT:LED_D5.0mm
- D1: renamed from D2; footprint LEDs:LED_D5.0mm -> LED_THT:LED_D5.0mm
- D2: renamed from D3; footprint LEDs:LED_D5.0mm -> LED_THT:LED_D5.0mm
- D3: renamed from D4; footprint LEDs:LED_D5.0mm -> LED_THT:LED_D5.0mm
- D4: renamed from D5; footprint LEDs:LED_D5.0mm -> LED_THT:LED_D5.0mm
- D5: renamed from D6; footprint LEDs:LED_D5.0mm -> LED_THT:LED_D5.0mm
- D6: renamed from D7; footprint LEDs:LED_D5.0mm -> LED_THT:LED_D5.0mm
- D7: renamed from D8; footprint LEDs:LED_D5.0mm -> LED_THT:LED_D5.0mm
- P1: footprint Pin_Headers:Pin_Header_Angled_2x10_Pitch2.54mm -> Connector_PinHeader_2.54mm:PinHeader_2x10_P2.54mm_Vertical
- SW0: renamed from SW1; value Switch_SPDT_x2 -> SS12D00G3; footprint Pin_Headers:Pin_Header_Straight_1x03_Pitch2.54mm -> Connector_PinHeader_2.54mm:PinHeader_1x03_P2.54mm_Vertical; symbol SWLEDX8-rescue:Switch_SPDT_x2 -> Switch:SW_SPDT
- SW1: renamed from SW2; value Switch_SPDT_x2 -> SS12D00G3; footprint Pin_Headers:Pin_Header_Straight_1x03_Pitch2.54mm -> Connector_PinHeader_2.54mm:PinHeader_1x03_P2.54mm_Vertical; symbol SWLEDX8-rescue:Switch_SPDT_x2 -> Switch:SW_SPDT
- SW2: renamed from SW3; value Switch_SPDT_x2 -> SS12D00G3; footprint Pin_Headers:Pin_Header_Straight_1x03_Pitch2.54mm -> Connector_PinHeader_2.54mm:PinHeader_1x03_P2.54mm_Vertical; symbol SWLEDX8-rescue:Switch_SPDT_x2 -> Switch:SW_SPDT
- SW3: renamed from SW4; value Switch_SPDT_x2 -> SS12D00G3; footprint Pin_Headers:Pin_Header_Straight_1x03_Pitch2.54mm -> Connector_PinHeader_2.54mm:PinHeader_1x03_P2.54mm_Vertical; symbol SWLEDX8-rescue:Switch_SPDT_x2 -> Switch:SW_SPDT
- SW4: renamed from SW5; value Switch_SPDT_x2 -> SS12D00G3; footprint Pin_Headers:Pin_Header_Straight_1x03_Pitch2.54mm -> Connector_PinHeader_2.54mm:PinHeader_1x03_P2.54mm_Vertical; symbol SWLEDX8-rescue:Switch_SPDT_x2 -> Switch:SW_SPDT
- SW5: renamed from SW6; value Switch_SPDT_x2 -> SS12D00G3; footprint Pin_Headers:Pin_Header_Straight_1x03_Pitch2.54mm -> Connector_PinHeader_2.54mm:PinHeader_1x03_P2.54mm_Vertical; symbol SWLEDX8-rescue:Switch_SPDT_x2 -> Switch:SW_SPDT
- SW6: renamed from SW7; value Switch_SPDT_x2 -> SS12D00G3; footprint Pin_Headers:Pin_Header_Straight_1x03_Pitch2.54mm -> Connector_PinHeader_2.54mm:PinHeader_1x03_P2.54mm_Vertical; symbol SWLEDX8-rescue:Switch_SPDT_x2 -> Switch:SW_SPDT
- SW7: renamed from SW8; value Switch_SPDT_x2 -> SS12D00G3; footprint Pin_Headers:Pin_Header_Straight_1x03_Pitch2.54mm -> Connector_PinHeader_2.54mm:PinHeader_1x03_P2.54mm_Vertical; symbol SWLEDX8-rescue:Switch_SPDT_x2 -> Switch:SW_SPDT
Connections:
- net GND: now also P1.1 (P1), P1.2 (P2); no longer P1.19 (P19), P1.20 (P20)
- net VCC: now also P1.19 (P19), P1.20 (P20); no longer P1.1 (P1)
Other:
- moved on the sheet: R1, R2, R3, R4, R5, R6, R7, R8
