File: Raspberry Pi Cards/PiPicoMite01/Rev1/PiPicoMite01.kicad_sch (KiCad schematic)
At the start: 46 parts, among them J1 Conn_01x02, J10 CONN, DB15HD, BLUE (VGA), J2 USB-B, J3 Socket, Female. 1x20, J4 Header, Vert, 2x3, J5 Socket, Female. 1x20, J6 Header, Vert, 2x8, J7 AudioJack3, J8 PS2_DIN6, J9 Header, Vert, 2x10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

Commit message: More card work
Changed lines of the file:
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@@
   )
   (symbol (lib_id "Connector_Generic:Conn_02x08_Odd_Even") (at 133.35 237.49 0) (unit 1)
-    (in_bom yes) (on_board yes) (fields_autoplaced)
+    (in_bom yes) (on_board yes)
     (property "Reference" "J6" (id 0) (at 134.62 224.6335 0))
     (property "Value" "Header, Vert, 2x8" (id 1) (at 134.62 227.4086 0))
-    (property "Footprint" "Connector_PinSocket_2.54mm:PinSocket_2x08_P2.54mm_Vertical" (id 2) (at 133.35 237.49 0)
-      (effects (font (size 1.27 1.27)) hide)
+    (property "Footprint" "Connector_PinSocket_2.54mm:PinSocket_2x08_P2.54mm_Vertical" (id 2) (at 133.35 255.27 0)
+      (effects (font (size 0.762 0.762)))
     )
     (property "Datasheet" "~" (id 3) (at 133.35 237.49 0)
