File: Arduino Cards/MyMenu/MyMenu.kicad_pcb (KiCad board)
At the start: 2 copper layers, 49 x 49 mm, 43 parts, among them P1 CONN_4, P2 CONN_5, P3 CONN_4, SW1 SW_PUSH_OMRON, SW2 SW_PUSH_OMRON, SW3 SW_PUSH_OMRON, SW4 SW_PUSH_OMRON, SW5 SW_PUSH_OMRON, U1 MCP23008SO

Commit message: MyMenu
Parts:
- removed ADDR, TESTED: VAL**, DougsNewMods:TEST_BLK-REAR
- added 0x2_: VAL**, LandBoards_Marking:TEST_BLK-REAR, F.Cu at (13.0, 45.5)
- R13, R15, R17: value OPEN -> DNP
Connections:
- net Net-(P2-Pad5) renamed /INT*
- MTG1 pad 1: (no net) -> unconnected-(MTG1-Pad1)
- MTG2 pad 1: (no net) -> unconnected-(MTG2-Pad1)
- MTG3 pad 1: (no net) -> unconnected-(MTG3-Pad1)
- MTG4 pad 1: (no net) -> unconnected-(MTG4-Pad1)
- MTG5 pad 1: (no net) -> unconnected-(MTG5-Pad1)
- MTG6 pad 1: (no net) -> unconnected-(MTG6-Pad1)
- MTG7 pad 1: (no net) -> unconnected-(MTG7-Pad1)
- MTG8 pad 1: (no net) -> unconnected-(MTG8-Pad1)
Routing:
- net /SDA: track 36.6 -> 34.3 mm
- net Net-(R8-Pad2): track 41.8 -> 40.3 mm
- net /A2: track 16.4 -> 15.2 mm
- net /A0: track 15.9 -> 14.8 mm
- net Net-(R4-Pad1): track 18.9 -> 17.8 mm
- net /SCL: track 36.5 -> 35.8 mm
- net Net-(R9-Pad2): track 24.6 -> 24.0 mm
Other:
- net class Default removed
- rule pad_to_mask_clearance: 0.2 -> 0
- board text added: "1=G"
- board text added: "1=V"
- board text added: "2=G"
- board text added: "2=V"
- board text removed: "1G"
- board text removed: "1V"
- board text removed: "2G"
- board text removed: "2V"
- board text removed: "x2"

Commit message: KiCad Temptates and cards
Parts:
- removed 0x2_: VAL**, LandBoards_Marking:TEST_BLK-REAR
- removed R10, R11, R20, R21: 0/OP, Resistors_SMD:R_0805_HandSoldering
- removed R14, R16, R18: 0, Resistors_SMD:R_0805_HandSoldering
- added ADR=: COUPON, LandBoards_Marking:TEST_BLK-REAR, B.Cu at (45.5, 37.1)
- added J1: Conn_02x03_Odd_Even, Connector_PinHeader_2.54mm:PinHeader_2x03_P2.54mm_Vertical, F.Cu at (34.5, 6.87)
- added J2: Conn_02x03_Odd_Even, Connector_PinHeader_2.54mm:PinHeader_2x03_P2.54mm_Vertical, F.Cu at (38.9, 17.0)
- added TESTED: COUPON, LandBoards_Marking:TEST_BLK-REAR, B.Cu at (11.9, 45.2)
- moved R13 8.56 mm to (32.8, 17.3), turned to -90 degrees
- moved R15 7.13 mm to (41.9, 27.2), turned to 90 degrees
- moved R12 4.15 mm to (45.3, 13.5)
- moved R17 3.23 mm to (39.1, 27.2), turned to 90 degrees
Routing:
- net Net-(R12-Pad2): track 12.0 -> 17.0 mm
- net /VCC: track 0.55 -> 5.39 mm
- net /A0: track 14.8 -> 10.1 mm
- net Net-(J1-Pad4): track 10.1 -> 14.4 mm, vias 1 -> 0
- net /A1: track 14.2 -> 17.0 mm
- net Net-(J1-Pad3): track 16.8 -> 14.9 mm, vias 1 -> 0
- net /A2: track 15.2 -> 13.7 mm
- net /GND: track 5.20 -> 4.32 mm, vias 4 -> 1
Other:
- board text added: "1=G,2=V"
- board text added: "1=V,2-G"
- board text added: "A0 A1 A2"
- board text added: "IN=0 OUT=1"
- board text added: "REV 5"
- board text removed: "1 0"
- board text removed: "1=G"
- board text removed: "1=V"
- board text removed: "2=G"
- board text removed: "2=V"
- board text removed: "A0"
- board text removed: "A1"
- board text removed: "A2"
- board text removed: "Rev X4"

Commit message: MyMenu_Rev5
Other:
- board text added: "I C D V G"
- board text removed: "I"
Changed lines of the file:
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@@
   (gr_line (start 14.224 13.716) (end 14.478 13.716) (layer "F.SilkS") (width 0.15))
   (gr_line (start 8.89 7.366) (end 8.89 5.334) (layer "F.SilkS") (width 0.15))
+  (gr_line (start 7.14 7.49) (end 15.61 7.51) (layer "F.SilkS") (width 0.15))
   (gr_line (start 8.89 9.906) (end 8.89 13.716) (layer "F.SilkS") (width 0.15))
   (gr_line (start 8.89 13.716) (end 14.224 13.716) (layer "F.SilkS") (width 0.15))
@@
     (effects (font (size 1.27 1.27) (thickness 0.3)))
   )
-  (gr_text "I" (at 18.03 9.168) (layer "F.SilkS")
+  (gr_text "I C D V G" (at 23.36 4.38) (layer "F.SilkS")
     (effects (font (size 1.5 1.5) (thickness 0.3)))
   )
@@
     (pts (xy 28.194 0) (xy 28.194 6.604))
     (height -22.733)
-    (gr_text "0.2600 in" (at 49.127 3.302 90) (layer "Dwgs.User")
+    (gr_text "0.26 in" (at 53.22 5.17 90) (layer "Dwgs.User")
       (effects (font (size 1.5 1.5) (thickness 0.3)))
     )
-    (format (units 0) (units_format 1) (precision 4))
-    (style (thickness 0.3) (arrow_length 1.27) (text_position_mode 0) (extension_height 0.58642) (extension_offset 0) keep_text_aligned)
+    (format (units 0) (units_format 1) (precision 2))
+    (style (thickness 0.3) (arrow_length 1.27) (text_position_mode 2) (extension_height 0.58642) (extension_offset 0) keep_text_aligned)
   )
   (dimension (type aligned) (layer "Dwgs.User")
     (pts (xy 0 6.604) (xy 28.194 6.604))
     (height -9.017)
-    (gr_text "1.1100 in" (at 14.097 -4.213) (layer "Dwgs.User")
+    (gr_text "1.11 in" (at 14.097 -2.413) (layer "Dwgs.User")
       (effects (font (size 1.5 1.5) (thickness 0.3)))
     )
-    (format (units 0) (units_format 1) (precision 4))
-    (style (thickness 0.3) (arrow_length 1.27) (text_position_mode 0) (extension_height 0.58642) (extension_offset 0) keep_text_aligned)
+    (format (units 0) (units_format 1) (precision 2))
+    (style (thickness 0.3) (arrow_length 1.27) (text_position_mode 1) (extension_height 0.58642) (extension_offset 0) keep_text_aligned)
   )
   (dimension (type aligned) (layer "Dwgs.User")
     (pts (xy 45 49) (xy 45 0))
     (height 11)
-    (gr_text "49.0000 mm" (at 54.2 24.5 90) (layer "Dwgs.User")
+    (gr_text "49.0 mm" (at 56 24.5 90) (layer "Dwgs.User")
       (effects (font (size 1.5 1.5) (thickness 0.3)))
     )
-    (format (units 2) (units_format 1) (precision 4))
-    (style (thickness 0.3) (arrow_length 1.27) (text_position_mode 0) (extension_height 0.58642) (extension_offset 0) keep_text_aligned)
+    (format (units 2) (units_format 1) (precision 1))
+    (style (thickness 0.3) (arrow_length 1.27) (text_position_mode 1) (extension_height 0.58642) (extension_offset 0) keep_text_aligned)
+  )
+  (dimension (type aligned) (layer "Dwgs.User")
+    (pts (xy 0 4) (xy 49 4))
+    (height -11)
+    (gr_text "49.0 mm" (at 24.5 -7) (layer "Dwgs.User")
+      (effects (font (size 1.5 1.5) (thickness 0.3)))
+    )
+    (format (units 2) (units_format 1) (precision 1))
+    (style (thickness 0.3) (arrow_length 1.27) (text_position_mode 1) (extension_height 0.58642) (extension_offset 0.5) keep_text_aligned)
   )
   (dimension (type aligned) (layer "Dwgs.User")
     (pts (xy 49.022 6.604) (xy 28.194 6.604))
     (height 9.144)
-    (gr_text "0.8200 in" (at 38.608 -4.34) (layer "Dwgs.User")
+    (gr_text "0.82 in" (at 38.608 -2.54) (layer "Dwgs.User")
       (effects (font (size 1.5 1.5) (thickness 0.3)))
     )
-    (format (units 0) (units_format 1) (precision 4))
-    (style (thickness 0.3) (arrow_length 1.27) (text_position_mode 0) (extension_height 0.58642) (extension_offset 0) keep_text_aligned)
+    (format (units 0) (units_format 1) (precision 2))
+    (style (thickness 0.3) (arrow_length 1.27) (text_position_mode 1) (extension_height 0.58642) (extension_offset 0) keep_text_aligned)
   )
   (segment (start 34.335489 17.052511) (end 32.766 18.622) (width 0.254) (layer "F.Cu") (net 1))
