File: Raspberry Pi Cards/PicoVGA/PicoVGA.kicad_sch (KiCad schematic)
At the start: 30 parts, among them J1 Conn_01x20, J2 AudioJack3, J3 Conn_01x20, J4 USB-B, J5 M09H, P1 VGA, U1 RPi-PICO

Commit message: PicoVGA build
Parts:
- J5: renamed from BRD?; footprint (none) -> Connector_PinHeader_2.54mm:PinHeader_1x12_P2.54mm_Vertical
- renumbered J5 to J6
Connections:
- net +3V3: now also J5.1 (+V), J5.2 (+V)
- net GND: now also J5.11 (GD)
- net GP16: now also J5.10 (UL); no longer J5.4 (UR)
- net GP17: now also J5.9 (RT); no longer J5.6 (CF)
- net GP18: now also J5.8 (FR); no longer J5.5 (DN)
- net GP21: now also J5.6 (CF); no longer J5.9 (RT)
- net GP22: now also J5.5 (DN)
- net GP26: now also J5.4 (UR)
- net GP27: now also J5.3 (UP)
- net RED: now reaches P1.1 (P1), R6.1, R7.1, R8.1
- net CSY: now reaches P1.13 (P13), R9.1
- net GRN: now reaches P1.2 (P2), R3.1, R4.1, R5.1
- net BLU: now reaches P1.3 (P3), R1.1, R2.1
Other:
- note added: "BLU"
- note added: "BRN"
- note added: "GRN"
- note added: "GRY"
- note added: "ORG"
- note added: "VIO"
- note added: "WHIT"
- note added: "YEL"
- title: PicoVGA -> PicoVGA01
- moved on the sheet: J5

Commit message: QTPy apps
Parts:
- added J7: Conn_01x02, Connector_PinHeader_2.54mm:PinHeader_1x02_P2.54mm_Vertical, symbol Connector_Generic:Conn_01x02
- J1, J3: value Conn_01x20 -> Hdr, Strt, 1x20
- J6: value M09H -> Conn, DB-9M
Connections:
- net +3V3: now also J7.1 (Pin_1), J7.2 (Pin_2)
Changed lines of the file:
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@@
   (junction (at 106.68 111.76) (diameter 0) (color 0 0 0 0)
+  )
+  (junction (at 156.21 26.67) (diameter 0) (color 0 0 0 0)
   )
   (junction (at 95.25 151.13) (diameter 0) (color 0 0 0 0)
@@
     (stroke (width 0) (type default) (color 0 0 0 0))
   )
+  (wire (pts (xy 160.02 26.67) (xy 156.21 26.67))
+    (stroke (width 0) (type default) (color 0 0 0 0))
+  )
+  (wire (pts (xy 156.21 26.67) (xy 156.21 22.86))
+    (stroke (width 0) (type default) (color 0 0 0 0))
+  )
   (wire (pts (xy 50.8 60.96) (xy 50.8 73.66))
     (stroke (width 0) (type default) (color 0 0 0 0))
@@
     (stroke (width 0) (type default) (color 0 0 0 0))
   )
+  (wire (pts (xy 156.21 29.21) (xy 156.21 26.67))
+    (stroke (width 0) (type default) (color 0 0 0 0))
+  )
   (wire (pts (xy 106.68 153.67) (xy 106.68 151.13))
     (stroke (width 0) (type default) (color 0 0 0 0))
@@
   )
   (wire (pts (xy 138.43 73.66) (xy 140.97 73.66))
+    (stroke (width 0) (type default) (color 0 0 0 0))
+  )
+  (wire (pts (xy 160.02 29.21) (xy 156.21 29.21))
     (stroke (width 0) (type default) (color 0 0 0 0))
   )
@@
       (effects (font (size 1.524 1.524)) (justify left))
     )
-    (property "Datasheet" "" (id 3) (at 237.49 83.82 0)
+    (property "Datasheet" "https://www.mouser.com/ProductDetail/587-634-015-274-906" (id 3) (at 237.49 83.82 0)
       (effects (font (size 1.524 1.524)))
     )
@@
       (effects (font (size 0.762 0.762)))
     )
-    (property "Datasheet" "https://www.mouser.com/datasheet/2/670/uj2_bh_th-1779177.pdf" (id 3) (at 62.23 165.1 0)
+    (property "Datasheet" "https://www.mouser.com/ProductDetail/490-UJ2-BH-1-TH" (id 3) (at 62.23 165.1 0)
       (effects (font (size 1.524 1.524)) hide)
     )
@@
     (pin "1")
     (pin "2")
+  )
+  (symbol (lib_id "power:+3.3V") (at 156.21 22.86 0) (unit 1)
+    (in_bom yes) (on_board yes) (fields_autoplaced)
+    (property "Reference" "#PWR0112" (id 0) (at 156.21 26.67 0)
+      (effects (font (size 1.27 1.27)) hide)
+    )
+    (property "Value" "+3.3V" (id 1) (at 156.21 19.2555 0))
+    (property "Footprint" "" (id 2) (at 156.21 22.86 0)
+      (effects (font (size 1.27 1.27)) hide)
+    )
+    (property "Datasheet" "" (id 3) (at 156.21 22.86 0)
+      (effects (font (size 1.27 1.27)) hide)
+    )
+    (pin "1")
   )
   (symbol (lib_id "LandBoards:COUPON") (at 100.33 195.58 0) (unit 1)
@@
       (effects (font (size 1.27 1.27)) (justify left))
     )
-    (property "Value" "Conn_01x20" (id 1) (at 139.7 81.28 0)
+    (property "Value" "Hdr, Strt, 1x20" (id 1) (at 139.7 81.28 0)
       (effects (font (size 1.27 1.27)) (justify left))
     )
@@
       (effects (font (size 0.762 0.762)))
     )
-    (property "Datasheet" "https://www.mouser.com/datasheet/2/345/1n5817-1n5819-24580.pdf" (id 3) (at 101.6 151.13 0)
+    (property "Datasheet" "https://www.mouser.com/ProductDetail/STMicroelectronics/1N5819?qs=G5AQjGfRJcKKUy9S%252BaTHRQ%3D%3D" (id 3) (at 101.6 151.13 0)
       (effects (font (size 1.27 1.27)) hide)
     )
@@
       (effects (font (size 1.27 1.27)) hide)
     )
-    (property "Datasheet" "DOCUMENTATION" (id 3) (at 91.44 83.82 0)
+    (property "Datasheet" "https://www.mouser.com/ProductDetail/Seeed-Studio/102110537?qs=pUKx8fyJudDPj27tABVsxg%3D%3D" (id 3) (at 91.44 83.82 0)
       (effects (font (size 1.27 1.27)) hide)
     )
@@
   (symbol (lib_id "con-subd:M09H") (at 209.55 154.94 0) (unit 1)
     (in_bom yes) (on_board yes)
-    (property "Reference" "J6" (id 0) (at 209.55 142.5702 0))
-    (property "Value" "M09H" (id 1) (at 209.55 144.8816 0))
+    (property "Reference" "J6" (id 0) (at 209.55 144.78 0))
+    (property "Value" "Conn, DB-9M" (id 1) (at 209.55 165.1 0))
     (property "Footprint" "Connector_Dsub:DSUB-9_Male_Horizontal_P2.77x2.84mm_EdgePinOffset4.94mm_Housed_MountingHolesOffset7.48mm" (id 2) (at 209.55 151.13 0)
       (effects (font (size 1.27 1.27)) hide)
     )
-    (property "Datasheet" "" (id 3) (at 209.55 154.94 0)
+    (property "Datasheet" "https://www.mouser.com/ProductDetail/649-D09P13B4PA00LF" (id 3) (at 209.55 154.94 0)
       (effects (font (size 1.27 1.27)) hide)
     )
@@
       (effects (font (size 1.27 1.27)) hide)
     )
-    (property "Datasheet" "https://www.mouser.com/datasheet/2/670/sj1_352xn-1779157.pdf" (id 3) (at 115.57 114.3 0)
+    (property "Datasheet" "https://www.mouser.com/ProductDetail/490-SJ1-3523N" (id 3) (at 115.57 114.3 0)
       (effects (font (size 1.27 1.27)) hide)
     )
@@
     (pin "2")
   )
+  (symbol (lib_id "Connector_Generic:Conn_01x02") (at 165.1 26.67 0) (unit 1)
+    (in_bom yes) (on_board yes) (fields_autoplaced)
+    (property "Reference" "J7" (id 0) (at 167.132 27.0315 0)
+      (effects (font (size 1.27 1.27)) (justify left))
+    )
+    (property "Value" "Conn_01x02" (id 1) (at 167.132 29.8066 0)
+      (effects (font (size 1.27 1.27)) (justify left))
+    )
+    (property "Footprint" "Connector_PinHeader_2.54mm:PinHeader_1x02_P2.54mm_Vertical" (id 2) (at 165.1 26.67 0)
+      (effects (font (size 1.27 1.27)) hide)
+    )
+    (property "Datasheet" "~" (id 3) (at 165.1 26.67 0)
+      (effects (font (size 1.27 1.27)) hide)
+    )
+    (pin "1")
+    (pin "2")
+  )
   (symbol (lib_id "Connector_Generic:Conn_01x20") (at 27.94 53.34 0) (mirror y) (unit 1)
     (in_bom yes) (on_board yes)
     (property "Reference" "J1" (id 0) (at 27.94 27.94 0))
-    (property "Value" "Conn_01x20" (id 1) (at 27.94 81.28 0))
+    (property "Value" "Hdr, Strt, 1x20" (id 1) (at 27.94 81.28 0))
     (property "Footprint" "Connector_PinHeader_2.54mm:PinHeader_1x20_P2.54mm_Vertical" (id 2) (at 31.75 91.44 0)
       (effects (font (size 0.762 0.762)))
@@
       (reference "#PWR0111") (unit 1) (value "+3.3V") (footprint "")
     )
+    (path "/25e43232-69b6-46a1-b860-f6300f04c1bb"
+      (reference "#PWR0112") (unit 1) (value "+3.3V") (footprint "")
+    )
     (path "/8f5abcb3-9b34-46ae-bc22-4a3fbd45051b"
       (reference "C1") (unit 1) (value "0.1uF") (footprint "Capacitor_THT:C_Rect_L4.0mm_W2.5mm_P2.50mm")
@@
     )
     (path "/e4f0b19b-5c3e-4326-b844-19ce566527d6"
-      (reference "J1") (unit 1) (value "Conn_01x20") (footprint "Connector_PinHeader_2.54mm:PinHeader_1x20_P2.54mm_Vertical")
+      (reference "J1") (unit 1) (value "Hdr, Strt, 1x20") (footprint "Connector_PinHeader_2.54mm:PinHeader_1x20_P2.54mm_Vertical")
     )
     (path "/a2e56043-99e0-49b8-a470-aacbbe828f84"
@@
     )
     (path "/89dc7f23-ac8d-4ccf-a836-107fd80333da"
-      (reference "J3") (unit 1) (value "Conn_01x20") (footprint "Connector_PinHeader_2.54mm:PinHeader_1x20_P2.54mm_Vertical")
+      (reference "J3") (unit 1) (value "Hdr, Strt, 1x20") (footprint "Connector_PinHeader_2.54mm:PinHeader_1x20_P2.54mm_Vertical")
     )
     (path "/02f5a918-cdd6-4f3a-ad29-2afaffaa3e50"
@@
     )
     (path "/98fc0f37-db71-4902-b35f-aa57517c9aa7"
-      (reference "J6") (unit 1) (value "M09H") (footprint "Connector_Dsub:DSUB-9_Male_Horizontal_P2.77x2.84mm_EdgePinOffset4.94mm_Housed_MountingHolesOffset7.48mm")
+      (reference "J6") (unit 1) (value "Conn, DB-9M") (footprint "Connector_Dsub:DSUB-9_Male_Horizontal_P2.77x2.84mm_EdgePinOffset4.94mm_Housed_MountingHolesOffset7.48mm")
+    )
+    (path "/e44bf172-fb48-4f04-ade0-21fe71f08b88"
+      (reference "J7") (unit 1) (value "Conn_01x02") (footprint "Connector_PinHeader_2.54mm:PinHeader_1x02_P2.54mm_Vertical")
     )
     (path "/00000000-0000-0000-0000-00005030f2a7"
