File: RetroCPUs/JoyPad/JoyPad.kicad_pcb (KiCad board)
At the start: 2 copper layers, 49 x 49 mm, 23 parts, among them J1 Conn_01x12, J2 M09H, SW1 SW_Push, SW2 SW_Push, SW3 SW_Push, SW4 SW_Push, SW5 SW_Push, SW6 SW_Push, SW7 SW_Push, SW8 SW_Push

Commit message: QTPy apps
Other:
- net class Default removed

Commit message: New cards order
Parts:
- J2: footprint Connector_Dsub:DSUB-9_Male_Horizontal_P2.77x2.84mm_EdgePinOffset4.94mm_Housed_MountingHolesOffset7.48mm -> Connector_Dsub:DSUB-9_Female_Horizontal_P2.77x2.84mm_EdgePinOffset4.94mm_Housed_MountingHolesOffset7.48mm
- R1, R2, R3, R4, R5, R6, R7, R8: moved to B.Cu
- moved J2 11.2 mm to (19.2, 7.77)
- moved R1 4.90 mm to (15.7, 34.3), turned to 0 degrees
- moved R2 4.90 mm to (24.6, 34.3), turned to 0 degrees
- moved R4 4.79 mm to (24.7, 43.7), turned to 0 degrees
- moved R6 4.79 mm to (43.4, 18.0), turned to 180 degrees
- moved R5 4.78 mm to (24.9, 24.6), turned to 0 degrees
- moved R8 4.78 mm to (15.8, 18.0), turned to 0 degrees
- moved R3 4.70 mm to (33.7, 34.3), turned to 0 degrees
- moved R7 3.91 mm to (34.4, 18.3), turned to 180 degrees
- moved TEST 3.08 mm to (44.1, 29.9)
- moved SW5 0.31 mm to (22.8, 28.1)
- moved SW4 0.19 mm to (22.8, 47.2)
- moved SW1 0.18 mm to (14.0, 37.7)
- moved SW3 0.13 mm to (31.8, 37.7)
- moved SW2 0.10 mm to (22.8, 37.6)
Connections:
- J2 pad 5: (no net) -> unconnected-(J2-Pad5)
- J2 pad 6: /UR -> /FR
- J2 pad 7: (no net) -> unconnected-(J2-Pad7)
- J2 pad 9: (no net) -> unconnected-(J2-Pad9)
Routing:
- net /UR: track 31.5 -> 20.3 mm
- net VCC: track 0.00 -> 10.6 mm, vias 0 -> 8
- net /FR: track 20.3 -> 29.4 mm
- net /DN: track 56.9 -> 50.5 mm
- net /UP: track 35.6 -> 41.6 mm
- net /RT: track 61.0 -> 56.1 mm, vias 2 -> 3
- net /UL: track 13.1 -> 13.7 mm
- net /LT: track 37.3 -> 36.7 mm
Other:
- board text added: "PWB Rev 2"
- board text removed: "PWB Rev 1"
