File: FPGA Cards/FPGA-ITX-01/FPGA-ITX-01.kicad_sch (KiCad schematic)
At the start: 73 parts, among them J1 AudioJack3_Ground_SwitchTR, J10 Header, Strt, 2x40, J11 Header, Strt, 2x40, J12 Header, Strt, 2x40, J13 Conn_02x05_Odd_Even, J14 Conn_02x05_Odd_Even, J15 Conn_01x02, J16 Conn_01x02, J2 PS2_DIN6, J3 Conn, USB B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

Commit message: New pics renamed
Parts:
- MTG1, MTG2, MTG3, MTG4: footprint MountingHole:MountingHole_4.3mm_M4 -> MountingHole:MountingHole_4.3mm_M4_DIN965_Pad
Changed lines of the file:
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@@
     (effects (font (size 1.27 1.27)) (justify left bottom))
   )
-  (text "(vgaVSync)" (at 417.83 265.43 0)
+  (text "(vgaVSync)" (at 417.83 270.51 0)
     (effects (font (size 1.27 1.27)) (justify left bottom))
   )
@@
       (effects (font (size 1.524 1.524)))
     )
-    (property "Footprint" "MountingHole:MountingHole_4.3mm_M4" (id 2) (at 406.4 410.21 0)
+    (property "Footprint" "MountingHole:MountingHole_4.3mm_M4_DIN965_Pad" (id 2) (at 406.4 410.21 0)
       (effects (font (size 1.524 1.524)))
     )
@@
       (effects (font (size 1.524 1.524)))
     )
-    (property "Footprint" "MountingHole:MountingHole_4.3mm_M4" (id 2) (at 406.4 394.97 0)
+    (property "Footprint" "MountingHole:MountingHole_4.3mm_M4_DIN965_Pad" (id 2) (at 406.4 394.97 0)
       (effects (font (size 1.524 1.524)))
     )
@@
       (effects (font (size 1.524 1.524)))
     )
-    (property "Footprint" "MountingHole:MountingHole_4.3mm_M4" (id 2) (at 406.4 402.59 0)
+    (property "Footprint" "MountingHole:MountingHole_4.3mm_M4_DIN965_Pad" (id 2) (at 406.4 402.59 0)
       (effects (font (size 1.524 1.524)))
     )
@@
       (effects (font (size 1.524 1.524)))
     )
-    (property "Footprint" "MountingHole:MountingHole_4.3mm_M4" (id 2) (at 406.4 387.35 0)
+    (property "Footprint" "MountingHole:MountingHole_4.3mm_M4_DIN965_Pad" (id 2) (at 406.4 387.35 0)
       (effects (font (size 1.524 1.524)))
     )
@@
     )
     (path "/00000000-0000-0000-0000-0000586ad6d2"
-      (reference "MTG1") (unit 1) (value "MTG_HOLE") (footprint "MountingHole:MountingHole_4.3mm_M4")
+      (reference "MTG1") (unit 1) (value "MTG_HOLE") (footprint "MountingHole:MountingHole_4.3mm_M4_DIN965_Pad")
     )
     (path "/00000000-0000-0000-0000-0000586ad65d"
-      (reference "MTG2") (unit 1) (value "MTG_HOLE") (footprint "MountingHole:MountingHole_4.3mm_M4")
+      (reference "MTG2") (unit 1) (value "MTG_HOLE") (footprint "MountingHole:MountingHole_4.3mm_M4_DIN965_Pad")
     )
     (path "/00000000-0000-0000-0000-0000586ad691"
-      (reference "MTG3") (unit 1) (value "MTG_HOLE") (footprint "MountingHole:MountingHole_4.3mm_M4")
+      (reference "MTG3") (unit 1) (value "MTG_HOLE") (footprint "MountingHole:MountingHole_4.3mm_M4_DIN965_Pad")
     )
     (path "/00000000-0000-0000-0000-0000586ad5e2"
-      (reference "MTG4") (unit 1) (value "MTG_HOLE") (footprint "MountingHole:MountingHole_4.3mm_M4")
+      (reference "MTG4") (unit 1) (value "MTG_HOLE") (footprint "MountingHole:MountingHole_4.3mm_M4_DIN965_Pad")
     )
     (path "/58a4a3fc-10f6-4aee-a8a9-abb54162050f"

Commit message: More FGPA-ITX-01 card tweeks
Parts:
- added J17: Conn_02x05_Odd_Even, Connector_PinHeader_2.54mm:PinHeader_2x05_P2.54mm_Vertical, symbol Connector_Generic:Conn_02x05_Odd_Even
Connections:
- net GND: now also J17.7 (Pin_7), J17.8 (Pin_8)
- net VS: now also J17.1 (Pin_1), J17.2 (Pin_2)
- no-connect marks 17 -> 23
Changed lines of the file:
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@@
   (junction (at 177.8 391.16) (diameter 0) (color 0 0 0 0)
   )
+  (junction (at 243.84 336.55) (diameter 0) (color 0 0 0 0)
+  )
   (junction (at 234.95 378.46) (diameter 0) (color 0 0 0 0)
   )
@@
   (no_connect (at 445.77 317.5))
   (no_connect (at 473.71 267.97))
+  (no_connect (at 241.3 353.06))
+  (no_connect (at 241.3 347.98))
+  (no_connect (at 241.3 345.44))
+  (no_connect (at 228.6 353.06))
+  (no_connect (at 228.6 345.44))
+  (no_connect (at 228.6 347.98))
   (no_connect (at 491.49 325.12))
   (no_connect (at 491.49 330.2))
@@
     (stroke (width 0) (type default) (color 0 0 0 0))
   )
+  (wire (pts (xy 243.84 334.01) (xy 243.84 336.55))
+    (stroke (width 0) (type default) (color 0 0 0 0))
+  )
   (wire (pts (xy 107.95 387.35) (xy 107.95 391.16))
     (stroke (width 0) (type default) (color 0 0 0 0))
@@
     (stroke (width 0) (type default) (color 0 0 0 0))
   )
+  (wire (pts (xy 246.38 350.52) (xy 241.3 350.52))
+    (stroke (width 0) (type default) (color 0 0 0 0))
+  )
   (wire (pts (xy 283.21 261.62) (xy 283.21 262.89))
     (stroke (width 0) (type default) (color 0 0 0 0))
@@
     (stroke (width 0) (type default) (color 0 0 0 0))
   )
+  (wire (pts (xy 222.25 350.52) (xy 228.6 350.52))
+    (stroke (width 0) (type default) (color 0 0 0 0))
+  )
   (wire (pts (xy 372.11 130.81) (xy 389.89 130.81))
     (stroke (width 0) (type default) (color 0 0 0 0))
@@
     (stroke (width 0) (type default) (color 0 0 0 0))
   )
+  (wire (pts (xy 222.25 360.68) (xy 222.25 350.52))
+    (stroke (width 0) (type default) (color 0 0 0 0))
+  )
   (wire (pts (xy 72.39 107.95) (xy 82.55 107.95))
     (stroke (width 0) (type default) (color 0 0 0 0))
@@
     (stroke (width 0) (type default) (color 0 0 0 0))
   )
+  (wire (pts (xy 226.06 342.9) (xy 226.06 336.55))
+    (stroke (width 0) (type default) (color 0 0 0 0))
+  )
   (wire (pts (xy 300.99 387.35) (xy 300.99 379.73))
     (stroke (width 0) (type default) (color 0 0 0 0))
@@
     (stroke (width 0) (type default) (color 0 0 0 0))
   )
+  (wire (pts (xy 226.06 336.55) (xy 243.84 336.55))
+    (stroke (width 0) (type default) (color 0 0 0 0))
+  )
   (wire (pts (xy 92.71 176.53) (xy 92.71 175.26))
     (stroke (width 0) (type default) (color 0 0 0 0))
@@
     (stroke (width 0) (type default) (color 0 0 0 0))
   )
+  (wire (pts (xy 228.6 342.9) (xy 226.06 342.9))
+    (stroke (width 0) (type default) (color 0 0 0 0))
+  )
   (wire (pts (xy 430.53 219.71) (xy 408.94 219.71))
     (stroke (width 0) (type default) (color 0 0 0 0))
@@
     (stroke (width 0) (type default) (color 0 0 0 0))
   )
+  (wire (pts (xy 243.84 336.55) (xy 243.84 342.9))
+    (stroke (width 0) (type default) (color 0 0 0 0))
+  )
   (wire (pts (xy 340.36 99.06) (xy 326.39 99.06))
     (stroke (width 0) (type default) (color 0 0 0 0))
@@
     (stroke (width 0) (type default) (color 0 0 0 0))
   )
+  (wire (pts (xy 243.84 342.9) (xy 241.3 342.9))
+    (stroke (width 0) (type default) (color 0 0 0 0))
+  )
   (wire (pts (xy 488.95 92.71) (xy 474.98 92.71))
     (stroke (width 0) (type default) (color 0 0 0 0))
@@
     (stroke (width 0) (type default) (color 0 0 0 0))
   )
+  (wire (pts (xy 246.38 360.68) (xy 246.38 350.52))
+    (stroke (width 0) (type default) (color 0 0 0 0))
+  )
   (wire (pts (xy 317.5 203.2) (xy 317.5 205.74))
     (stroke (width 0) (type default) (color 0 0 0 0))
@@
     (effects (font (size 1.27 1.27)) (justify left bottom))
   )
+  (text "KEY" (at 223.52 353.06 0)
+    (effects (font (size 1.27 1.27)) (justify left bottom))
+  )
   (text "(IO_AA22)" (at 54.61 59.69 0)
     (effects (font (size 1.27 1.27)) (justify left bottom))
@@
     (pin "2")
   )
+  (symbol (lib_id "Connector_Generic:Conn_02x05_Odd_Even") (at 233.68 347.98 0) (unit 1)
+    (in_bom yes) (on_board yes)
+    (property "Reference" "J17" (id 0) (at 234.95 340.36 0))
+    (property "Value" "Conn_02x05_Odd_Even" (id 1) (at 234.95 355.6 0))
+    (property "Footprint" "Connector_PinHeader_2.54mm:PinHeader_2x05_P2.54mm_Vertical" (id 2) (at 233.68 356.87 0)
+      (effects (font (size 0.762 0.762)))
+    )
+    (property "Datasheet" "~" (id 3) (at 233.68 347.98 0)
+      (effects (font (size 1.27 1.27)) hide)
+    )
+    (pin "1")
+    (pin "10")
+    (pin "2")
+    (pin "3")
+    (pin "4")
+    (pin "5")
+    (pin "6")
+    (pin "7")
+    (pin "8")
+    (pin "9")
+  )
   (symbol (lib_id "power:GND") (at 261.62 304.8 0) (unit 1)
     (in_bom yes) (on_board yes)
@@
     (pin "9")
   )
+  (symbol (lib_id "power:GND") (at 222.25 360.68 0) (unit 1)
+    (in_bom yes) (on_board yes)
+    (property "Reference" "#PWR0161" (id 0) (at 222.25 367.03 0)
+      (effects (font (size 1.27 1.27)) hide)
+    )
+    (property "Value" "GND" (id 1) (at 222.25 364.49 0))
+    (property "Footprint" "" (id 2) (at 222.25 360.68 0)
+      (effects (font (size 1.524 1.524)))
+    )
+    (property "Datasheet" "" (id 3) (at 222.25 360.68 0)
+      (effects (font (size 1.524 1.524)))
+    )
+    (pin "1")
+  )
   (symbol (lib_id "Connector_Generic:Conn_02x07_Odd_Even") (at 171.45 325.12 0) (unit 1)
     (in_bom yes) (on_board yes)
@@
     (pin "TN")
   )
+  (symbol (lib_id "power:VS") (at 243.84 334.01 0) (unit 1)
+    (in_bom yes) (on_board yes) (fields_autoplaced)
+    (property "Reference" "#PWR0163" (id 0) (at 238.76 337.82 0)
+      (effects (font (size 1.27 1.27)) hide)
+    )
+    (property "Value" "VS" (id 1) (at 245.237 333.219 0)
+      (effects (font (size 1.27 1.27)) (justify left))
+    )
+    (property "Footprint" "" (id 2) (at 243.84 334.01 0)
+      (effects (font (size 1.27 1.27)) hide)
+    )
+    (property "Datasheet" "" (id 3) (at 243.84 334.01 0)
+      (effects (font (size 1.27 1.27)) hide)
+    )
+    (pin "1")
+  )
   (symbol (lib_id "power:VS") (at 72.39 107.95 90) (unit 1)
     (in_bom yes) (on_board yes) (fields_autoplaced)
@@
     (pin "1")
   )
+  (symbol (lib_id "power:GND") (at 246.38 360.68 0) (unit 1)
+    (in_bom yes) (on_board yes)
+    (property "Reference" "#PWR0162" (id 0) (at 246.38 367.03 0)
+      (effects (font (size 1.27 1.27)) hide)
+    )
+    (property "Value" "GND" (id 1) (at 246.38 364.49 0))
+    (property "Footprint" "" (id 2) (at 246.38 360.68 0)
+      (effects (font (size 1.524 1.524)))
+    )
+    (property "Datasheet" "" (id 3) (at 246.38 360.68 0)
+      (effects (font (size 1.524 1.524)))
+    )
+    (pin "1")
+  )
   (symbol (lib_id "power:+3.3V") (at 101.6 25.4 0) (unit 1)
     (in_bom yes) (on_board yes)
@@
       (reference "#PWR0160") (unit 1) (value "VDD") (footprint "")
     )
+    (path "/862404ad-623e-4a2f-ae2c-79c39541eefe"
+      (reference "#PWR0161") (unit 1) (value "GND") (footprint "")
+    )
+    (path "/e90f36e2-0a78-4911-93e6-7c180ac1a0f4"
+      (reference "#PWR0162") (unit 1) (value "GND") (footprint "")
+    )
+    (path "/e7daa137-b0b1-49cc-bda1-a69ee2c5c568"
+      (reference "#PWR0163") (unit 1) (value "VS") (footprint "")
+    )
     (path "/9c15ae36-4e5d-45bc-ad22-b346fe75f679"
       (reference "C1") (unit 1) (value "0.1uF") (footprint "Capacitor_THT:C_Rect_L4.0mm_W2.5mm_P2.50mm")
@@
       (reference "J16") (unit 1) (value "Conn_01x02") (footprint "Connector_PinHeader_2.54mm:PinHeader_1x02_P2.54mm_Vertical")
     )
+    (path "/6377d728-1038-40d4-8681-ce7fe79c5248"
+      (reference "J17") (unit 1) (value "Conn_02x05_Odd_Even") (footprint "Connector_PinHeader_2.54mm:PinHeader_2x05_P2.54mm_Vertical")
+    )
     (path "/00000000-0000-0000-0000-00005ef1421b"
