File: ODAS Cards/ODAS-PSOC5/ODAS-PSOC5.kicad_pcb (KiCad board)
At the start: 2 copper layers, 55 x 95 mm, 48 parts, among them J1 DCJ0202, J2 USB-MICRO-B, P1 CONN_01X40, P2 CONN_01X04, P3 CONN_02X02, P4 CONN_01X06, U1 24C32, U2 CY8C5267AXI-LP051, U3 AP1117, U4 AP1117, Y1 Crystal_Small

Commit message: PSOC5 card
Parts:
- removed the C13 at (33.3, 19.9)
- removed the C14 at (47.2, 27.3)
- removed C16: 0.1uF, Capacitors_SMD:C_0805_HandSoldering
- removed F2: FUSE, Resistors_SMD:R_1206_HandSoldering
- removed J1: DCJ0202, dougsLib:JACK_3.5MM
- removed the TEST at (16.3, 88.9)
- removed the U3 at (42.3, 17.7)
- added C1: 0.1uF, Capacitor_SMD:C_1206_3216Metric_Pad1.33x1.80mm_HandSolder, F.Cu at (24.1, 25.1)
- added TEST: COUPON, LandBoards_Marking:TEST_BLK-REAR, F.Cu at (30.0, 99.6)
- C10: renamed from C3; footprint Capacitors_SMD:C_0805_HandSoldering -> Capacitor_SMD:C_0805_2012Metric_Pad1.18x1.45mm_HandSolder
- C11: renamed from C8; footprint Capacitors_SMD:C_0805_HandSoldering -> Capacitor_SMD:C_0805_2012Metric_Pad1.18x1.45mm_HandSolder
- C12: renamed from C9; footprint Capacitors_SMD:C_0805_HandSoldering -> Capacitor_SMD:C_0805_2012Metric_Pad1.18x1.45mm_HandSolder
- C13: renamed from C1; footprint Capacitors_SMD:C_0805_HandSoldering -> Capacitor_SMD:C_0805_2012Metric_Pad1.18x1.45mm_HandSolder
- C14: renamed from C5; footprint Capacitors_SMD:C_0805_HandSoldering -> Capacitor_SMD:C_0805_2012Metric_Pad1.18x1.45mm_HandSolder
- C2: renamed from C15; footprint Capacitors_SMD:C_0805_HandSoldering -> Capacitor_SMD:C_0805_2012Metric_Pad1.18x1.45mm_HandSolder
- C3: renamed from C12; footprint Capacitors_SMD:C_0805_HandSoldering -> Capacitor_SMD:C_0805_2012Metric_Pad1.18x1.45mm_HandSolder
- C4: renamed from C7; value C -> 12pF; footprint Capacitors_SMD:C_0805_HandSoldering -> Capacitor_SMD:C_0805_2012Metric_Pad1.18x1.45mm_HandSolder
- C5: renamed from C10; value C -> 12pF; footprint Capacitors_SMD:C_0805_HandSoldering -> Capacitor_SMD:C_0805_2012Metric_Pad1.18x1.45mm_HandSolder
- C6: renamed from C4; footprint Capacitors_SMD:C_0805_HandSoldering -> Capacitor_SMD:C_0805_2012Metric_Pad1.18x1.45mm_HandSolder
- C7: renamed from C6; footprint Capacitors_SMD:C_0805_HandSoldering -> Capacitor_SMD:C_0805_2012Metric_Pad1.18x1.45mm_HandSolder
- C8: renamed from C11; footprint Capacitors_SMD:C_0805_HandSoldering -> Capacitor_SMD:C_0805_2012Metric_Pad1.18x1.45mm_HandSolder
- C9: renamed from C2; footprint Capacitors_SMD:C_0805_HandSoldering -> Capacitor_SMD:C_0805_2012Metric_Pad1.18x1.45mm_HandSolder
- F1: value FUSE -> Poly Fuse (1206)
- P2: renamed from J2; value USB-MICRO-B -> USB-B; footprint DougsNewMods:USB_Micro-B-Wellco-SMT -> Connector_USB:USB_B_Lumberg_2411_02_Horizontal
- R1: renamed from R6; footprint Resistors_SMD:R_0805_HandSoldering -> Resistor_SMD:R_0805_2012Metric_Pad1.20x1.40mm_HandSolder
- R2: renamed from R7; footprint Resistors_SMD:R_0805_HandSoldering -> Resistor_SMD:R_0805_2012Metric_Pad1.20x1.40mm_HandSolder
- R3: renamed from R5; footprint Resistors_SMD:R_0805_HandSoldering -> Resistor_SMD:R_0805_2012Metric_Pad1.20x1.40mm_HandSolder
- R4: footprint Resistors_SMD:R_0805_HandSoldering -> Resistor_SMD:R_0805_2012Metric_Pad1.20x1.40mm_HandSolder
- R5: renamed from R1; footprint Resistors_SMD:R_0805_HandSoldering -> Resistor_SMD:R_0805_2012Metric_Pad1.20x1.40mm_HandSolder
- R6: renamed from R2; footprint Resistors_SMD:R_0805_HandSoldering -> Resistor_SMD:R_0805_2012Metric_Pad1.20x1.40mm_HandSolder
- R7: renamed from R3; footprint Resistors_SMD:R_0805_HandSoldering -> Resistor_SMD:R_0805_2012Metric_Pad1.20x1.40mm_HandSolder
- U1: renamed from U4; value AP1117 -> AZ1117-3.3
- U3: renamed from U1; value 24C32 -> CAT24C32WI-GT3
- moved FID2 27.3 mm to (51.1, 95.2)
- moved C3 12.0 mm to (44.5, 30.5), turned to -90 degrees
- moved P2 11.4 mm to (52.9, 32.0), turned to 0 degrees
- moved U1 11.2 mm to (36.8, 19.1)
- moved R1 9.74 mm to (48.3, 36.2)
- moved R2 8.39 mm to (48.3, 38.7)
- moved C2 2.87 mm to (30.0, 24.9)
- moved F1 2.87 mm to (27.4, 24.9)
- moved U3 2.84 mm to (38.4, 83.8)
- moved DS1 2.47 mm to (58.4, 43.7)
- moved C7 0.51 mm to (29.2, 49.0)
- moved R6 0.51 mm to (34.8, 92.2)
- moved C9 0.38 mm to (51.9, 57.1)
- renumbered H3 to H1, H4 to H2, H2 to H3, P3 to H4, H1 to P3, P2 to P5
Connections:
- C3 pad 1: /+9V -> +5VP
- FID1 pad 1: (no net) -> unconnected-(FID1-Pad1)
- FID2 pad 1: (no net) -> unconnected-(FID2-Pad1)
- MTG1 pad 1: (no net) -> unconnected-(MTG1-Pad1)
- MTG2 pad 1: (no net) -> unconnected-(MTG2-Pad1)
- MTG3 pad 1: (no net) -> unconnected-(MTG3-Pad1)
- MTG4 pad 1: (no net) -> unconnected-(MTG4-Pad1)
- P1 pad 39: (no net) -> GND
- P1 pad 40: (no net) -> GND
- P2 pad 1: (no net) -> +5VP
- P2 pad 4: (no net) -> GND
- P2 pad 5: GND -> (no net)
- U1 pad 3: +5V -> +5VP
- U2 pad 1: (no net) -> unconnected-(U2-Pad1)
- U2 pad 11: (no net) -> unconnected-(U2-Pad11)
- U2 pad 16: (no net) -> unconnected-(U2-Pad16)
- U2 pad 17: (no net) -> unconnected-(U2-Pad17)
- U2 pad 18: (no net) -> unconnected-(U2-Pad18)
- U2 pad 19: (no net) -> unconnected-(U2-Pad19)
- U2 pad 2: (no net) -> unconnected-(U2-Pad2)
- U2 pad 22: (no net) -> unconnected-(U2-Pad22)
- U2 pad 23: (no net) -> unconnected-(U2-Pad23)
- U2 pad 24: (no net) -> unconnected-(U2-Pad24)
- U2 pad 25: (no net) -> unconnected-(U2-Pad25)
- U2 pad 27: (no net) -> unconnected-(U2-Pad27)
- U2 pad 28: (no net) -> unconnected-(U2-Pad28)
- U2 pad 29: (no net) -> unconnected-(U2-Pad29)
- U2 pad 3: (no net) -> unconnected-(U2-Pad3)
- U2 pad 30: (no net) -> unconnected-(U2-Pad30)
- U2 pad 32: (no net) -> unconnected-(U2-Pad32)
- U2 pad 33: (no net) -> unconnected-(U2-Pad33)
- U2 pad 34: (no net) -> unconnected-(U2-Pad34)
- U2 pad 40: (no net) -> unconnected-(U2-Pad40)
- U2 pad 41: (no net) -> unconnected-(U2-Pad41)
- U2 pad 57: (no net) -> unconnected-(U2-Pad57)
- U2 pad 58: (no net) -> unconnected-(U2-Pad58)
- U2 pad 59: (no net) -> unconnected-(U2-Pad59)
- U2 pad 60: (no net) -> unconnected-(U2-Pad60)
- U2 pad 61: (no net) -> unconnected-(U2-Pad61)
- U2 pad 62: (no net) -> unconnected-(U2-Pad62)
- U2 pad 89: (no net) -> unconnected-(U2-Pad89)
- U2 pad 90: (no net) -> unconnected-(U2-Pad90)
- U2 pad 91: (no net) -> unconnected-(U2-Pad91)
- U2 pad 92: (no net) -> unconnected-(U2-Pad92)
- U2 pad 93: (no net) -> unconnected-(U2-Pad93)
- U2 pad 94: (no net) -> unconnected-(U2-Pad94)
- U2 pad 95: (no net) -> unconnected-(U2-Pad95)
- U2 pad 96: (no net) -> unconnected-(U2-Pad96)
- U2 pad 97: (no net) -> unconnected-(U2-Pad97)
- U2 pad 98: (no net) -> unconnected-(U2-Pad98)
- U2 pad 99: (no net) -> unconnected-(U2-Pad99)
Routing:
- net +5V: track 67.9 -> 39.8 mm, vias 4 -> 2
- net +3V3: track 63.5 -> 50.4 mm
- net Net-(R2-Pad2): track 23.8 -> 13.6 mm, vias 2 -> 0
- net GND: track 56.5 -> 47.5 mm, vias 25 -> 22
- net +5VP: track 57.2 -> 52.1 mm, vias 1 -> 2
- net /USB-DP: track 4.01 -> 8.07 mm
- net Net-(R1-Pad2): track 21.1 -> 17.3 mm
- net /WR: track 14.5 -> 18.3 mm
- net /VZ3: track 3.77 -> 0.00 mm
- net /SCL: track 55.1 -> 51.5 mm
- net +3.3VP: track 119.8 -> 117.8 mm
- net /USB-DM: track 3.08 -> 4.70 mm
- net /SDA: track 52.3 -> 50.9 mm
- net Net-(C8-Pad2): track 6.63 -> 5.38 mm
- net /IO_22: track 9.50 -> 8.71 mm
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- added copper zone on F.Cu, net +5VP
- removed copper zone on F.Cu, net +5V
- removed copper zone on F.Cu, net /+9V
Other:
- net class Default removed
- net class POWER removed
- board text added: "55"
- board text added: "67"
- board text added: "73"
- board text added: "76"
- board text added: "82"
- board text added: "84"
- board text added: "G VZ3"
- board text added: "REV 5"
- board text added: "USB"
- board text added: "V0 G"
- board text removed: "67 68"
- board text removed: "73 74"
- board text removed: "76 77"
- board text removed: "82 83"
- board text removed: "9V"
- board text removed: "G N D"
- board text removed: "G V"
- board text removed: "REV X4"
- board text removed: "V G"

Commit message: ODAS-PSOC5 card
Parts:
- moved R1 4.24 mm to (45.0, 38.9), turned to -90 degrees
- moved R3 4.19 mm to (50.5, 43.7)
- moved U3 3.81 mm to (40.6, 80.8)
- moved C14 3.59 mm to (32.8, 74.7)
- moved P4 1.78 mm to (54.4, 63.2)
- moved R6 0.51 mm to (34.8, 91.7)
- moved R2 0.13 mm to (48.3, 38.9), turned to -90 degrees
Routing:
- net /USB-DM: track 4.70 -> 10.4 mm
- net Net-(R1-Pad2): track 17.3 -> 11.9 mm
- net /WR: track 18.3 -> 22.7 mm
- net /P5-4: track 6.60 -> 11.0 mm
- net Net-(DS1-Pad2): track 9.96 -> 5.82 mm
- net /SPISCK: track 22.7 -> 20.1 mm
- net +3.3VP: track 117.8 -> 120.4 mm
- net /SPICE0: track 23.8 -> 21.6 mm
- net /SPIMOSI: track 11.2 -> 9.74 mm
- net /USB-DP: track 8.07 -> 9.06 mm
- net /SPIMISO: track 17.2 -> 16.5 mm
- net /SDA: track 50.9 -> 51.1 mm, vias 2 -> 3
Other:
- board text added: "3V 5V"
- board text added: "GND 3.3V SDA SCL"
- board text added: "GND VZ3 44 45 46 47 48 49 51 53 54 55 67 69 70 71 72 73 76 78 79 80 81 82 84 V0 GD"
- board text added: "MO MI CK CE 3V GND"
- board text removed: "3.3V"
- board text removed: "3V"
- board text removed: "44 45"
- board text removed: "46 47"
- board text removed: "48 49"
- board text removed: "53 54"
- board text removed: "55"
- board text removed: "5V"
- board text removed: "67"
- board text removed: "69 70"
- board text removed: "71 72"
- board text removed: "73"
- board text removed: "76"
- board text removed: "78 79"
- board text removed: "80 81"
- board text removed: "82"
- board text removed: "84"
- board text removed: "G VZ3"
- board text removed: "MO MI CE E +V GND"
- board text removed: "SDA"
- board text removed: "SPI"
- board text removed: "V0 G"
