File: SYNTHS/ER-ADSR-555-01_SET/ER-ADSR-555-01-controls/Rev1/ER-ADSR-555-01.kicad_sch (KiCad schematic)
At the start: 32 parts, among them J1 Conn_02x05, J2 PJ-301BM, J3 PJ-301BM, Q1 2N3904, Q2 2N3904, Q3 2N3904, U1 TL072, U2 LM555N

Commit message: ADSR working
Parts:
- added R12: 10K, Resistor_THT:R_Axial_DIN0204_L3.6mm_D1.6mm_P7.62mm_Horizontal, symbol Device:R
- C3: value 4.7uF -> 1uF
- D1: value BAT41 -> 1N4148
- RV1, RV2, RV4: value 1M -> A1M
- RV3: value 10M -> B10K
- renumbered R11 to R10
Connections:
- net BUFA: now also R12.1
- net RST: now also R12.2
Other:
- note added: "ADDED IN REWORK"
- moved on the sheet: R4
Changed lines of the file:
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@@
     (stroke (width 0) (type default) (color 0 0 0 0))
   )
-  (wire (pts (xy 184.15 116.84) (xy 184.15 119.38))
+  (wire (pts (xy 184.15 114.3) (xy 184.15 116.84))
     (stroke (width 0) (type default) (color 0 0 0 0))
   )
@@
     (stroke (width 0) (type default) (color 0 0 0 0))
   )
-  (wire (pts (xy 184.15 127) (xy 184.15 128.27))
+  (wire (pts (xy 184.15 124.46) (xy 184.15 128.27))
     (stroke (width 0) (type default) (color 0 0 0 0))
   )
@@
     (stroke (width 0) (type default) (color 0 0 0 0))
   )
+  (wire (pts (xy 154.305 110.49) (xy 162.56 110.49))
+    (stroke (width 0) (type default) (color 0 0 0 0))
+  )
   (wire (pts (xy 138.43 140.97) (xy 146.05 140.97))
     (stroke (width 0) (type default) (color 0 0 0 0))
@@
   )
   (wire (pts (xy 213.995 46.99) (xy 213.995 49.53))
+    (stroke (width 0) (type default) (color 0 0 0 0))
+  )
+  (wire (pts (xy 135.255 110.49) (xy 146.685 110.49))
     (stroke (width 0) (type default) (color 0 0 0 0))
   )
@@
     (effects (font (size 1.27 1.27)) (justify left bottom))
   )
+  (text "ADDED IN REWORK" (at 140.335 105.41 0)
+    (effects (font (size 1.27 1.27)) (justify left bottom))
+  )
   (label "BUFB" (at 168.91 134.62 0)
     (effects (font (size 1.27 1.27)) (justify left bottom))
@@
     (effects (font (size 1.27 1.27)) (justify left bottom))
   )
+  (label "RST" (at 157.48 110.49 0)
+    (effects (font (size 1.27 1.27)) (justify left bottom))
+  )
   (label "BUFC" (at 210.82 128.27 0)
     (effects (font (size 1.27 1.27)) (justify left bottom))
@@
   )
   (label "THR" (at 88.265 69.85 0)
+    (effects (font (size 1.27 1.27)) (justify left bottom))
+  )
+  (label "BUFA" (at 138.43 110.49 0)
     (effects (font (size 1.27 1.27)) (justify left bottom))
   )
@@
   (symbol (lib_id "Device:R") (at 93.345 35.56 90) (unit 1)
     (in_bom yes) (on_board yes)
-    (property "Reference" "R11" (id 0) (at 93.345 33.02 90))
+    (property "Reference" "R10" (id 0) (at 93.345 33.02 90))
     (property "Value" "RR" (id 1) (at 93.345 35.56 90))
     (property "Footprint" "Resistor_THT:R_Axial_DIN0204_L3.6mm_D1.6mm_P7.62mm_Horizontal" (id 2) (at 92.075 83.82 90)
@@
       (effects (font (size 1.27 1.27)) (justify left))
     )
-    (property "Value" "BAT41" (id 1) (at 140.462 148.8691 90)
+    (property "Value" "1N4148" (id 1) (at 140.462 148.8691 90)
       (effects (font (size 1.27 1.27)) (justify left))
     )
@@
     (in_bom yes) (on_board yes)
     (property "Reference" "C3" (id 0) (at 183.515 39.37 0))
-    (property "Value" "4.7uF" (id 1) (at 184.785 44.45 0))
+    (property "Value" "1uF" (id 1) (at 184.785 44.45 0))
     (property "Footprint" "Capacitor_THT:CP_Radial_D5.0mm_P2.50mm" (id 2) (at 180.975 74.93 0)
       (effects (font (size 0.762 0.762)))
@@
     (pin "1")
   )
-  (symbol (lib_id "Device:R") (at 184.15 123.19 180) (unit 1)
-    (in_bom yes) (on_board yes)
-    (property "Reference" "R4" (id 0) (at 181.61 123.19 90))
-    (property "Value" "4.7K" (id 1) (at 184.15 123.19 90))
+  (symbol (lib_id "Device:R") (at 184.15 120.65 180) (unit 1)
+    (in_bom yes) (on_board yes)
+    (property "Reference" "R4" (id 0) (at 181.61 120.65 90))
+    (property "Value" "4.7K" (id 1) (at 184.15 120.65 90))
     (property "Footprint" "Resistor_THT:R_Axial_DIN0204_L3.6mm_D1.6mm_P7.62mm_Horizontal" (id 2) (at 181.61 161.29 0)
       (effects (font (size 0.762 0.762)))
     )
-    (property "Datasheet" "" (id 3) (at 184.15 123.19 0)
+    (property "Datasheet" "" (id 3) (at 184.15 120.65 0)
       (effects (font (size 1.27 1.27)) hide)
     )
@@
     (in_bom yes) (on_board yes)
     (property "Reference" "RV1" (id 0) (at 111.125 45.085 90))
-    (property "Value" "1M" (id 1) (at 107.315 51.435 90))
+    (property "Value" "A1M" (id 1) (at 107.315 51.435 90))
     (property "Footprint" "LandBoards_Conns:RV09ACF" (id 2) (at 97.155 86.36 90)
       (effects (font (size 0.762 0.762)))
@@
     (pin "3")
   )
+  (symbol (lib_id "Device:R") (at 150.495 110.49 90) (unit 1)
+    (in_bom yes) (on_board yes)
+    (property "Reference" "R12" (id 0) (at 150.495 107.95 90))
+    (property "Value" "10K" (id 1) (at 150.495 110.49 90))
+    (property "Footprint" "Resistor_THT:R_Axial_DIN0204_L3.6mm_D1.6mm_P7.62mm_Horizontal" (id 2) (at 196.215 165.1 90)
+      (effects (font (size 0.762 0.762)))
+    )
+    (property "Datasheet" "" (id 3) (at 150.495 110.49 0)
+      (effects (font (size 1.27 1.27)) hide)
+    )
+    (pin "1")
+    (pin "2")
+  )
   (symbol (lib_id "Amplifier_Operational:TL072") (at 161.925 59.69 0) (unit 1)
     (in_bom yes) (on_board yes) (fields_autoplaced)
@@
     (in_bom yes) (on_board yes)
     (property "Reference" "RV2" (id 0) (at 167.64 36.195 90))
-    (property "Value" "1M" (id 1) (at 173.355 40.64 90))
+    (property "Value" "A1M" (id 1) (at 173.355 40.64 90))
     (property "Footprint" "LandBoards_Conns:RV09ACF" (id 2) (at 170.815 72.39 0)
       (effects (font (size 0.762 0.762)))
@@
       (effects (font (size 1.27 1.27)) (justify right))
     )
-    (property "Value" "10M" (id 1) (at 135.8995 59.0166 0)
+    (property "Value" "B10K" (id 1) (at 135.8995 59.0166 0)
       (effects (font (size 1.27 1.27)) (justify right))
     )
@@
     (in_bom yes) (on_board yes)
     (property "Reference" "RV4" (id 0) (at 111.76 32.385 90))
-    (property "Value" "1M" (id 1) (at 107.315 38.1 90))
+    (property "Value" "A1M" (id 1) (at 107.315 38.1 90))
     (property "Footprint" "LandBoards_Conns:RV09ACF" (id 2) (at 121.92 85.09 90)
       (effects (font (size 0.762 0.762)))
@@
     (pin "1")
   )
-  (symbol (lib_id "power:+12V") (at 184.15 116.84 0) (unit 1)
-    (in_bom yes) (on_board yes) (fields_autoplaced)
-    (property "Reference" "#PWR0109" (id 0) (at 184.15 120.65 0)
-      (effects (font (size 1.27 1.27)) hide)
-    )
-    (property "Value" "+12V" (id 1) (at 184.15 113.2355 0))
-    (property "Footprint" "" (id 2) (at 184.15 116.84 0)
-      (effects (font (size 1.27 1.27)) hide)
-    )
-    (property "Datasheet" "" (id 3) (at 184.15 116.84 0)
+  (symbol (lib_id "power:+12V") (at 184.15 114.3 0) (unit 1)
+    (in_bom yes) (on_board yes) (fields_autoplaced)
+    (property "Reference" "#PWR0109" (id 0) (at 184.15 118.11 0)
+      (effects (font (size 1.27 1.27)) hide)
+    )
+    (property "Value" "+12V" (id 1) (at 184.15 110.6955 0))
+    (property "Footprint" "" (id 2) (at 184.15 114.3 0)
+      (effects (font (size 1.27 1.27)) hide)
+    )
+    (property "Datasheet" "" (id 3) (at 184.15 114.3 0)
       (effects (font (size 1.27 1.27)) hide)
     )
@@
     )
     (path "/4d9ddca8-237d-4fed-afce-2dc8bfdc81da"
-      (reference "C3") (unit 1) (value "4.7uF") (footprint "Capacitor_THT:CP_Radial_D5.0mm_P2.50mm")
+      (reference "C3") (unit 1) (value "1uF") (footprint "Capacitor_THT:CP_Radial_D5.0mm_P2.50mm")
     )
     (path "/385944b7-b92f-48d1-aba2-2e2851ac8880"
-      (reference "D1") (unit 1) (value "BAT41") (footprint "Diode_THT:D_DO-35_SOD27_P7.62mm_Horizontal")
+      (reference "D1") (unit 1) (value "1N4148") (footprint "Diode_THT:D_DO-35_SOD27_P7.62mm_Horizontal")
     )
     (path "/fce335e6-7a2a-4a7b-a2a4-dd31f2593c10"
@@
     )
     (path "/29f47cc6-270a-4f64-88b2-0f43ec88976e"
-      (reference "R11") (unit 1) (value "RR") (footprint "Resistor_THT:R_Axial_DIN0204_L3.6mm_D1.6mm_P7.62mm_Horizontal")
+      (reference "R10") (unit 1) (value "RR") (footprint "Resistor_THT:R_Axial_DIN0204_L3.6mm_D1.6mm_P7.62mm_Horizontal")
     )
     (path "/f4047145-9d9a-4593-9216-cccdd673bb27"
       (reference "R11") (unit 1) (value "10K") (footprint "Resistor_THT:R_Axial_DIN0204_L3.6mm_D1.6mm_P7.62mm_Horizontal")
     )
+    (path "/a3f11492-7936-40fd-853f-e2b42a257f46"
+      (reference "R12") (unit 1) (value "10K") (footprint "Resistor_THT:R_Axial_DIN0204_L3.6mm_D1.6mm_P7.62mm_Horizontal")
+    )
     (path "/9ce23001-4bd5-46ab-ac87-cb915687a3df"
-      (reference "RV1") (unit 1) (value "1M") (footprint "LandBoards_Conns:RV09ACF")
+      (reference "RV1") (unit 1) (value "A1M") (footprint "LandBoards_Conns:RV09ACF")
     )
     (path "/b7ad75e5-01c2-4b94-bc64-2241e8ac8d34"
-      (reference "RV2") (unit 1) (value "1M") (footprint "LandBoards_Conns:RV09ACF")
+      (reference "RV2") (unit 1) (value "A1M") (footprint "LandBoards_Conns:RV09ACF")
     )
     (path "/c042aded-2414-4721-91f9-54216ce8e0c0"
-      (reference "RV3") (unit 1) (value "10M") (footprint "LandBoards_Conns:RV09ACF")
+      (reference "RV3") (unit 1) (value "B10K") (footprint "LandBoards_Conns:RV09ACF")
     )
     (path "/ecc008dc-5f2b-47eb-9522-092e9f50e7d1"
-      (reference "RV4") (unit 1) (value "1M") (footprint "LandBoards_Conns:RV09ACF")
+      (reference "RV4") (unit 1) (value "A1M") (footprint "LandBoards_Conns:RV09ACF")
     )
     (path "/a49f7437-7605-4a08-b3ab-0ea16e8bc6c8"
