File: SYNTHS/ER-VCA2-01_SET/ER-VCA2-01-CTRLS/ER-VCA2-01-CTRLS.kicad_pcb (KiCad board)
At the start: 2 copper layers, 28 x 86 mm, 12 parts, among them J1 Conn_01x06, J2 Conn_01x08, J3 AudioJack3, J4 AudioJack3, J5 AudioJack3, J6 AudioJack3, J7 AudioJack3, J8 AudioJack3

Commit message: SYNTH CARDS
Parts:
- removed ? (x2): , 
- moved J2 4.00 mm to (59.0, 113.5)
Routing:
- net /IN2: track 56.6 -> 60.6 mm
- net /OUT2: track 22.3 -> 26.3 mm
- net /OUT1: track 20.1 -> 24.1 mm
- net /MOD2: track 40.7 -> 44.7 mm
- net /MOD1: track 38.1 -> 42.1 mm
- net /IN1: track 58.2 -> 62.2 mm
Other:
- board size 28 x 86 mm -> 28 x 88 mm
- board text added: "ER-VCA2-01-DB"
- board text added: "GND IN2 IN1 MOD2 MOD1 OUT2 OUT1 GND"
- board text added: "REV 2"
- board text removed: "ADJ 1"
- board text removed: "ADJ 2"
- board text removed: "IN 1"
- board text removed: "IN 2"
- board text removed: "MOD 1"
- board text removed: "MOD 2"
- board text removed: "OUT 1"
- board text removed: "OUT 2"
- board text removed: "land-boards.com/ SYNTH-VCA2-01"

Commit message: CARD UPDATES
Parts:
- J1: value Conn_01x06 -> HDR, FEM, 1x6
- J2: value Conn_01x08 -> HDR, FEM, 1x8
- J3, J4, J5, J6, J7, J8: value AudioJack3 -> JACK, 3.5MM, PJ301BM
- RV1, RV2: value POT -> B100K
Changed lines of the file:
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@@
   (paper "A")
   (title_block
-    (date "2022-10-17")
-    (rev "1")
+    (title "ER-VCA2-01-CTRLS")
+    (date "2022-11-29")
+    (rev "2")
+    (company "LAND BOARDS LLC")
   )
   (layers
@@
     (descr "Through hole straight socket strip, 1x08, 2.54mm pitch, single row (from Kicad 4.0.7), script generated")
     (tags "Through hole socket strip THT 1x08 2.54mm single row")
-    (property "Sheetfile" "SYNTH-VCA2-01-CTRLS.kicad_sch")
+    (property "Sheetfile" "ER-VCA2-01-CTRLS.kicad_sch")
     (property "Sheetname" "")
     (attr through_hole)
@@
       (effects (font (size 1.397 1.397) (thickness 0.3048)))
     )
-    (fp_text value "Conn_01x08" (at 0 20.55 90) (layer "F.Fab")
+    (fp_text value "HDR, FEM, 1x8" (at 0 20.55 90) (layer "F.Fab")
       (effects (font (size 1 1) (thickness 0.15)))
     )
@@
     (descr "Through hole straight socket strip, 1x06, 2.54mm pitch, single row (from Kicad 4.0.7), script generated")
     (tags "Through hole socket strip THT 1x06 2.54mm single row")
-    (property "Sheetfile" "SYNTH-VCA2-01-CTRLS.kicad_sch")
+    (property "Sheetfile" "ER-VCA2-01-CTRLS.kicad_sch")
     (property "Sheetname" "")
     (attr through_hole)
@@
       (effects (font (size 1.397 1.397) (thickness 0.3048)))
     )
-    (fp_text value "Conn_01x06" (at 0 15.47 90) (layer "F.Fab")
+    (fp_text value "HDR, FEM, 1x6" (at 0 15.47 90) (layer "F.Fab")
       (effects (font (size 1 1) (thickness 0.15)))
     )
@@
     (descr "TRS 3.5mm, horizontal, through-hole, https://www.cui.com/product/resource/sj1-353xng.pdf")
     (tags "TRS audio jack stereo horizontal")
-    (property "Sheetfile" "SYNTH-VCA2-01-CTRLS.kicad_sch")
+    (property "Sheetfile" "ER-VCA2-01-CTRLS.kicad_sch")
     (property "Sheetname" "")
     (attr through_hole)
@@
       (effects (font (size 1.397 1.397) (thickness 0.3048)) (justify mirror))
     )
-    (fp_text value "AudioJack3" (at 0.3 -6.7) (layer "B.Fab")
+    (fp_text value "JACK, 3.5MM, PJ301BM" (at 0.3 -6.7) (layer "B.Fab")
       (effects (font (size 1 1) (thickness 0.15)) (justify mirror))
     )
@@
     (descr "TRS 3.5mm, horizontal, through-hole, https://www.cui.com/product/resource/sj1-353xng.pdf")
     (tags "TRS audio jack stereo horizontal")
-    (property "Sheetfile" "SYNTH-VCA2-01-CTRLS.kicad_sch")
+    (property "Sheetfile" "ER-VCA2-01-CTRLS.kicad_sch")
     (property "Sheetname" "")
     (attr through_hole)
@@
       (effects (font (size 1.397 1.397) (thickness 0.3048)) (justify mirror))
     )
-    (fp_text value "AudioJack3" (at 0.3 -6.7) (layer "B.Fab")
+    (fp_text value "JACK, 3.5MM, PJ301BM" (at 0.3 -6.7) (layer "B.Fab")
       (effects (font (size 1 1) (thickness 0.15)) (justify mirror))
     )
@@
     (descr "TRS 3.5mm, horizontal, through-hole, https://www.cui.com/product/resource/sj1-353xng.pdf")
     (tags "TRS audio jack stereo horizontal")
-    (property "Sheetfile" "SYNTH-VCA2-01-CTRLS.kicad_sch")
+    (property "Sheetfile" "ER-VCA2-01-CTRLS.kicad_sch")
     (property "Sheetname" "")
     (attr through_hole)
@@
       (effects (font (size 1.397 1.397) (thickness 0.3048)) (justify mirror))
     )
-    (fp_text value "AudioJack3" (at 0.3 -6.7) (layer "B.Fab")
+    (fp_text value "JACK, 3.5MM, PJ301BM" (at 0.3 -6.7) (layer "B.Fab")
       (effects (font (size 1 1) (thickness 0.15)) (justify mirror))
     )
@@
     (descr "TRS 3.5mm, horizontal, through-hole, https://www.cui.com/product/resource/sj1-353xng.pdf")
     (tags "TRS audio jack stereo horizontal")
-    (property "Sheetfile" "SYNTH-VCA2-01-CTRLS.kicad_sch")
+    (property "Sheetfile" "ER-VCA2-01-CTRLS.kicad_sch")
     (property "Sheetname" "")
     (attr through_hole)
@@
       (effects (font (size 1.397 1.397) (thickness 0.3048)) (justify mirror))
     )
-    (fp_text value "AudioJack3" (at 0.3 -6.7) (layer "B.Fab")
+    (fp_text value "JACK, 3.5MM, PJ301BM" (at 0.3 -6.7) (layer "B.Fab")
       (effects (font (size 1 1) (thickness 0.15)) (justify mirror))
     )
@@
     (descr "TRS 3.5mm, horizontal, through-hole, https://www.cui.com/product/resource/sj1-353xng.pdf")
     (tags "TRS audio jack stereo horizontal")
-    (property "Sheetfile" "SYNTH-VCA2-01-CTRLS.kicad_sch")
+    (property "Sheetfile" "ER-VCA2-01-CTRLS.kicad_sch")
     (property "Sheetname" "")
     (attr through_hole)
@@
       (effects (font (size 1.397 1.397) (thickness 0.3048)) (justify mirror))
     )
-    (fp_text value "AudioJack3" (at 0.3 -6.7) (layer "B.Fab")
+    (fp_text value "JACK, 3.5MM, PJ301BM" (at 0.3 -6.7) (layer "B.Fab")
       (effects (font (size 1 1) (thickness 0.15)) (justify mirror))
     )
@@
     (descr "TRS 3.5mm, horizontal, through-hole, https://www.cui.com/product/resource/sj1-353xng.pdf")
     (tags "TRS audio jack stereo horizontal")
-    (property "Sheetfile" "SYNTH-VCA2-01-CTRLS.kicad_sch")
+    (property "Sheetfile" "ER-VCA2-01-CTRLS.kicad_sch")
     (property "Sheetname" "")
     (attr through_hole)
@@
       (effects (font (size 1.397 1.397) (thickness 0.3048)) (justify mirror))
     )
-    (fp_text value "AudioJack3" (at 0.3 -6.7) (layer "B.Fab")
+    (fp_text value "JACK, 3.5MM, PJ301BM" (at 0.3 -6.7) (layer "B.Fab")
       (effects (font (size 1 1) (thickness 0.15)) (justify mirror))
     )
@@
     (descr "Potentiometer, vertical, Bourns PTV09A-1 Single, http://www.bourns.com/docs/Product-Datasheets/ptv09.pdf")
     (tags "Potentiometer vertical Bourns PTV09A-1 Single")
-    (property "Sheetfile" "SYNTH-VCA2-01-CTRLS.kicad_sch")
+    (property "Sheetfile" "ER-VCA2-01-CTRLS.kicad_sch")
     (property "Sheetname" "")
     (attr through_hole)
@@
       (effects (font (size 1.397 1.397) (thickness 0.3048)) (justify mirror))
     )
-    (fp_text value "POT" (at 6.05 -5.15 90) (layer "B.Fab")
+    (fp_text value "B100K" (at 6.05 -5.15 90) (layer "B.Fab")
       (effects (font (size 1 1) (thickness 0.15)) (justify mirror))
     )
@@
     (descr "Potentiometer, vertical, Bourns PTV09A-1 Single, http://www.bourns.com/docs/Product-Datasheets/ptv09.pdf")
     (tags "Potentiometer vertical Bourns PTV09A-1 Single")
-    (property "Sheetfile" "SYNTH-VCA2-01-CTRLS.kicad_sch")
+    (property "Sheetfile" "ER-VCA2-01-CTRLS.kicad_sch")
     (property "Sheetname" "")
     (attr through_hole)
@@
       (effects (font (size 1.397 1.397) (thickness 0.3048)) (justify mirror))
     )
-    (fp_text value "POT" (at 6.05 -5.15 90) (layer "B.Fab")
-      (effects (font (size 1 1) (thickness 0.15)) (justify mirror))
-    )
+    (fp_text value "B100K" (at 6.05 -5.15 90) (layer "B.Fab")
+      (effects (font (size 1 1) (thickness 0.15)) (justify mirror))
+    )
