File: SYNTHS/ER-VCO-03_SET/ER-VCO-03_CTL/ER-VCO-03_CTL.kicad_pcb (KiCad board)
At the start: 2 copper layers, 28 x 100 mm, 32 parts, among them J1 PJ-301BM, J2 PJ-301BM, J3 PJ-301BM, J4 PJ-301BM, J5 Conn_01x16, J6 Conn_01x03, SW1 SW_Push, SW2 SW_SPDT_MSM, SW4 SW_SPDT_MSM

Commit message: SYNTHS
Parts:
- J1: renamed from J6; value Conn_01x03 -> HEADER, STRT, 1X3
- J6: renamed from J5; value Conn_01x16 -> HEADER, STRT, 2X8
- SW2: renamed from SW4; moved to B.Cu
- SW3: renamed from SW2; moved to B.Cu
- turned SW2 to 0 degrees
- turned SW3 to 0 degrees
- renumbered C5 to C1, C6 to C2, C8 to C3, C7 to C4, C4 to C5, C1 to C6, D6 to D1, D5 to D2, D8 to D3, D7 to D4, D4 to D5, D3 to D6, J3 to J2, J4 to J3, J1 to J4, J2 to J5, R10 to R1, R9 to R2, R11 to R3, R12 to R4, R14 to R5, R13 to R6, R8 to R7, R7 to R8, R1 to R9, RV2 to RV1, RV1 to RV2
