File: SYNTHS/ER-PROTO-02_SET/ER-PROTO-02-MOZZI-DB/ER-PROTO-02-MOZZI-DB.kicad_pcb (KiCad board)
At the start: 2 copper layers, 28 x 108.5 mm, 48 parts, among them J1 Conn_01x04, J10 Conn_01x12, J7 Conn_2x8, J8 HEADER, 2X10, J9 CONN, IDC, 2X5

Commit message: BOARD UPDATES
Parts:
- J7: value Conn_2x8 -> PROTO02_JACKS
- J8: value HEADER, 2X10 -> PROTO01_POTS
Connections:
- net Net-(A1-Pad25) renamed /ANA6
- net Net-(A1-Pad26) renamed /ANA7
- A1 pad 22: /J1-R_N -> /ANA3
- A1 pad 23: /J2-R_N -> /ANA4
- A1 pad 24: /J3-R_N -> /ANA5
- C1 pad 1: /J3-R_N -> /POT6-2
- C10 pad 1: /J1-R_N -> /ANA3
- C12 pad 1: /J3-R_N -> /ANA5
- C2 pad 1: /J1-R_N -> /POT4-2
- C4 pad 1: /J2-R_N -> /POT5-2
- C9 pad 1: /J2-R_N -> /ANA4
- D1 pad 1: /J2-R_N -> /ANA4
- D2 pad 2: /J2-R_N -> /ANA4
- D3 pad 1: /J1-R_N -> /ANA3
- D4 pad 2: /J1-R_N -> /ANA3
- D7 pad 1: /J3-R_N -> /ANA5
- D8 pad 2: /J3-R_N -> /ANA5
- J1 pad 3: /J2-R_N -> /ANA4
- J1 pad 4: /J3-R_N -> /ANA5
- J7 pad 11: /J3-R_N -> /POT6-2
- J7 pad 7: /J2-R_N -> /POT5-2
- J7 pad 9: /J1-R_N -> /POT4-2
- J8 pad 12: /J2-R_N -> /POT5-2
- J8 pad 3: /J3-R_N -> /POT6-2
- J8 pad 6: /J1-R_N -> /POT4-2
- R1 pad 2: /J2-R_N -> /ANA4
- R3 pad 2: /J1-R_N -> /ANA3
- R7 pad 2: /J3-R_N -> /ANA5
Routing:
- net /J3-R_N: track 127.4 -> 0.00 mm, vias 4 -> 0
- net /J1-R_N: track 126.1 -> 0.00 mm, vias 6 -> 0
- net /J2-R_N: track 124.0 -> 0.00 mm, vias 4 -> 0
- net /POT5-2: track 0.00 -> 103.6 mm, vias 0 -> 3
- net /POT6-2: track 0.00 -> 103.4 mm, vias 0 -> 3
- net /POT4-2: track 0.00 -> 102.5 mm, vias 0 -> 4
- net /ANA5: track 0.00 -> 58.1 mm, vias 0 -> 1
- net /ANA4: track 0.00 -> 54.6 mm, vias 0 -> 1
- net /ANA3: track 0.00 -> 41.3 mm, vias 0 -> 1
- net +5V: track 28.2 -> 9.43 mm, vias 3 -> 0
- net /J1-T: track 38.0 -> 35.5 mm
- net /ANA7: track 66.5 -> 68.1 mm
Other:
- outline, holes or cut-outs redrawn
- board text added: "REV 2"
- board text removed: "REV 1"

Commit message: CARD DOC UPDATES
Connections:
- net /POT1-2 renamed /ANA0
- net /POT2-2 renamed /ANA1
- net /POT3-2 renamed /ANA2
- C15 pad 1: /J6-R_N -> /J6-T
- J7 pad 3: /J6-R_N -> /POT5-2
- J7 pad 4: /J6-R_N -> /J2-T
- J7 pad 7: /POT5-2 -> Net-(J7-Pad7)
- J7 pad 8: /J2-T -> /J6-T
- R14 pad 2: /J6-R_N -> /J6-T
Routing:
- net /J6-T: track 0.00 -> 13.6 mm, vias 0 -> 1
- net +5V: track 9.43 -> 19.8 mm, vias 0 -> 1
- net /J6-R_N: track 7.88 -> 0.00 mm
- net /J2-T: track 27.5 -> 32.3 mm, vias 0 -> 2
- net /POT5-2: track 103.6 -> 105.9 mm
- net /J4-T: track 20.4 -> 21.5 mm
Other:
- board text added: "REV 3"
- board text removed: "REV 2"
