File: SYNTHS/ER-PROTO-02_SET/ER-PROTO-02_S-H/ER-PROTO-02_S-H.kicad_pcb (KiCad board)
At the start: 2 copper layers, 28 x 110 mm, 30 parts, among them J9 HDR, IDC, 2x5, Q1 2N3904, U1 LF398_DIP8, U2 CD4093, U3 LF398_DIP8

Commit message: CARD DOC UPDATES
Parts:
- removed R10: 2.2K, Resistor_THT:R_Axial_DIN0204_L3.6mm_D1.6mm_P2.54mm_Vertical
- removed R8: 10K, Resistor_THT:R_Axial_DIN0204_L3.6mm_D1.6mm_P2.54mm_Vertical
- removed R9: 4.7K, Resistor_THT:R_Axial_DIN0204_L3.6mm_D1.6mm_P2.54mm_Vertical
- removed RX3, RX6: 1K, Resistor_THT:R_Axial_DIN0204_L3.6mm_D1.6mm_P2.54mm_Vertical
- added J15: Conn_01x10, Connector_PinHeader_2.54mm:PinHeader_1x10_P2.54mm_Vertical, F.Cu at (68.3, 78.9)
- added J28: PROTO02_POTS, Connector_PinHeader_2.54mm:PinHeader_2x10_P2.54mm_Vertical, F.Cu at (61.1, 78.9)
- added J29: PROTO02_JACKS, Connector_PinHeader_2.54mm:PinHeader_2x08_P2.54mm_Vertical, F.Cu at (73.0, 78.9)
- added R3: 10K, Resistor_THT:R_Axial_DIN0204_L3.6mm_D1.6mm_P2.54mm_Vertical, F.Cu at (79.4, 78.2)
- added R6: 1.8K, Resistor_THT:R_Axial_DIN0204_L3.6mm_D1.6mm_P2.54mm_Vertical, F.Cu at (79.4, 87.6)
- added RX1: 2.2K, Resistor_THT:R_Axial_DIN0204_L3.6mm_D1.6mm_P2.54mm_Vertical, F.Cu at (66.0, 105.7)
- added RX11: 4.7K, Resistor_THT:R_Axial_DIN0204_L3.6mm_D1.6mm_P2.54mm_Vertical, F.Cu at (79.4, 81.3)
- added RX12: 4.7K, Resistor_THT:R_Axial_DIN0204_L3.6mm_D1.6mm_P2.54mm_Vertical, F.Cu at (85.0, 78.2)
- added RX15: 1K, Resistor_THT:R_Axial_DIN0204_L3.6mm_D1.6mm_P2.54mm_Vertical, F.Cu at (85.0, 81.3)
- added RX17: 1K, Resistor_THT:R_Axial_DIN0204_L3.6mm_D1.6mm_P2.54mm_Vertical, F.Cu at (79.4, 90.8)
- added RX2: 2.2K, Resistor_THT:R_Axial_DIN0204_L3.6mm_D1.6mm_P2.54mm_Vertical, F.Cu at (79.4, 84.5)
- added RX7: 4.7K, Resistor_THT:R_Axial_DIN0204_L3.6mm_D1.6mm_P2.54mm_Vertical, F.Cu at (60.4, 105.7)
- added RX9: 4.7K, Resistor_THT:R_Axial_DIN0204_L3.6mm_D1.6mm_P2.54mm_Vertical, F.Cu at (85.0, 84.5)
- D1, D2: value 1N4148 -> 1N5218
- R4: value 2.2K -> 10K
- R7: value 1.8K -> 2.7K
Connections:
- net Net-(D4-Pad1) renamed /J1-T
- C1 pad 1: Net-(C1-Pad1) -> /POT1-2
- DS1 pad 1: Net-(DS1-Pad1) -> /LED-
- JX1 pad T: /TRIG_IN -> Net-(JX1-PadT)
- JX1 pad TN: /INT_CLK -> Net-(JX1-PadTN)
- JX3 pad T: /SH_IN_1 -> Net-(JX3-PadT)
- JX4 pad T: /SH_IN2 -> /SH_OUT_2
- JX5 pad T: /SH_OUT_2 -> Net-(JX5-PadT)
- Q1 pad 3: Net-(DS1-Pad1) -> Net-(Q1-Pad3)
- R4 pad 1: /INT_CLK -> GND
- R4 pad 2: Net-(R4-Pad2) -> Net-(C6-Pad2)
- R7 pad 1: GND -> Net-(Q1-Pad3)
- R7 pad 2: /SAM_CLK -> +12V
- RVX1 pad 1: Net-(R4-Pad2) -> /INT_CLK
- RVX1 pad 2: Net-(C1-Pad1) -> Net-(RVX1-Pad2)
- RVX1 pad 3: Net-(C1-Pad1) -> unconnected-(RVX1-Pad3)
- U1 pad 3: /SH_IN_1 -> /J3-T
- U1 pad 5: Net-(RX3-Pad1) -> /J4-T
- U2 pad 1: Net-(C1-Pad1) -> /POT1-2
- U2 pad 2: Net-(C1-Pad1) -> /POT1-2
- U2 pad 5: Net-(DS1-Pad1) -> Net-(Q1-Pad3)
- U2 pad 6: Net-(DS1-Pad1) -> Net-(Q1-Pad3)
- U3 pad 3: /SH_IN2 -> /J5-T
- U3 pad 5: Net-(RX6-Pad1) -> /J6-T
