File: SYNTHS/ER-PROTO-02_SET/ER-DELAY-02/ER-DELAY-02.kicad_pcb (KiCad board)
At the start: 2 copper layers, 28 x 108.5 mm, 47 parts, among them J11 JUMPER, J14 JUMPER, J15 Conn_01x10, J28 PROTO02_POTS, J29 PROTO02_JACKS, J5 PJ-398, J6 PJ-398, J7 PROTO02_JACKS, J8 PROTO02_POTS, J9 ER-PWR-2X5, U1 PT2399, U2 L78L05_TO92

Commit message: cards
Parts:
- removed C17: 4.7uF, Capacitor_THT:CP_Radial_D5.0mm_P2.50mm
- removed J11, J14: JUMPER, Connector_PinHeader_1.00mm:PinHeader_1x02_P1.00mm_Vertical
- removed J5, J6: PJ-398, AudioJacks:Jack_3.5mm_QingPu_WQP-PJ366ST_Vertical
- removed J7: PROTO02_JACKS, Connector_PinHeader_2.54mm:PinHeader_2x08_P2.54mm_Vertical
- removed J8: PROTO02_POTS, Connector_PinHeader_2.54mm:PinHeader_2x10_P2.54mm_Vertical
- removed RA1: 10, Resistor_THT:R_Axial_DIN0204_L3.6mm_D1.6mm_P2.54mm_Vertical
- removed RB1: 18K, Resistor_THT:R_Axial_DIN0204_L3.6mm_D1.6mm_P2.54mm_Vertical
- removed RB7: 0, Resistor_THT:R_Axial_DIN0204_L3.6mm_D1.6mm_P2.54mm_Vertical
- removed RV1: 50K, LandBoards_Conns:RV09ACF
- removed RV2: 20K, LandBoards_Conns:RV09ACF
- added C19: 47pF, Capacitor_THT:C_Rect_L4.0mm_W2.5mm_P2.50mm, B.Cu at (140.9, 42.4)
- added C21: 0.22uF, Capacitor_THT:C_Rect_L4.0mm_W2.5mm_P2.50mm, B.Cu at (140.9, 46.5)
- added C22: 2.2nF, Capacitor_THT:C_Rect_L4.0mm_W2.5mm_P2.50mm, B.Cu at (140.9, 50.5)
- added C23: 1uF, Capacitor_THT:CP_Radial_D5.0mm_P2.50mm, B.Cu at (144.0, 34.3)
- added C24: 4.7nF, Capacitor_THT:C_Rect_L4.0mm_W2.5mm_P2.50mm, B.Cu at (140.9, 54.6)
- added D2: BAT41, Diode_THT:D_DO-35_SOD27_P2.54mm_Vertical_KathodeUp, B.Cu at (142.0, 71.9)
- added JX1: JUMPER, Connector_PinHeader_1.00mm:PinHeader_1x02_P1.00mm_Vertical, B.Cu at (140.2, 76.7)
- added JX13: JUMPER, Connector_PinHeader_1.00mm:PinHeader_1x02_P1.00mm_Vertical, B.Cu at (136.9, 76.7)
- added JX14: JUMPER, Connector_PinHeader_1.00mm:PinHeader_1x02_P1.00mm_Vertical, B.Cu at (145.3, 71.5)
- added JX5: PJ-398, AudioJacks:Jack_3.5mm_QingPu_WQP-PJ366ST_Vertical, F.Cu at (155.0, 102.4)
- added JX6: PJ-398, AudioJacks:Jack_3.5mm_QingPu_WQP-PJ366ST_Vertical, F.Cu at (168.0, 101.7)
- added JX7: PROTO02_JACKS, Connector_PinHeader_2.54mm:PinHeader_2x08_P2.54mm_Vertical, F.Cu at (124.0, 105.4)
- added JX8: PROTO02_POTS, Connector_PinHeader_2.54mm:PinHeader_2x10_P2.54mm_Vertical, F.Cu at (124.5, 17.8)
- added R10: 1M, Resistor_THT:R_Axial_DIN0204_L3.6mm_D1.6mm_P2.54mm_Vertical, B.Cu at (144.6, 20.0)
- added R11: 10K, Resistor_THT:R_Axial_DIN0204_L3.6mm_D1.6mm_P2.54mm_Vertical, B.Cu at (144.6, 23.1)
- added R14: 100K, Resistor_THT:R_Axial_DIN0204_L3.6mm_D1.6mm_P2.54mm_Vertical, B.Cu at (144.6, 26.3)
- added R15: 100K, Resistor_THT:R_Axial_DIN0204_L3.6mm_D1.6mm_P2.54mm_Vertical, B.Cu at (144.6, 29.4)
- added R16: 1M, Resistor_THT:R_Axial_DIN0204_L3.6mm_D1.6mm_P2.54mm_Vertical, B.Cu at (139.0, 16.8)
- added R18: 10K, Resistor_THT:R_Axial_DIN0204_L3.6mm_D1.6mm_P2.54mm_Vertical, B.Cu at (139.0, 20.0)
- added R19: 68K, Resistor_THT:R_Axial_DIN0204_L3.6mm_D1.6mm_P2.54mm_Vertical, B.Cu at (139.0, 23.1)
- added R2: 10, Resistor_THT:R_Axial_DIN0204_L3.6mm_D1.6mm_P2.54mm_Vertical, B.Cu at (144.6, 16.8)
- added R20: 100K, Resistor_THT:R_Axial_DIN0204_L3.6mm_D1.6mm_P2.54mm_Vertical, B.Cu at (139.0, 26.3)
- added RBX3: 0, Resistor_THT:R_Axial_DIN0204_L3.6mm_D1.6mm_P2.54mm_Vertical, B.Cu at (139.0, 29.4)
- added RVX1: B50K, LandBoards_Conns:RV09ACF, F.Cu at (156.6, 31.8)
- added RVX2: B10K, LandBoards_Conns:RV09ACF, F.Cu at (169.2, 32.0)
- added RVX3: B10K, LandBoards_Conns:RV09ACF, F.Cu at (156.5, 46.7)
- added RX1: 1K, Resistor_THT:R_Axial_DIN0204_L3.6mm_D1.6mm_P2.54mm_Vertical, B.Cu at (133.4, 16.8)
- added RX17: 1K, Resistor_THT:R_Axial_DIN0204_L3.6mm_D1.6mm_P2.54mm_Vertical, B.Cu at (133.4, 26.3)
- added RX4: 0, Resistor_THT:R_Axial_DIN0204_L3.6mm_D1.6mm_P2.54mm_Vertical, B.Cu at (133.4, 20.0)
- added RX7: 0, Resistor_THT:R_Axial_DIN0204_L3.6mm_D1.6mm_P2.54mm_Vertical, B.Cu at (133.4, 23.1)
- added U3: L78L05_TO92, Package_TO_SOT_THT:TO-92_Inline, B.Cu at (137.5, 34.2)
- C11: value 560pF -> 2.2uF
- C12: value 10uF -> 10nF
- C13: value 0.01uF -> 2.2uF
- C14: value 10uF -> 47uF
- C15: value 4.7uF -> 47pF; footprint Capacitor_THT:CP_Radial_D5.0mm_P2.50mm -> Capacitor_THT:C_Rect_L4.0mm_W2.5mm_P2.50mm
- C16: value 3.3nF -> 0.1uF
- C3: value 47uF -> 1uF
- C6, C7: value 82nF -> 100nF
- C8: value 560pF -> 2.2nF
- C9: value 3.3nF -> 15nF
- R1: value 1K -> 10
- R12: value 15K -> 100K
- R13: value 100K -> 10K
- R17: value 0 -> 100K; moved to B.Cu
- R5: value 15K -> 20K
- R8: value 4.7K -> 20K
- R9: value 5.6K -> 10K
- U2: value L78L05_TO92 -> PT2399; footprint Package_TO_SOT_THT:TO-92_Inline -> Package_DIP:DIP-16_W7.62mm_LongPads
- moved R17 63.9 mm to (139.4, 64.3)
- moved U2 39.9 mm to (109.2, 55.9), turned to 0 degrees
- moved C9 18.6 mm to (95.7, 70.4)
- moved U1 17.8 mm to (109.2, 81.3)
- moved C3 16.9 mm to (92.8, 77.5)
- moved C4 12.9 mm to (103.1, 40.7)
- moved C7 7.69 mm to (119.9, 38.1)
- moved C11 7.67 mm to (119.9, 55.9)
- moved C6 7.67 mm to (119.9, 43.2)
- moved C8 7.67 mm to (119.9, 50.8)
- moved C5 7.65 mm to (105.9, 38.1)
Connections:
- C11 pad 1: Net-(C11-Pad1) -> /P16
- C11 pad 2: Net-(C11-Pad2) -> /P15
- C12 pad 2: /POT1-3 -> Net-(U1C-+)
- C14 pad 1: Net-(C14-Pad1) -> GND
- C14 pad 2: /OUT -> Net-(U1E-V-)
- C15 pad 1: Net-(C15-Pad1) -> Net-(U1D--)
- C15 pad 2: /POT1-2 -> /OUT
- C16 pad 1: Net-(C15-Pad1) -> Net-(U1E-V-)
- C3 pad 1: Net-(C3-Pad1) -> /P2
- C4 pad 1: Net-(C4-Pad1) -> /P7
- C5 pad 1: Net-(C5-Pad1) -> /P8
- C6 pad 1: Net-(C6-Pad1) -> /P11
- C6 pad 2: Net-(C6-Pad2) -> /P12
- C7 pad 1: Net-(C7-Pad1) -> /P9
- C7 pad 2: Net-(C7-Pad2) -> /P10
- C8 pad 1: Net-(C8-Pad1) -> /P14
- C8 pad 2: Net-(C8-Pad2) -> /P13
- D1 pad 2: Net-(D1-Pad2) -> Net-(D1-A)
- J15 pad 10: unconnected-(J15-Pad10) -> -12V
- J15 pad 6: unconnected-(J15-Pad6) -> -12V
- J15 pad 7: unconnected-(J15-Pad7) -> -12V
- J15 pad 8: unconnected-(J15-Pad8) -> -12V
- J15 pad 9: unconnected-(J15-Pad9) -> -12V
- J28 pad 10: unconnected-(J28-Pad10) -> /BUF
- J28 pad 14: /POT3-1 -> unconnected-(J28-POT3_1_CW-Pad14)
- J28 pad 15: /POT3-2 -> /WET
- J28 pad 16: /POT3-3 -> /BUF
- J28 pad 18: /POT1-2 -> /VCO
- J28 pad 19: /POT1-3 -> unconnected-(J28-POT1_3_CCW-Pad19)
- J28 pad 8: /VCO -> unconnected-(J28-POT2_1_CW-Pad8)
- J28 pad 9: unconnected-(J28-Pad9) -> /REPEAT
- J29 pad 6: /J4-T -> unconnected-(J29-J4_T-Pad6)
- J9 pad 1: unconnected-(J9-Pad1) -> -12VA
- J9 pad 2: unconnected-(J9-Pad2) -> -12VA
- R1 pad 1: Net-(R1-Pad1) -> Net-(D1-A)
- R1 pad 2: /VCO -> +12VA
- R12 pad 1: Net-(C17-Pad1) -> Net-(U1C--)
- R12 pad 2: Net-(C15-Pad1) -> /BUF
- R13 pad 1: GND -> /OUT
- R13 pad 2: /IN -> Net-(U1D--)
- R17 pad 2: Net-(J7-Pad8) -> /DRY
- R3 pad 2: Net-(C6-Pad2) -> /P12
- R4 pad 2: Net-(C8-Pad2) -> /P13
- R5 pad 2: Net-(C8-Pad1) -> /P14
- R6 pad 1: Net-(C11-Pad2) -> /P15
- R6 pad 2: Net-(C15-Pad1) -> Net-(C24-Pad2)
- R7 pad 1: Net-(C11-Pad1) -> /P16
- R7 pad 2: Net-(C15-Pad1) -> Net-(C24-Pad2)
- R8 pad 1: Net-(C11-Pad2) -> Net-(U1C--)
- R8 pad 2: Net-(C14-Pad1) -> GND
- R9 pad 1: Net-(C8-Pad1) -> /P14
- U2 pad 2: GND -> /P2
- U2 pad 3: +12V -> GND
Routing:
- net unconnected-(J7-Pad5): track 7.86 -> 0.00 mm
- net unconnected-(J29-J4_R_N-Pad5): track 0.00 -> 7.86 mm
- net unconnected-(J7-Pad4): track 7.72 -> 0.00 mm
- net unconnected-(J29-J2_T-Pad4): track 0.00 -> 7.72 mm
- net unconnected-(J7-Pad3): track 7.56 -> 0.00 mm
- net unconnected-(J29-J2_R_N-Pad3): track 0.00 -> 7.56 mm
- net unconnected-(J7-Pad6): track 7.56 -> 0.00 mm
- net unconnected-(J29-J4_T-Pad6): track 0.00 -> 7.56 mm
- net Net-(J7-Pad14): track 7.29 -> 0.00 mm
- net /IN: track 0.00 -> 7.29 mm
- net unconnected-(J7-Pad12): track 7.29 -> 0.00 mm
- net unconnected-(J29-J3_T-Pad12): track 0.00 -> 7.29 mm
- added copper zone on F.Cu, net -12V
- added copper zone on F.Cu, net -12VA
- removed copper zone on F.Cu, net unconnected-(J15-Pad10)
- removed copper zone on F.Cu, net unconnected-(J9-Pad2)
