File: SYNTHS/ER-MIXER5-02_SET/ER-MIXER5-02/ER-MIXER5-02.kicad_sch (KiCad schematic)
At the start: 30 parts, among them J1 PJ-398SM, J2 PJ-398SM, J3 PJ-398SM, J4 PJ-398SM, J5 PJ-398SM, J6 PJ-398SM, J8 Conn_02x05, U1 TL072

Commit message: card updates
Parts:
- C3, C4: value 10uF -> 47uF
- RV1, RV2, RV3, RV4, RV5, RV6: value B100K -> 100K
Other:
- title: SYNTH-MIXER5-01 -> SYNTH-MIXER5-02
