File: SYNTHS/ER-MIXER5-02_SET/ER-MIXER5-02/ER-MIXER5-02.kicad_pcb (KiCad board)
At the start: 2 copper layers, 28 x 111.5 mm, 30 parts, among them J1 PJ-398SM, J2 PJ-398SM, J3 PJ-398SM, J4 PJ-398SM, J5 PJ-398SM, J6 PJ-398SM, J8 Conn_02x05, U1 TL072

Commit message: cards
Parts:
- moved RV2 0.11 mm to (8.60, 15.0)
- moved J5 0.10 mm to (22.6, 73.0)
- moved RV1 0.10 mm to (22.6, 44.0)
- moved RV3 0.10 mm to (22.6, 15.0)
- moved RV5 0.10 mm to (22.6, 29.5)
- moved J4 0.10 mm to (8.60, 73.0)
- moved RV4 0.10 mm to (8.60, 29.5)
- moved RV6 0.10 mm to (8.60, 44.0)
Changed lines of the file:
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@@
   (net 23 "Net-(D2-K)")
   (footprint "LandBoards_Conns:RV09ACF" (layer "F.Cu")
-    (at 22.5 29.5 90)
+    (at 22.6 29.5 90)
     (descr "Potentiometer, vertical, Bourns PTV09A-1 Single, http://www.bourns.com/docs/Product-Datasheets/ptv09.pdf")
     (tags "Potentiometer vertical Bourns PTV09A-1 Single")
@@
   )
   (footprint "LandBoards_Conns:RV09ACF" (layer "F.Cu")
-    (at 22.5 44 90)
+    (at 22.6 44 90)
     (descr "Potentiometer, vertical, Bourns PTV09A-1 Single, http://www.bourns.com/docs/Product-Datasheets/ptv09.pdf")
     (tags "Potentiometer vertical Bourns PTV09A-1 Single")
@@
   )
   (footprint "LandBoards_Conns:RV09ACF" (layer "F.Cu")
-    (at 22.5 15 90)
+    (at 22.6 15 90)
     (descr "Potentiometer, vertical, Bourns PTV09A-1 Single, http://www.bourns.com/docs/Product-Datasheets/ptv09.pdf")
     (tags "Potentiometer vertical Bourns PTV09A-1 Single")
@@
   )
   (footprint "LandBoards_Conns:RV09ACF" (layer "F.Cu")
-    (at 8.5 44 90)
+    (at 8.6 44 90)
     (descr "Potentiometer, vertical, Bourns PTV09A-1 Single, http://www.bourns.com/docs/Product-Datasheets/ptv09.pdf")
     (tags "Potentiometer vertical Bourns PTV09A-1 Single")
@@
   )
   (footprint "AudioJacks:Jack_3.5mm_QingPu_WQP-PJ398SM_Vertical" (layer "F.Cu")
-    (at 22.5 73)
+    (at 22.6 73)
     (descr "T-S-SN Vertical mount jack AKA WQP-WQP518MA or Thonkiconn")
     (tags "WQP-WQP518MA, Thonkiconn")
@@
   )
   (footprint "AudioJacks:Jack_3.5mm_QingPu_WQP-PJ398SM_Vertical" (layer "F.Cu")
-    (at 8.55 87.5)
+    (at 8.6 87.5)
     (descr "T-S-SN Vertical mount jack AKA WQP-WQP518MA or Thonkiconn")
     (tags "WQP-WQP518MA, Thonkiconn")
@@
   )
   (footprint "AudioJacks:Jack_3.5mm_QingPu_WQP-PJ398SM_Vertical" (layer "F.Cu")
-    (at 8.636 58.5)
+    (at 8.6 58.5)
     (descr "T-S-SN Vertical mount jack AKA WQP-WQP518MA or Thonkiconn")
     (tags "WQP-WQP518MA, Thonkiconn")
@@
   )
   (footprint "AudioJacks:Jack_3.5mm_QingPu_WQP-PJ398SM_Vertical" (layer "F.Cu")
-    (at 8.5 73)
+    (at 8.6 73)
     (descr "T-S-SN Vertical mount jack AKA WQP-WQP518MA or Thonkiconn")
     (tags "WQP-WQP518MA, Thonkiconn")
@@
   )
   (footprint "LandBoards_Conns:RV09ACF" (layer "F.Cu")
-    (at 8.5 15.05 90)
+    (at 8.6 15 90)
     (descr "Potentiometer, vertical, Bourns PTV09A-1 Single, http://www.bourns.com/docs/Product-Datasheets/ptv09.pdf")
     (tags "Potentiometer vertical Bourns PTV09A-1 Single")
@@
   )
   (footprint "LandBoards_Conns:RV09ACF" (layer "F.Cu")
-    (at 8.5 29.5 90)
+    (at 8.6 29.5 90)
     (descr "Potentiometer, vertical, Bourns PTV09A-1 Single, http://www.bourns.com/docs/Product-Datasheets/ptv09.pdf")
     (tags "Potentiometer vertical Bourns PTV09A-1 Single")
@@
   )
   (footprint "AudioJacks:Jack_3.5mm_QingPu_WQP-PJ398SM_Vertical" (layer "F.Cu")
-    (at 22.606 58.5)
+    (at 22.6 58.5)
     (descr "T-S-SN Vertical mount jack AKA WQP-WQP518MA or Thonkiconn")
     (tags "WQP-WQP518MA, Thonkiconn")

Commit message: card updates
Parts:
- C3, C4: value 10uF -> 47uF
- RV1, RV2, RV3, RV4, RV5, RV6: value B100K -> 100K
- moved C5 3.25 mm to (16.4, 97.1), turned to 180 degrees
- moved R9 3.05 mm to (13.8, 94.5)
- moved R7 2.85 mm to (5.62, 96.0), turned to 180 degrees
Routing:
- net /VSUM: track 106.8 -> 101.7 mm
- net /VOL1: track 51.2 -> 48.2 mm
- net /VOL2: track 59.3 -> 61.5 mm
- net /VO: track 13.9 -> 11.9 mm
- net Net-(R7-Pad2): track 37.6 -> 38.7 mm
Other:
- board text added: "REV 2"
- board text removed: "REV 1"

Commit message: ER-VCF-02 working
Other:
- outline, holes or cut-outs redrawn
- board text added: "[A] [B] POTS"
Changed lines of the file:
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@@
         (effects (font (size 1 1) (thickness 0.15)))
     )
-    (fp_text user "K" (at -1.8 0 90) (layer "F.SilkS")
+    (fp_text user "K" (at -0.078315 1.63 90) (layer "F.SilkS")
         (effects (font (size 1 1) (thickness 0.15)))
     )
@@
   (gr_circle (center 62.5 73) (end 64.5 73)
     (stroke (width 0.15) (type solid)) (fill none) (layer "Dwgs.User"))
+  (gr_circle (center 8.6 73) (end 10.1 73)
+    (stroke (width 0.1) (type default)) (fill none) (layer "Edge.Cuts"))
+  (gr_circle (center 8.6 87.5) (end 10.1 87.5)
+    (stroke (width 0.1) (type default)) (fill none) (layer "Edge.Cuts"))
   (gr_rect (start 1.1 8.5) (end 29.1 120)
     (stroke (width 0.1) (type solid)) (fill none) (layer "Edge.Cuts"))
+  (gr_circle (center 22.6 87.5) (end 24.1 87.5)
+    (stroke (width 0.1) (type default)) (fill none) (layer "Edge.Cuts"))
+  (gr_circle (center 22.6 73) (end 24.1 73)
+    (stroke (width 0.1) (type default)) (fill none) (layer "Edge.Cuts"))
+  (gr_circle (center 22.6 58.5) (end 24.1 58.5)
+    (stroke (width 0.1) (type default)) (fill none) (layer "Edge.Cuts"))
+  (gr_circle (center 8.6 58.5) (end 10.1 58.5)
+    (stroke (width 0.1) (type default)) (fill none) (layer "Edge.Cuts"))
   (gr_text "REV 2" (at 8.75 98.5) (layer "B.SilkS")
     (effects (font (size 1.25 1.25) (thickness 0.3125)) (justify mirror))
@@
   (gr_text "TL072" (at 18.2 104.648) (layer "B.SilkS")
     (effects (font (size 1.905 1.524) (thickness 0.381)) (justify left mirror))
+  )
+  (gr_text "[A] [B] POTS" (at 16 17.9) (layer "B.SilkS")
+    (effects (font (size 1.25 1.25) (thickness 0.3125)) (justify mirror))
   )
   (gr_text "land-boards.com/\nER-MIXER5-02" (at 15 11) (layer "B.SilkS")
@@
     (pts (xy 46.499998 128.5) (xy 62 128.5))
     (height 4.000003)
-    (gr_text "610.2363 mils" (at 54.249999 131.350003) (layer "Dwgs.User")
+    (gr_text "15.5000 mm" (at 54.249999 131.350003) (layer "Dwgs.User")
       (effects (font (size 1 1) (thickness 0.15)))
     )
@@
     (pts (xy 39.999996 128.499997) (xy 40 125.5))
     (height 40)
-    (gr_text "118.1101 mils" (at 78.849998 127.00005 89.99992361) (layer "Dwgs.User")
+    (gr_text "3.0000 mm" (at 78.849998 127.00005 89.99992361) (layer "Dwgs.User")
       (effects (font (size 1 1) (thickness 0.15)))
     )
@@
     (pts (xy 39.999996 0) (xy 39.999996 3))
     (height -39.750004)
-    (gr_text "118.1 mils" (at 78.6 1.5 90) (layer "Dwgs.User")
+    (gr_text "3.0 mm" (at 78.6 1.5 90) (layer "Dwgs.User")
       (effects (font (size 1 1) (thickness 0.15)))
     )
@@
     (pts (xy 62 128.5) (xy 70.000012 128.499997))
     (height 4.000003)
-    (gr_text "314.9611 mils" (at 66.000007 131.350001 2.864784676e-05) (layer "Dwgs.User")
+    (gr_text "8.0000 mm" (at 66.000007 131.350001 2.864784676e-05) (layer "Dwgs.User")
       (effects (font (size 1 1) (thickness 0.15)))
     )
@@
   (segment (start 16.35 97.1) (end 16.35 94.53) (width 0.25) (layer "F.Cu") (net 14))
   (segment (start 16.35 97.1) (end 16.35 100.670012) (width 0.25) (layer "B.Cu") (net 14))
-  (segment (start 16.35 100.670012) (end 16.36 100.680012) (width 0.25) (layer "B.Cu") (net 14))
   (segment (start 7.375 52.535) (end 8.5 53.66) (width 0.25) (layer "F.Cu") (net 15))
   (segment (start 7.375 29.875) (end 7.375 52.535) (width 0.25) (layer "F.Cu") (net 15))
