File: SYNTHS/ER-ADSR-555-01_SET/ER-ADSR-555-01-controls/ER-ADSR-555-01.kicad_sch (KiCad schematic)
At the start: 32 parts, among them J1 Conn_02x05, J2 PJ-301BM, J3 PJ-301BM, Q1 2N3904, Q2 2N3904, Q3 2N3904, U1 TL072, U2 LM555N

Commit message: SYNTHS
Parts:
- added R7: 1M, Resistor_THT:R_Axial_DIN0204_L3.6mm_D1.6mm_P7.62mm_Horizontal, symbol Device:R
- C1: value 0.1uF -> 10nF
- C3: value 1uF -> 4.7uF
- R11: renamed from R10; value 100 -> RR
- R8: renamed from R7; value 100 -> RA
- R9: renamed from R8; value 100 -> RD
- renumbered R9 to R10, R11 to R12
Connections:
- net BUFA: now also R7.1
- net BUFC: now reaches Q3.2 (B), R5.2
- net at Q1.3 (C), R2.1, R3.1: now also R7.2
- net BUFB: now reaches Q2.2 (B), R2.2
- net DIS renamed DISCH
- net RES renamed RST
- net TR renamed TRIG
Other:
- note added: "RA=220 RD=220 RR=220"
- moved on the sheet: C1, C2, C3, D1, D2, D3, D4, D5, D6, J1, J2, J3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

Commit message: ADSR working
Parts:
- removed R7: 1M, Resistor_THT:R_Axial_DIN0204_L3.6mm_D1.6mm_P7.62mm_Horizontal, symbol Device:R
- removed RV1, RV2, RV4: 1M, LandBoards_Conns:RV09ACF, symbol LandBoards:POT
- removed RV3: 10K, LandBoards_Conns:RV09ACF, symbol LandBoards:POT
- added C4, C5, C6: 0.1uF, Capacitor_THT:C_Rect_L4.0mm_W2.5mm_P2.50mm, symbol Device:C
- added R4: 10K, Resistor_THT:R_Axial_DIN0204_L3.6mm_D1.6mm_P7.62mm_Horizontal, symbol Device:R
- added RV1, RV2, RV4: A1M, LandBoards_Conns:RV09ACF, symbol LandBoards_Conns:R_Pot_CW_PIN3UP
- added RV3: A1M, LandBoards_Conns:RV09ACF, symbol LandBoards_Conns:R_Pot_CW
- C3: value 4.7uF -> 1uF
- D1: value BAT41 -> 1N4148
- Q1, Q2, Q3: footprint Package_TO_SOT_THT:TO-92_Inline -> Package_TO_SOT_THT:TO-92_HandSolder
- R11: value RR -> 100
- R8: value RA -> 100
- R9: value RD -> 100
- renumbered D6 to DS1, R4 to R5, R5 to R6, R6 to R7
Connections:
- net +12V: now also C4.2, C5.2
- net -12V: now also C6.1
- net ATT: now also RV1.1, RV1.2
- net BUFA: now also R4.1
- net DEC: now also RV2.1, RV2.2
- net DISCH: now also RV3.3
- net GND: now also C4.1, C5.1, C6.2
- net REL: now also RV4.1, RV4.2
- net RST: now also R4.2
- net SUSPOT: now also RV3.2
- net at D4.2 (A): now also RV1.3
- net at D5.1 (K): now also RV2.3
- net at D3.1 (K): now also RV4.3
- net at R10.1: now also RV3.1
Other:
- note added: "ADDED IN REWORK"
- title: (none) -> ADSR GENERATOR
- moved on the sheet: C1, C2, C3, D1, D2, D3, D4, D5, DS1, J2, J3, Q1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

Commit message: SHUFFLE PLUS ADD PICS
Other:
- note added: "RA=100 RD=100 RR=100"
- note removed: "RA=220 RD=220 RR=220"
Changed lines of the file:
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@@
     (effects (font (size 1.905 1.905) (thickness 0.381) bold) (justify left bottom))
   )
-  (text "RA=220\nRD=220\nRR=220" (at 118.11 192.405 0)
+  (text "RA=100\nRD=100\nRR=100" (at 118.11 192.405 0)
     (effects (font (size 2.54 2.54) (thickness 0.508) bold) (justify left bottom))
   )

Commit message: SAMPLE AND HOLD
Parts:
- added R13: 10K, Resistor_THT:R_Axial_DIN0204_L3.6mm_D1.6mm_P7.62mm_Horizontal, symbol Device:R
- R4: value 10K -> 1M
- RV3: value A1M -> B10K
Connections:
- net BUFC: now also R13.2
- net GND: now also R13.1
Other:
- note added: "3.3K BUFC to GND"

Commit message: cards
Parts:
- removed D1, D2, D3, D4, D5: 1N4148, Diode_THT:D_DO-35_SOD27_P7.62mm_Horizontal, symbol Device:D_Schottky
- added D1, D2, D3, D4, D5: 1N4148, Diode_THT:D_DO-35_SOD27_P7.62mm_Horizontal, symbol Device:D_Small
Connections:
- net BUFA: now also D1.1 (K)
- net GND: now also D1.2 (A), D2.2 (A)
- net THR: now also D3.2 (A), D4.1 (K), D5.2 (A)
- net at C1.2, R6.1: now also D2.1 (K)
- net at RV2.3: now also D5.1 (K)
- net at RV1.3: now also D4.2 (A)
- net at RV4.3: now also D3.1 (K)
Other:
- note added: "R13 - 3.3K BUFC to GND"
- note removed: "3.3K BUFC to GND"
- note removed: "ADDED IN REWORK"
- moved on the sheet: C1, J2, Q1, Q2, Q3, R1, R13, R2, R3, R4, R5, R6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
